File: LRUs/Pad Control Unit/Electrical/Main Controller Board/KICAD PROJECT/master_gse_pcb_project/master_gse_pcb_project.kicad_pcb (KiCad board)
At the start: 6 copper layers, 200 x 150 mm, 554 parts, among them J1 Conn_01x02_Pin, J10 B3B-XH-A, J11 Conn_02x04_Odd_Even, J12 Conn_Coaxial, J13 Conn_01x02_Pin, J14 B4B-XH-A, J15 1x2 Screw Terminal, J16 1x2 Screw Terminal, J17 B4B-XH-A, J18 B4B-XH-A, J19 B5B-XH-A, J2 RAPC722X, J20 B5B-XH-A, J21 B5B-XH-A, J22 B5B-XH-A, J23 B2B-XH-A, J24 B2B-XH-A, J25 61202021721, J26 61200621721, J27 09242206824, J3 Conn_01x02_Pin, J4 B2B-XH-A, J5 GSB1C41110SSHR, J6 Conn_ST_STDC14, J7 Micro_SD_Card_Det2, J8 B3B-XH-A, J9 B3B-XH-A, K1 J107F1CS205VDC.45, Q1 AO3400A, Q10 AO3400A, Q11 AO3400A, Q12 STD52P3LLH6, Q13 AO3400A, Q14 AO3400A, Q15 SS8550, Q16 SS8550, Q17 SS8550, Q18 SS8550, Q19 AO3400A, Q2 AO3400A, Q20 AO3400A, Q3 SiR882ADP, Q4 SiR882ADP, Q5 SiR882ADP, Q6 SiR882ADP, Q7 AO3400A, Q8 AO3400A, Q9 AO3400A, SW1 SW_SPDT, SW2 SW_Push, U1 LTC4359-MS8, U10 TPS22917DBV, U11 TPS22917DBV, U12 AMS1117-3.3, U13 STM32L496ZGTx, U14 TPD6E05U06RVZ, U15 TMP102xxDRL, U16 TMP102xxDRL, U17 74LVC1G17, U18 74LVC1G17, U19 SP485EEN-L/TR, U2 LTC4359-MS8, U20 SP485EEN-L/TR, U21 TJA1051T-3, U22 RFM69HW, U23 TPS259830ONRGER, U24 MAX31856, U25 MAX31856, U26 MAX31856, U27 MAX31856, U28 HX711, U29 HX711, U3 TPS259830ONRGER, U30 HX711, U31 HX711, U32 TPD6E05U06RVZ, U33 TPD6E05U06RVZ, U4 TPS62933P, U5 TPS62933P, U6 TPS62933P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

Commit message: Layout changes
Routing:
- net /power_distribution/3V3_DIGITAL/3V3_EN: track 59.7 -> 61.3 mm
- net GND: track 346.6 -> 345.7 mm, vias 554 -> 553
- added copper zone on B.Cu, net GND
- added copper zone on In3.Cu, net GND
