File: LRUs/Pad Control Unit/Electrical/Main Controller Board/KICAD PROJECT/master_gse_pcb_project/master_gse_pcb_project.kicad_pcb (KiCad board)
At the start: 6 copper layers, 200 x 150 mm, 583 parts, among them J1 XT-60, J10 Micro_SD_Card_Det2, J11 Conn_01x04, J12 B3B-XH-A, J13 Conn_02x04_Odd_Even, J14 Conn_Coaxial, J15 Conn_01x02_Pin, J16 B4B-XH-A, J17 1x2 Screw Terminal, J18 1x2 Screw Terminal, J19 B4B-XH-A, J2 RAPC722X, J20 B4B-XH-A, J21 B5B-XH-A, J22 B5B-XH-A, J23 B5B-XH-A, J24 B5B-XH-A, J25 B2B-XH-A, J26 B2B-XH-A, J27 61202021721, J28 61200621721, J29 09242206824, J3 01x02_PinHeader, J4 B2B-XH-A, J5 01x02_PinHeader, J6 01x02_PinHeader, J7 01x02_PinHeader, J8 GSB1C41110SSHR, J9 Conn_ST_STDC14, K1 J107F1CS205VDC.45, Q1 AO3400A, Q10 AO3400A, Q11 AO3400A, Q12 STD52P3LLH6, Q13 AO3400A, Q14 AO3400A, Q15 SS8550, Q16 SS8550, Q17 SS8550, Q18 SS8550, Q19 AO3400A, Q2 AO3400A, Q20 AO3400A, Q3 SiR882ADP, Q4 SiR882ADP, Q5 SiR882ADP, Q6 SiR882ADP, Q7 AO3400A, Q8 AO3400A, Q9 AO3400A, SW1 SW_SPDT, SW2 SW_Push, U1 LTC4359-MS8, U10 TPS22917DBV, U11 TPS22917DBV, U12 AMS1117-3.3, U13 STM32L496ZGTx, U14 TPD6E05U06RVZ, U15 TMP102A, U16 TMP102A, U17 ADS1115, U18 74LVC1G17, U19 SN6505BDBV, U2 LTC4359-MS8, U20 ISO1450BDWR, U21 AMS1117-5.0, U22 TJA1051T-3, U23 RFM69HW, U24 TPS259830ONRGER, U25 MAX31856, U26 MAX31856, U27 MAX31856, U28 MAX31856, U29 HX711, U3 TPS259830ONRGER, U30 HX711, U31 HX711, U32 HX711, U33 TPD6E05U06RVZ, U34 TPD6E05U06RVZ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

Commit message: Commit da changes
Parts:
- removed C127, C79: 100nF, Capacitor_SMD:C_0402_1005Metric
- added C169: 100nF, Capacitor_SMD:C_0402_1005Metric, F.Cu at (167.0, 117.0)
- added C70: 100nF, Capacitor_SMD:C_0402_1005Metric, F.Cu at (160.8, 189.7)
- added FID1: Fiducial, Fiducial:Fiducial_1mm_Mask3mm, F.Cu at (112.4, 212.1)
- added FID2: Fiducial, Fiducial:Fiducial_1mm_Mask3mm, F.Cu at (107.4, 80.1)
- added FID3: Fiducial, Fiducial:Fiducial_1mm_Mask3mm, F.Cu at (292.4, 80.1)
- added G***: LOGO, LOGO, F.Cu at (254.1, 82.3)
- added G***: LOGO, LOGO, F.Cu at (152.0, 182.8)
- added G***: LOGO, LOGO, F.Cu at (241.7, 196.5)
- added H8: M3 Mount, MountingHole:MountingHole_3.2mm_M3_DIN965_Pad, F.Cu at (204.4, 151.1)
- BZ1: footprint footprints:MURATA_ELECTRONICS_NORTH_AMERICA_PKM22EPPH2002-B0_0 -> Buzzer_Beeper:Buzzer_Murata_PKMCS0909E; moved to F.Cu
- F1: value Fuse -> 0297020
- J10: value Micro_SD_Card_Det2 -> DM3AT-SF-PEJM5
- J11: value Conn_01x04 -> 0436500415
- J13: value Conn_02x04_Odd_Even -> 02x04_PinHeader
- J14: value Conn_Coaxial -> SMA
- J15: value Conn_01x02_Pin -> XT-60
- U13: value STM32L496ZGTx -> STM32L496ZGT6
- moved BZ1 3.69 mm to (148.3, 168.5)
- moved C137 1.80 mm to (168.7, 116.4)
Connections:
- net /top-level/power_distribution/input_muxing/efuse/VIN_UNSAFE renamed /top-level/power_distribution/input_muxing/VIN_UNSAFE
- net Net-(BZ1-+) renamed /top-level/stm32_controller/BUZZ_P
- net Net-(D12-K) renamed /top-level/USB_C/CC1
- net Net-(D14-K) renamed /top-level/USB_C/CC2
- net Net-(D5-A) renamed /top-level/power_distribution/input_muxing/BAT_SRC
- net Net-(D5-K) renamed /top-level/power_distribution/input_muxing/BAT_GATE
- net Net-(D6-A) renamed /top-level/power_distribution/input_muxing/JACK_SRC
- net Net-(D6-K) renamed /top-level/power_distribution/input_muxing/JACK_GATE
- net Net-(J10-CLK) renamed /top-level/SD_card/SD_CLK_PIN
- net Net-(J10-CMD) renamed /top-level/SD_card/SD_MOSI_PIN
- net Net-(J10-DAT0) renamed /top-level/SD_card/SD_MISO_PIN
- net Net-(J10-DAT1) renamed /top-level/SD_card/DAT1_PIN
- net Net-(J10-DAT2) renamed /top-level/SD_card/DAT2_PIN
- net Net-(J10-DAT3/CD) renamed /top-level/SD_card/~{SD_CS_PIN}
- net Net-(J14-In) renamed /top-level/rf/ANT
- net Net-(J4-Pin_1) renamed /top-level/power_distribution/input_muxing/efuse/EN_H
- net Net-(J4-Pin_2) renamed /top-level/power_distribution/input_muxing/efuse/EN_UVLO
- net Net-(J8-SHIELD) renamed /top-level/USB_C/USB_SHIELD
- net Net-(Q1-D) renamed /top-level/power_distribution/input_muxing/~{BAT_SHDN}
- net Net-(Q1-G) renamed /top-level/power_distribution/input_muxing/BAT_DIS_GATE
- net Net-(Q2-D) renamed /top-level/power_distribution/input_muxing/~{JACK_SHDN}
- net Net-(Q2-G) renamed /top-level/power_distribution/input_muxing/JACK_DIS_GATE
- net Net-(R10-Pad1) renamed /top-level/power_distribution/input_muxing/VIN_RAW_UNFILT
- net Net-(U13-PC14) renamed /top-level/stm32_controller/OSC32_IN
- net Net-(U13-PC15) renamed /top-level/stm32_controller/OSC32_OUT
- net Net-(U13-PE15) renamed /top-level/stm32_controller/BUZZ_MCU
- net Net-(U3-NRETRY) renamed /top-level/power_distribution/input_muxing/efuse/NRETRY
- net Net-(U3-OVLO) renamed /top-level/power_distribution/input_muxing/efuse/OVLO
- net Net-(U3-RETRY_DLY) renamed /top-level/power_distribution/input_muxing/efuse/RETRY_DLY
- C137 pad 1: /top-level/DAQ/PT2_3WIRE_OUT -> /top-level/DAQ/PT1_3WIRE_OUT
Routing:
- net GND: track 203.1 -> 183.4 mm, vias 913 -> 916
- net /top-level/I2C1_SDA: track 169.3 -> 170.1 mm
- net /top-level/stm32_controller/BUZZ_P: track 6.46 -> 5.70 mm
Other:
- board text added: "RS-485"
- board text removed: "Designed by: Nicholas Alves"
- board text removed: "°C"
