File: LRUs/Pad Control Unit/Electrical/Main Controller Board/KICAD PROJECT/master_gse_pcb_project/lc2.kicad_sch (KiCad schematic)
At the start: 22 parts, among them J22 B5B-XH-A, Q18 SS8550, U31 HX711

Commit message: Committ latest changes
Parts:
- removed C146, C150, C152: 10uF, Capacitor_Tantalum_SMD:CP_EIA-3216-18_Kemet-A, symbol Device:C_Polarized_Small_US
- added C149, C153, C155: 10uF, Capacitor_SMD:C_0805_2012Metric, symbol Device:C_Small_US
- renumbered C147 to C150, C148 to C151, C149 to C152, C151 to C154, C153 to C156, D44 to D43, D45 to D44, J22 to J21, JP12 to JP11, R163 to R160, R164 to R161, R165 to R162, R166 to R163, R167 to R164
Connections:
- net +3V3A: now also C149.1
- net +5V: now also C153.1
- net GND: now also C149.2, C153.2, C155.2
- net LC2_E+: now also C155.1
