File: LRUs/Pad Control Unit/Electrical/Main Controller Board/KICAD PROJECT/master_gse_pcb_project/pt2.kicad_sch (KiCad schematic)
At the start: 29 parts, among them J20 B5B-XH-A, Q16 SS8550, U29 HX711

Commit message: Committ latest changes
Parts:
- removed C129, C134, C136: 10uF, Capacitor_Tantalum_SMD:CP_EIA-3216-18_Kemet-A, symbol Device:C_Polarized_Small_US
- added C132, C137, C139: 10uF, Capacitor_SMD:C_0805_2012Metric, symbol Device:C_Small_US
- renumbered C128 to C131, C130 to C133, C131 to C134, C132 to C135, C133 to C136, C135 to C138, C137 to C140, D40 to D39, D41 to D40, J20 to J19, JP7 to JP6, JP8 to JP7, JP9 to JP8, JP10 to JP9, R151 to R148, R152 to R149, R153 to R150, R154 to R151, R155 to R152, R156 to R153, R157 to R154, TP41 to TP51, TP42 to TP52
Connections:
- net +3V3A: now also C132.1
- net +5V: now also C137.1
- net GND: now also C132.2, C137.2, C139.2
- net PT2_E_PRE+: now also C139.1
