File: LRUs/Pad Control Unit/Electrical/Main Controller Board/KICAD PROJECT/master_gse_pcb_project/tc3.kicad_sch (KiCad schematic)
At the start: 21 parts, among them J17 B4B-XH-A, U24 MAX31856, U25 MAX31856

Commit message: Committ latest changes
Parts:
- removed C94, C95: 10uF, Capacitor_Tantalum_SMD:CP_EIA-3216-18_Kemet-A, symbol Device:C_Polarized_Small_US
- added C97, C98: 10uF, Capacitor_SMD:C_0805_2012Metric, symbol Device:C_Small_US
- renumbered C97 to C100, C98 to C101, C99 to C102, C100 to C103, C101 to C104, C102 to C105, C103 to C106, C104 to C107, C105 to C108, C96 to C99, D34 to D33, D35 to D34, J17 to J16, R136 to R133, R137 to R134, R138 to R135, R139 to R136
Connections:
- net +3V3A: now also C97.1, C98.1
- net GND: now also C97.2, C98.2
