File: LRUs/Pad Control Unit/Electrical/Main Controller Board/KICAD PROJECT/master_gse_pcb_project/12V_main.kicad_sch (KiCad schematic)
At the start: 25 parts, among them U4 TPS62933P

Commit message: Committ latest changes
Parts:
- added J5: Conn_01x02_Pin, Connector_PinHeader_2.54mm:PinHeader_1x02_P2.54mm_Vertical, symbol Connector:Conn_01x02_Pin
- renumbered D9 to D7
Connections:
- net 12V_EN: now also J5.1 (Pin_1)
- net GND: now also J5.2 (Pin_2)
Other:
- note added: "12V Inhibit"

Commit message: Committttt
Parts:
- C12, C13, C17, C18: Footprint_Size (none) -> 7343
- C14, C16: Footprint_Size (none) -> 0402
- D7, R26, R27, R28, R29, R30, R31, R32, R33, R34, R35: Footprint_Size (none) -> 0603
- J5: value Conn_01x02_Pin -> 01x02_PinHeader
- L1: Footprint_Size (none) -> XAL6060
