File: LRUs/Pad Control Unit/Electrical/Main Controller Board/KICAD PROJECT/master_gse_pcb_project/3V3_digital.kicad_sch (KiCad schematic)
At the start: 29 parts, among them U6 TPS62933P, U7 TPS2116DRL

Commit message: Committ latest changes
Parts:
- removed C26, C27: 10uF, Capacitor_Tantalum_SMD:CP_EIA-3216-18_Kemet-A, symbol Device:C_Polarized_Small_US
- added C26, C27: 10uF, Capacitor_SMD:C_0805_2012Metric, symbol Device:C_Small_US
- added J7: Conn_01x02_Pin, Connector_PinHeader_2.54mm:PinHeader_1x02_P2.54mm_Vertical, symbol Connector:Conn_01x02_Pin
- renumbered D12 to D10, D11 to D9
Connections:
- net 3V3_EN: now also J7.1 (Pin_1)
- net GND: now also C26.2, C27.2, J7.2 (Pin_2)
- net VIN: now also C26.1, C27.1
Other:
- note added: "3.3V Inhibit"

Commit message: Committttt
Parts:
- C26, C27: Footprint_Size (none) -> 0805
- C28, C29, C30: Footprint_Size (none) -> 0402
- C31, C32: Footprint_Size (none) -> 7343
- D10, D9, R46, R47, R48, R49, R50, R51, R52, R53, R54, R55, R56, R57: Footprint_Size (none) -> 0603
- J7: value Conn_01x02_Pin -> 01x02_PinHeader
- L3: Footprint_Size (none) -> XAL6030
Other:
- moved on the sheet: R47, R48
