File: LRUs/Pad Control Unit/Electrical/Main Controller Board/KICAD PROJECT/master_gse_pcb_project/5V_main.kicad_sch (KiCad schematic)
At the start: 25 parts, among them U5 TPS62933P

Commit message: Committ latest changes
Parts:
- added J6: Conn_01x02_Pin, Connector_PinHeader_2.54mm:PinHeader_1x02_P2.54mm_Vertical, symbol Connector:Conn_01x02_Pin
- renumbered D10 to D8
Connections:
- net GND: now also J6.2 (Pin_2)
- net VEN: now also J6.1 (Pin_1)
Other:
- note added: "5V Inhibit"

Commit message: Committttt
Parts:
- C19, C20, C24, C25: Footprint_Size (none) -> 7343
- C21, C22, C23: Footprint_Size (none) -> 0402
- D8, R36, R37, R38, R39, R40, R41, R42, R43, R44, R45: Footprint_Size (none) -> 0603
- J6: value Conn_01x02_Pin -> 01x02_PinHeader
- L2: Footprint_Size (none) -> XAL6060
