File: LRUs/Pad Control Unit/Electrical/Main Controller Board/KICAD PROJECT/master_gse_pcb_project/can_bus.kicad_sch (KiCad schematic)
At the start: 12 parts, among them J10 B3B-XH-A, U21 TJA1051T-3

Commit message: Committ latest changes
Parts:
- renumbered C76 to C85, C77 to C86, C78 to C87, C79 to C88, D25 to D24, J10 to J12, R105 to R115, R106 to R116, R107 to R117, R108 to R118, R109 to R119, U21 to U22

Commit message: Commit da changes
Parts:
- C85, C87, C88, R116, R117, R118, R119: Footprint_Size (none) -> 0402
- C86: Footprint_Size (none) -> 0805
- R115: Footprint_Size (none) -> 0603
