File: LRUs/Pad Control Unit/Electrical/Main Controller Board/KICAD PROJECT/master_gse_pcb_project/daq.kicad_sch (KiCad schematic)
At the start: 0 parts

Commit message: Committ latest changes
Other:
- removed sheet TC3
- added sheet TC2 (tc1.kicad_sch)
- sheet LC1 ports: added LC_DOUT, LC_SCK; removed LC1_DOUT, LC1_SCK
- sheet LC2: file lc2.kicad_sch -> lc1.kicad_sch
- sheet LC2 ports: added LC_DOUT, LC_SCK; removed LC2_DOUT, LC2_SCK
- sheet PT1 ports: added PT_3WIRE_OUT, PT_DOUT, PT_SCK; removed PT1_3WIRE_OUT, PT1_DOUT, PT1_SCK
- sheet PT2: file pt2.kicad_sch -> pt1.kicad_sch
- sheet PT2 ports: added PT_3WIRE_OUT, PT_DOUT, PT_SCK; removed PT2_3WIRE_OUT, PT2_DOUT, PT2_SCK
- sheet TC1 ports: added ~{TA_CS}, ~{TB_CS}, ~{TCA_DRDY}, ~{TCA_FAULT}, ~{TCB_DRDY}, ~{TCB_FAULT}; removed ~{T3_CS}, ~{T4_CS}, ~{TC3_DRDY}, ~{TC3_FAULT}, ~{TC4_DRDY}, ~{TC4_FAULT}
