File: LRUs/Pad Control Unit/Electrical/Main Controller Board/KICAD PROJECT/master_gse_pcb_project/efuse.kicad_sch (KiCad schematic)
At the start: 19 parts, among them J4 B2B-XH-A, U3 TPS259830ONRGER

Commit message: Committ latest changes
Other:
- moved on the sheet: C11
Changed lines of the file:
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@@
 	)
 	(junction
-		(at 220.98 97.79)
-		(diameter 0)
-		(color 0 0 0 0)
-	)
-	(junction
 		(at 185.42 90.17)
 		(diameter 0)
@@
 		(color 0 0 0 0)
 	)
+	(junction
+		(at 220.98 97.79)
+		(diameter 0)
+		(color 0 0 0 0)
+	)
 	(wire
 		(pts
@@
 	(wire
 		(pts
-			(xy 220.98 105.41) (xy 220.98 107.95)
+			(xy 220.98 104.14) (xy 220.98 105.41)
 		)
 		(stroke
@@
 	(wire
 		(pts
-			(xy 220.98 100.33) (xy 220.98 97.79)
+			(xy 220.98 99.06) (xy 220.98 97.79)
 		)
 		(stroke
@@
 	(symbol
 		(lib_id "Device:C_Small_US")
-		(at 220.98 102.87 0)
+		(at 220.98 101.6 0)
 		(unit 1)
 		(body_style 1)
@@
 		(dnp no)
 		(property "Reference" "C11"
-			(at 222.758 100.33 0)
+			(at 222.758 99.06 0)
 			(show_name no)
 			(do_not_autoplace no)
@@
 		)
 		(property "Value" "100nF"
-			(at 223.266 103.124 0)
+			(at 223.266 101.854 0)
 			(show_name no)
 			(do_not_autoplace no)
@@
 		)
 		(property "Footprint" "Capacitor_SMD:C_0402_1005Metric"
-			(at 220.98 102.87 0)
+			(at 220.98 101.6 0)
 			(hide yes)
 			(show_name no)
@@
 		)
 		(property "Datasheet" ""
-			(at 220.98 102.87 0)
+			(at 220.98 101.6 0)
 			(hide yes)
 			(show_name no)
@@
 		)
 		(property "Description" "100nF 50V X7R ±10% 0402 Capacitor"
-			(at 220.98 102.87 0)
+			(at 220.98 101.6 0)
 			(hide yes)
 			(show_name no)
@@
 		)
 		(property "Vmax" "50V"
-			(at 224.536 105.918 0)
+			(at 224.536 104.648 0)
 			(show_name no)
 			(do_not_autoplace no)
@@
 		)
 		(property "JLCPCB Part #" "C307331"
-			(at 220.98 102.87 0)
+			(at 220.98 101.6 0)
 			(hide yes)
 			(show_name no)
@@
 	(symbol
 		(lib_id "power:GND")
-		(at 220.98 107.95 0)
+		(at 220.98 105.41 0)
 		(unit 1)
 		(body_style 1)
@@
 		(fields_autoplaced yes)
 		(property "Reference" "#PWR035"
-			(at 220.98 114.3 0)
+			(at 220.98 111.76 0)
 			(hide yes)
 			(show_name no)
@@
 		)
 		(property "Value" "GND"
-			(at 220.98 113.03 0)
+			(at 220.98 110.49 0)
 			(hide yes)
 			(show_name no)
@@
 		)
 		(property "Footprint" ""
-			(at 220.98 107.95 0)
+			(at 220.98 105.41 0)
 			(hide yes)
 			(show_name no)
@@
 		)
 		(property "Datasheet" ""
-			(at 220.98 107.95 0)
+			(at 220.98 105.41 0)
 			(hide yes)
 			(show_name no)
@@
 		)
 		(property "Description" "Power symbol creates a global label with name \"GND\" , ground"
-			(at 220.98 107.95 0)
+			(at 220.98 105.41 0)
 			(hide yes)
 			(show_name no)

Commit message: Committttt
Parts:
- C10, C5: Footprint_Size (none) -> 0805
- C11, C6, C9: Footprint_Size (none) -> 0402
- C7, C8, R16, R17, R18, R19, R20, R21, R22, R23, R24, R25: Footprint_Size (none) -> 0603
Other:
- moved on the sheet: R23, R25

Commit message: Commit da changes
Parts:
- U3: JLCPCB Part # C20611808 -> (none)
Connections:
- net GND: now also U3.[33-35] (EPAD), U3.[4,5,14,26] (GND); no longer U3.14 (GND__2), U3.26 (GND__3), U3.33 (EPAD), U3.34 (EPAD), U3.35 (EPAD), U3.4 (GND), U3.5 (GND__1)
- net VIN_SAFE: now also U3.[17-24] (OUT); no longer U3.17 (OUT), U3.18 (OUT__1), U3.19 (OUT__2), U3.20 (OUT__3), U3.21 (OUT__4), U3.22 (OUT__5), U3.23 (OUT__6), U3.24 (OUT__7)
- net VIN_UNSAFE: now also U3.[1-3,16,25] (IN), U3.[27-32] (EPAD); no longer U3.1 (IN), U3.16 (IN__3), U3.2 (IN__1), U3.25 (IN__4), U3.27 (EPAD), U3.28 (EPAD), U3.29 (EPAD), U3.3 (IN__2), U3.30 (EPAD), U3.31 (EPAD), U3.32 (EPAD)
- net OVLO: now reaches R18.2, R19.2, U3.12 (OVLO)
- net EN_H: now reaches J4.1 (Pin_1), R16.2
- net EN_UVLO: now reaches J4.2 (Pin_2), R17.2, U3.6 (EN/UVLO)
- net RETRY_DLY: now reaches R20.2, U3.10 (RETRY_DLY)
- net NRETRY: now reaches R21.2, U3.11 (NRETRY)
Other:
- moved on the sheet: C10, C11, C5, C6, C7, C8, C9, J4, R16, R17, R18, R19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
