File: LRUs/Pad Control Unit/Electrical/Main Controller Board/KICAD PROJECT/master_gse_pcb_project/fans.kicad_sch (KiCad schematic)
At the start: 14 parts, among them J23 B2B-XH-A, J24 B2B-XH-A, Q19 AO3400A, Q20 AO3400A

Commit message: Committ latest changes
Parts:
- renumbered C154 to C163, C155 to C164, D46 to D45, D47 to D46, J23 to J25, J24 to J26, R168 to R178, R169 to R179, R170 to R180, R171 to R181, R172 to R182, R173 to R183
Changed lines of the file:
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@@
 		(dnp no)
 		(fields_autoplaced yes)
-		(property "Reference" "#PWR0347"
+		(property "Reference" "#PWR0367"
 			(at 161.29 44.45 0)
 			(hide yes)
@@
 			(project "master_gse_pcb_project"
 				(path "/5dea7f1e-c3ae-4a7c-865b-d3606d04c094/1d88e707-71bf-4514-8853-31370dba3cbd"
-					(reference "#PWR0347")
+					(reference "#PWR0367")
 					(unit 1)
 				)
@@
 		(in_pos_files yes)
 		(dnp no)
-		(property "Reference" "J24"
+		(property "Reference" "J26"
 			(at 186.182 102.87 0)
 			(show_name no)
@@
 			(project "master_gse_pcb_project"
 				(path "/5dea7f1e-c3ae-4a7c-865b-d3606d04c094/1d88e707-71bf-4514-8853-31370dba3cbd"
-					(reference "J24")
+					(reference "J26")
 					(unit 1)
 					(variant
@@
 		(in_pos_files yes)
 		(dnp no)
-		(property "Reference" "D46"
+		(property "Reference" "D45"
 			(at 130.556 75.946 90)
 			(show_name no)
@@
 			(project "master_gse_pcb_project"
 				(path "/5dea7f1e-c3ae-4a7c-865b-d3606d04c094/1d88e707-71bf-4514-8853-31370dba3cbd"
-					(reference "D46")
+					(reference "D45")
 					(unit 1)
 					(variant
@@
 		(in_pos_files yes)
 		(dnp no)
-		(property "Reference" "C154"
+		(property "Reference" "C163"
 			(at 163.068 45.974 0)
 			(show_name no)
@@
 			(project "master_gse_pcb_project"
 				(path "/5dea7f1e-c3ae-4a7c-865b-d3606d04c094/1d88e707-71bf-4514-8853-31370dba3cbd"
-					(reference "C154")
+					(reference "C163")
 					(unit 1)
 					(variant
@@
 		(dnp no)
 		(fields_autoplaced yes)
-		(property "Reference" "#PWR0350"
+		(property "Reference" "#PWR0370"
 			(at 162.56 120.65 0)
 			(hide yes)
@@
 			(project "master_gse_pcb_project"
 				(path "/5dea7f1e-c3ae-4a7c-865b-d3606d04c094/1d88e707-71bf-4514-8853-31370dba3cbd"
-					(reference "#PWR0350")
+					(reference "#PWR0370")
 					(unit 1)
 				)
@@
 		(dnp no)
 		(fields_autoplaced yes)
-		(property "Reference" "#PWR0349"
+		(property "Reference" "#PWR0369"
 			(at 162.56 106.68 0)
 			(hide yes)
@@
 			(project "master_gse_pcb_project"
 				(path "/5dea7f1e-c3ae-4a7c-865b-d3606d04c094/1d88e707-71bf-4514-8853-31370dba3cbd"
-					(reference "#PWR0349")
+					(reference "#PWR0369")
 					(unit 1)
 				)
@@
 		(in_pos_files yes)
 		(dnp no)
-		(property "Reference" "R173"
+		(property "Reference" "R183"
 			(at 162.306 128.27 0)
 			(show_name no)
@@
 			(project "master_gse_pcb_project"
 				(path "/5dea7f1e-c3ae-4a7c-865b-d3606d04c094/1d88e707-71bf-4514-8853-31370dba3cbd"
-					(reference "R173")
+					(reference "R183")
 					(unit 1)
 					(variant
@@
 		(dnp no)
 		(fields_autoplaced yes)
-		(property "Reference" "#PWR0352"
+		(property "Reference" "#PWR0372"
 			(at 172.72 153.67 0)
 			(hide yes)
@@
 			(project "master_gse_pcb_project"
 				(path "/5dea7f1e-c3ae-4a7c-865b-d3606d04c094/1d88e707-71bf-4514-8853-31370dba3cbd"
-					(reference "#PWR0352")
+					(reference "#PWR0372")
 					(unit 1)
 				)
@@
 		(in_pos_files yes)
 		(dnp no)
-		(property "Reference" "D47"
+		(property "Reference" "D46"
 			(at 134.366 138.176 90)
 			(show_name no)
@@
 			(project "master_gse_pcb_project"
 				(path "/5dea7f1e-c3ae-4a7c-865b-d3606d04c094/1d88e707-71bf-4514-8853-31370dba3cbd"
-					(reference "D47")
+					(reference "D46")
 					(unit 1)
 					(variant
@@
 		(dnp no)
 		(fields_autoplaced yes)
-		(property "Reference" "#PWR0346"
+		(property "Reference" "#PWR0366"
 			(at 132.08 153.67 0)
 			(hide yes)
@@
 			(project "master_gse_pcb_project"
 				(path "/5dea7f1e-c3ae-4a7c-865b-d3606d04c094/1d88e707-71bf-4514-8853-31370dba3cbd"
-					(reference "#PWR0346")
+					(reference "#PWR0366")
 					(unit 1)
 				)
@@
 		(dnp no)
 		(fields_autoplaced yes)
-		(property "Reference" "#PWR0351"
+		(property "Reference" "#PWR0371"
 			(at 172.72 91.44 0)
 			(hide yes)
@@
 			(project "master_gse_pcb_project"
 				(path "/5dea7f1e-c3ae-4a7c-865b-d3606d04c094/1d88e707-71bf-4514-8853-31370dba3cbd"
-					(reference "#PWR0351")
+					(reference "#PWR0371")
 					(unit 1)
 				)
@@
 		(in_pos_files yes)
 		(dnp no)
-		(property "Reference" "J23"
+		(property "Reference" "J25"
 			(at 186.182 40.64 0)
 			(show_name no)
@@
 			(project "master_gse_pcb_project"
 				(path "/5dea7f1e-c3ae-4a7c-865b-d3606d04c094/1d88e707-71bf-4514-8853-31370dba3cbd"
-					(reference "J23")
+					(reference "J25")
 					(unit 1)
 					(variant
@@
 		(dnp no)
 		(fields_autoplaced yes)
-		(property "Reference" "#PWR0345"
+		(property "Reference" "#PWR0365"
 			(at 128.27 91.44 0)
 			(hide yes)
@@
 			(project "master_gse_pcb_project"
 				(path "/5dea7f1e-c3ae-4a7c-865b-d3606d04c094/1d88e707-71bf-4514-8853-31370dba3cbd"
-					(reference "#PWR0345")
+					(reference "#PWR0365")
 					(unit 1)
 				)
@@
 		(in_pos_files yes)
 		(dnp no)
-		(property "Reference" "R170"
+		(property "Reference" "R180"
 			(at 147.574 60.706 90)
 			(show_name no)
@@
 			(project "master_gse_pcb_project"
 				(path "/5dea7f1e-c3ae-4a7c-865b-d3606d04c094/1d88e707-71bf-4514-8853-31370dba3cbd"
-					(reference "R170")
+					(reference "R180")
 					(unit 1)
 					(variant
@@
 		(in_pos_files yes)
 		(dnp no)
-		(property "Reference" "R172"
+		(property "Reference" "R182"
 			(at 162.306 66.04 0)
 			(show_name no)
@@
 			(project "master_gse_pcb_project"
 				(path "/5dea7f1e-c3ae-4a7c-865b-d3606d04c094/1d88e707-71bf-4514-8853-31370dba3cbd"
-					(reference "R172")
+					(reference "R182")
 					(unit 1)
 					(variant
@@
 		(in_pos_files yes)
 		(dnp no)
-		(property "Reference" "R171"
+		(property "Reference" "R181"
 			(at 147.574 122.936 90)
 			(show_name no)
@@
 			(project "master_gse_pcb_project"
 				(path "/5dea7f1e-c3ae-4a7c-865b-d3606d04c094/1d88e707-71bf-4514-8853-31370dba3cbd"
-					(reference "R171")
+					(reference "R181")
 					(unit 1)
 					(variant
@@
 		(in_pos_files yes)
 		(dnp no)
-		(property "Reference" "R169"
+		(property "Reference" "R179"
 			(at 135.382 129.54 0)
 			(show_name no)
@@
 			(project "master_gse_pcb_project"
 				(path "/5dea7f1e-c3ae-4a7c-865b-d3606d04c094/1d88e707-71bf-4514-8853-31370dba3cbd"
-					(reference "R169")
+					(reference "R179")
 					(unit 1)
 					(variant
@@
 		(dnp no)
 		(fields_autoplaced yes)
-		(property "Reference" "#PWR0348"
+		(property "Reference" "#PWR0368"
 			(at 161.29 58.42 0)
 			(hide yes)
@@
 			(project "master_gse_pcb_project"
 				(path "/5dea7f1e-c3ae-4a7c-865b-d3606d04c094/1d88e707-71bf-4514-8853-31370dba3cbd"
-					(reference "#PWR0348")
+					(reference "#PWR0368")
 					(unit 1)
 				)
@@
 		(in_pos_files yes)
 		(dnp no)
-		(property "Reference" "R168"
+		(property "Reference" "R178"
 			(at 131.572 67.31 0)
 			(show_name no)
@@
 			(project "master_gse_pcb_project"
 				(path "/5dea7f1e-c3ae-4a7c-865b-d3606d04c094/1d88e707-71bf-4514-8853-31370dba3cbd"
-					(reference "R168")
+					(reference "R178")
 					(unit 1)
 					(variant
@@
 		(in_pos_files yes)
 		(dnp no)
-		(property "Reference" "C155"
+		(property "Reference" "C164"
 			(at 164.338 108.204 0)
 			(show_name no)
@@
 			(project "master_gse_pcb_project"
 				(path "/5dea7f1e-c3ae-4a7c-865b-d3606d04c094/1d88e707-71bf-4514-8853-31370dba3cbd"
-					(reference "C155")
+					(reference "C164")
 					(unit 1)
 					(variant

Commit message: Commit da changes
Parts:
- C163, C164: Footprint_Size (none) -> 1206
- D45, D46, R178, R179, R180, R181, R182, R183: Footprint_Size (none) -> 0603
- Q19, Q20: Footprint_Size (none) -> SOT-23
