File: LRUs/Pad Control Unit/Electrical/Main Controller Board/KICAD PROJECT/master_gse_pcb_project/igniter_system.kicad_sch (KiCad schematic)
At the start: 69 parts, among them J13 Conn_01x02_Pin, J14 B4B-XH-A, J15 1x2 Screw Terminal, J16 1x2 Screw Terminal, K1 J107F1CS205VDC.45, Q11 AO3400A, Q12 STD52P3LLH6, Q13 AO3400A, Q14 AO3400A, U23 TPS259830ONRGER

Commit message: Committ latest changes
Parts:
- removed C92: 10uF, Capacitor_Tantalum_SMD:CP_EIA-3216-18_Kemet-A, symbol Device:C_Polarized_Small_US
- removed R116, R124: 2.2k, Resistor_SMD:R_0603_1608Metric, symbol Device:R_Small_US
- added C101: 10uF, Capacitor_SMD:C_0805_2012Metric, symbol Device:C_Small_US
- added R? (x2): 2.2k, Resistor_SMD:R_0603_1608Metric, symbol Device:R_Small_US
- R129: renamed from R119; Footprint_Size (none) -> 0603
- R132: renamed from R122; size (none) -> 0603
- renumbered C91 to C100, C93 to C102, C83 to C92, C84 to C93, C85 to C94, C86 to C95, C87 to C96, C88 to C97, C89 to C98, C90 to C99, D26 to D25, D27 to D26, D28 to D27, D29 to D28, D30 to D29, D31 to D30, D32 to D31, D33 to D32, J13 to J15, J14 to J16, J15 to J17, J16 to J18, R110 to R120, R111 to R121, R112 to R122, R113 to R123, R114 to R124, R115 to R125, R117 to R127, R118 to R128, R120 to R130, R121 to R131, R123 to R133, R125 to R135, R126 to R136, R127 to R137, R128 to R138, R129 to R139, R130 to R140, R131 to R141, R132 to R142, R133 to R143, R134 to R144, R135 to R145, TP26 to TP35, TP27 to TP36, TP28 to TP37, TP29 to TP38, TP30 to TP39, TP31 to TP40, TP32 to TP41, TP33 to TP42, TP34 to TP43, TP35 to TP44, TP36 to TP45, TP37 to TP46, TP38 to TP47, U23 to U24
Connections:
- net +3V3: now also R?.1
- net +5V: now also C101.1
- net GND: now also C101.2
- net IGNITER_FIRE: now also R?.1
- net at D30.2 (A), Q11.3 (D): now also R?.2
- net at D26.2 (A): now also R?.2

Commit message: Commit valve board updates
Parts:
- gave numbers to parts that had none: 2

Commit message: Commit da changes
Parts:
- C100, C102, C94: Footprint_Size (none) -> 0402
- C101, C93, C99: Footprint_Size (none) -> 0805
- C92: Footprint_Size (none) -> 6.3x5.4
- C95, C96, D25, D26, D27, D28, D30, R120, R121, R122, R123, R124, R127, R130, R131, R133, R135, R136, R137, R138, R139, R140, R141, R142, R143, R144, R145: Footprint_Size (none) -> 0603
- C97, C98: Footprint_Size (none) -> 8x10.5
- D29, D31: Footprint_Size (none) -> SOD-123
- D32: Footprint_Size (none) -> SMB
- F1: value Fuse -> 0297020; Footprint_Size (none) -> Plugin; IMAX 20A -> (none); JLCPCB Part # F1 -> C5249699; Rating (none) -> 32V/20A; VDS Fuse -> (none)
- J15: value Conn_01x02_Pin -> XT-60
- Q11, Q13, Q14: Footprint_Size (none) -> SOT-23
- Q12: Footprint_Size (none) -> TO-252-2
- U24: JLCPCB Part # C20611808 -> (none)
Connections:
- net GND: now also U24.[33-35] (EPAD), U24.[4,5,14,26] (GND); no longer U24.14 (GND__2), U24.26 (GND__3), U24.33 (EPAD), U24.34 (EPAD), U24.35 (EPAD), U24.4 (GND), U24.5 (GND__1)
- net IGNITER+: now also U24.[17-24] (OUT); no longer U24.17 (OUT), U24.18 (OUT__1), U24.19 (OUT__2), U24.20 (OUT__3), U24.21 (OUT__4), U24.22 (OUT__5), U24.23 (OUT__6), U24.24 (OUT__7)
- net VIN_EFUSE: now also U24.[1-3,16,25] (IN), U24.[27-32] (EPAD); no longer U24.1 (IN), U24.16 (IN__3), U24.2 (IN__1), U24.25 (IN__4), U24.27 (EPAD), U24.28 (EPAD), U24.29 (EPAD), U24.3 (IN__2), U24.30 (EPAD), U24.31 (EPAD), U24.32 (EPAD)
Other:
- moved on the sheet: C95, C96, D29, R120, R121, R122, R123, R130, R131, R132, R133, R135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
