File: LRUs/Pad Control Unit/Electrical/Main Controller Board/KICAD PROJECT/master_gse_pcb_project/input_muxing.kicad_sch (KiCad schematic)
At the start: 34 parts, among them Q1 AO3400A, Q2 AO3400A, Q3 SiR882ADP, Q4 SiR882ADP, Q5 SiR882ADP, Q6 SiR882ADP, U1 LTC4359-MS8, U2 LTC4359-MS8

Commit message: Committ latest changes
Parts:
- removed D1, D3: SMAT70A-13-F, Diode_SMD:D_SMA, symbol Device:D_Zener
- renumbered D2 to D1, D4 to D2, D5 to D3, D6 to D4, D7 to D5, D8 to D6
Connections:
- net VIN_BAT: now also D2.2 (A)
- net VIN_DC_JACK: now also D1.2 (A)
Other:
- moved on the sheet: D1, D2

Commit message: Committttt
Parts:
- C1, C2: Footprint_Size (none) -> 1206
- C3, C4: Footprint_Size (none) -> 0402
- D1, D2: Footprint_Size (none) -> DO214AC
- D3, D4: Footprint_Size (none) -> DO-214AC
- D5, D6: Footprint_Size (none) -> SOD-123
- Q1, Q2: Footprint_Size (none) -> SOT-23; VDS (none) -> 30V
- Q3, Q4, Q5, Q6: Footprint_Size (none) -> SO-8
- R10, R11, R12, R13, R14, R15, R2, R3, R4, R5, R6, R7, R8, R9: Footprint_Size (none) -> 0603
Other:
- moved on the sheet: R15

Commit message: Commit da changes
Connections:
- net JACK_DIS_GATE: now reaches Q2.1 (G), R4.1, R5.2
- net ~{JACK_SHDN}: now reaches Q2.3 (D), R7.1, U2.5 (~{SHDN})
- net BAT_SRC: now reaches D5.2 (A), Q3.1 (S), Q3.2 (S), Q3.3 (S), Q5.1 (S), Q5.2 (S), Q5.3 (S), U1.2 (SRC)
- net BAT_GATE: now reaches D5.1 (K), Q3.4 (G), Q5.4 (G), U1.1 (GATE)
- net JACK_SRC: now reaches D6.2 (A), Q4.1 (S), Q4.2 (S), Q4.3 (S), Q6.1 (S), Q6.2 (S), Q6.3 (S), U2.2 (SRC)
- net JACK_GATE: now reaches D6.1 (K), Q4.4 (G), Q6.4 (G), U2.1 (GATE)
- net VIN_RAW_UNFILT: now reaches R10.1, R11.2, R12.2
- net BAT_DIS_GATE: now reaches Q1.1 (G), R2.1, R3.2
- net ~{BAT_SHDN}: now reaches Q1.3 (D), R6.1, U1.5 (~{SHDN})
- net efuse/VIN_UNSAFE renamed VIN_UNSAFE
Other:
- moved on the sheet: C3, D1, D2, Q1, Q2, R12, R2, R3, R4, R5, R6, R7
