File: LRUs/Pad Control Unit/Electrical/Main Controller Board/KICAD PROJECT/master_gse_pcb_project/lc1.kicad_sch (KiCad schematic)
At the start: 22 parts, among them J21 B5B-XH-A, Q17 SS8550, U30 HX711

Commit message: Committ latest changes
Parts:
- removed C138, C142, C144: 10uF, Capacitor_Tantalum_SMD:CP_EIA-3216-18_Kemet-A, symbol Device:C_Polarized_Small_US
- added C147, C151, C153: 10uF, Capacitor_SMD:C_0805_2012Metric, symbol Device:C_Small_US
- renumbered C139 to C148, C140 to C149, C141 to C150, C143 to C152, C145 to C154, D42 to D41, D43 to D42, J21 to J23, JP11 to JP10, R158 to R168, R159 to R169, R160 to R170, R161 to R171, R162 to R172, TP43 to TP52, TP44 to TP53, U30 to U31
Connections:
- net +3V3A: now also C147.1
- net +5V: now also C151.1
- net GND: now also C147.2, C151.2, C153.2
- net LC1_E+: now also C153.1
- net LC1_DOUT renamed LC_DOUT
- net LC1_SCK renamed LC_SCK

Commit message: Commit da changes
Parts:
- C147, C151, C153: Footprint_Size (none) -> 0805
- C148, C149, C150, C152, C154: Footprint_Size (none) -> 0402
- L6, R168, R169, R170, R171, R172: Footprint_Size (none) -> 0603
- Q17: Footprint_Size (none) -> SOT-23; Vce (none) -> 25V
