File: LRUs/Pad Control Unit/Electrical/Main Controller Board/KICAD PROJECT/master_gse_pcb_project/master_gse_pcb_project.kicad_sch (KiCad schematic)
At the start: 0 parts

Commit message: Committ latest changes
Other:
- sheet RS_485 ports: added none; removed {RS485_AUX}
- sheet pcb_sensors ports: added ADC_RDY, SENS_SCL, SENS_SDA; removed TEMP_SCL, TEMP_SDA
- sheet stm32_controller ports: added ADC_RDY; removed {RS485_AUX}
Changed lines of the file:
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@@
 	(bus
 		(pts
-			(xy 166.37 111.76) (xy 205.74 111.76)
+			(xy 166.37 118.11) (xy 205.74 118.11)
 		)
 		(stroke
@@
 	(bus
 		(pts
-			(xy 80.01 59.69) (xy 119.38 59.69)
+			(xy 80.01 63.5) (xy 119.38 63.5)
 		)
 		(stroke
@@
 	(wire
 		(pts
-			(xy 80.01 104.14) (xy 119.38 104.14)
+			(xy 80.01 95.25) (xy 119.38 95.25)
 		)
 		(stroke
@@
 	(wire
 		(pts
-			(xy 80.01 101.6) (xy 119.38 101.6)
+			(xy 80.01 92.71) (xy 119.38 92.71)
 		)
 		(stroke
@@
 	(wire
 		(pts
-			(xy 80.01 88.9) (xy 119.38 88.9)
+			(xy 80.01 78.74) (xy 119.38 78.74)
 		)
 		(stroke
@@
 	(wire
 		(pts
-			(xy 80.01 106.68) (xy 119.38 106.68)
+			(xy 80.01 97.79) (xy 119.38 97.79)
 		)
 		(stroke
@@
 	(wire
 		(pts
-			(xy 80.01 91.44) (xy 119.38 91.44)
+			(xy 80.01 81.28) (xy 119.38 81.28)
 		)
 		(stroke
@@
 	(wire
 		(pts
-			(xy 80.01 109.22) (xy 119.38 109.22)
+			(xy 80.01 100.33) (xy 119.38 100.33)
 		)
 		(stroke
@@
 		)
 	)
-	(bus
+	(wire
 		(pts
-			(xy 80.01 62.23) (xy 119.38 62.23)
+			(xy 80.01 102.87) (xy 119.38 102.87)
 		)
 		(stroke
@@
 	(bus
 		(pts
-			(xy 166.37 91.44) (xy 205.74 91.44)
+			(xy 166.37 96.52) (xy 205.74 96.52)
 		)
 		(stroke
@@
 	(wire
 		(pts
-			(xy 80.01 86.36) (xy 119.38 86.36)
+			(xy 80.01 76.2) (xy 119.38 76.2)
 		)
 		(stroke
@@
 	)
 	(label "I2C1_SDA"
-		(at 93.98 101.6 0)
+		(at 93.98 92.71 0)
 		(effects
 			(font
@@
 	)
 	(label "I2C1_SCL"
-		(at 93.98 104.14 0)
+		(at 93.98 95.25 0)
 		(effects
 			(font
@@
 	)
 	(sheet
-		(at 205.74 89.408)
-		(size 29.21 14.732)
+		(at 205.74 92.71)
+		(size 29.21 7.62)
 		(exclude_from_sim no)
 		(in_bom yes)
@@
 		)
 		(property "Sheetname" "SD_card"
-			(at 205.74 88.6964 0)
+			(at 205.74 91.9984 0)
 			(show_name no)
 			(do_not_autoplace no)
@@
 		)
 		(property "Sheetfile" "sd_card.kicad_sch"
-			(at 205.74 104.7246 0)
+			(at 205.74 100.9146 0)
 			(show_name no)
 			(do_not_autoplace no)
@@
 		)
 		(pin "{SD_CARD}" bidirectional
-			(at 205.74 91.44 180)
+			(at 205.74 96.52 180)
 			(effects
 				(font
@@
 		)
 		(pin "CAN1_RX" bidirectional
-			(at 119.38 88.9 180)
+			(at 119.38 78.74 180)
 			(effects
 				(font
@@
 		)
 		(pin "CAN1_TX" bidirectional
-			(at 119.38 86.36 180)
+			(at 119.38 76.2 180)
 			(effects
 				(font
@@
 		)
 		(pin "I2C1_SCL" output
-			(at 119.38 104.14 180)
+			(at 119.38 95.25 180)
 			(effects
 				(font
@@
 		)
 		(pin "I2C1_SDA" bidirectional
-			(at 119.38 101.6 180)
+			(at 119.38 92.71 180)
 			(effects
 				(font
@@
 		)
 		(pin "CAN_SILENT" output
-			(at 119.38 91.44 180)
+			(at 119.38 81.28 180)
 			(effects
 				(font
@@
 		)
 		(pin "TEMP1_ALERT" output
-			(at 119.38 106.68 180)
+			(at 119.38 97.79 180)
 			(effects
 				(font
@@
 		)
 		(pin "TEMP2_ALERT" output
-			(at 119.38 109.22 180)
+			(at 119.38 100.33 180)
 			(effects
 				(font
@@
 		)
 		(pin "{SD_CARD}" bidirectional
-			(at 166.37 91.44 0)
+			(at 166.37 96.52 0)
 			(effects
 				(font
@@
 		)
 		(pin "{RS485_MAIN}" bidirectional
-			(at 119.38 59.69 180)
+			(at 119.38 63.5 180)
 			(effects
 				(font
@@
 			)
 		)
-		(pin "{RS485_AUX}" bidirectional
-			(at 119.38 62.23 180)
+		(pin "{RADIO}" bidirectional
+			(at 166.37 118.11 0)
 			(effects
 				(font
 					(size 1.27 1.27)
 				)
-				(justify left)
+				(justify right)
 			)
 		)
-		(pin "{RADIO}" bidirectional
-			(at 166.37 111.76 0)
+		(pin "ADC_RDY" input
+			(at 119.38 102.87 180)
 			(effects
 				(font
 					(size 1.27 1.27)
 				)
-				(justify right)
+				(justify left)
 			)
 		)
@@
 	)
 	(sheet
-		(at 49.784 83.82)
+		(at 49.784 73.66)
 		(size 30.226 10.16)
 		(exclude_from_sim no)
@@
 		)
 		(property "Sheetname" "can_bus"
-			(at 49.784 83.1084 0)
+			(at 49.784 72.9484 0)
 			(show_name no)
 			(do_not_autoplace no)
@@
 		)
 		(property "Sheetfile" "can_bus.kicad_sch"
-			(at 49.784 94.5646 0)
+			(at 49.784 84.4046 0)
 			(show_name no)
 			(do_not_autoplace no)
@@
 		)
 		(pin "SILENT" input
-			(at 80.01 91.44 0)
+			(at 80.01 81.28 0)
 			(effects
 				(font
@@
 		)
 		(pin "RX" output
-			(at 80.01 88.9 0)
+			(at 80.01 78.74 0)
 			(effects
 				(font
@@
 		)
 		(pin "TX" input
-			(at 80.01 86.36 0)
+			(at 80.01 76.2 0)
 			(effects
 				(font
@@
 	)
 	(sheet
-		(at 205.74 109.22)
-		(size 29.21 17.399)
+		(at 205.74 111.76)
+		(size 29.21 12.7)
 		(exclude_from_sim no)
 		(in_bom yes)
@@
 		)
 		(property "Sheetname" "rf"
-			(at 205.74 108.5084 0)
+			(at 205.74 111.0484 0)
 			(show_name no)
 			(do_not_autoplace no)
@@
 		)
 		(property "Sheetfile" "rf.kicad_sch"
-			(at 205.74 127.2036 0)
+			(at 205.74 125.0446 0)
 			(show_name no)
 			(do_not_autoplace no)
@@
 		)
 		(property "Field2" ""
-			(at 205.74 109.22 0)
+			(at 205.74 111.76 0)
 			(show_name no)
 			(do_not_autoplace no)
@@
 		)
 		(pin "{RADIO}" bidirectional
-			(at 205.74 111.76 180)
+			(at 205.74 118.11 180)
 			(effects
 				(font
@@
 	)
 	(sheet
-		(at 49.53 99.06)
-		(size 30.48 12.7)
+		(at 49.53 90.17)
+		(size 30.48 15.24)
 		(exclude_from_sim no)
 		(in_bom yes)
@@
 		)
 		(property "Sheetname" "pcb_sensors"
-			(at 49.53 98.3484 0)
+			(at 49.53 89.4584 0)
 			(show_name no)
 			(do_not_autoplace no)
@@
 		)
 		(property "Sheetfile" "pcb_sensors.kicad_sch"
-			(at 49.53 112.3446 0)
+			(at 49.53 105.9946 0)
 			(show_name no)
 			(do_not_autoplace no)
@@
 		)
 		(pin "TEMP1_ALERT" output
-			(at 80.01 106.68 0)
+			(at 80.01 97.79 0)
 			(effects
 				(font
@@
 		)
 		(pin "TEMP2_ALERT" output
-			(at 80.01 109.22 0)
+			(at 80.01 100.33 0)
+			(effects
+				(font
+					(size 1.27 1.27)
+				)
+				(justify right)
+			)
+		)
+		(pin "ADC_RDY" output
+			(at 80.01 102.87 0)
 			(effects
 				(font
@@
 			)
 		)
-		(pin "TEMP_SDA" bidirectional
-			(at 80.01 101.6 0)
+		(pin "SENS_SCL" input
+			(at 80.01 95.25 0)
 			(effects
 				(font
@@
 			)
 		)
-		(pin "TEMP_SCL" input
-			(at 80.01 104.14 0)
+		(pin "SENS_SDA" bidirectional
+			(at 80.01 92.71 0)
 			(effects
 				(font
@@
 	(sheet
 		(at 49.53 57.658)
-		(size 30.48 21.336)
+		(size 30.48 10.922)
 		(exclude_from_sim no)
 		(in_bom yes)
@@
 		)
 		(property "Sheetfile" "RS_485.kicad_sch"
-			(at 49.53 79.5786 0)
+			(at 49.53 69.1646 0)
 			(show_name no)
 			(do_not_autoplace no)
@@
 			)
 		)
-		(pin "{RS485_AUX}" bidirectional
-			(at 80.01 62.23 0)
-			(effects
-				(font
-					(size 1.27 1.27)
-				)
-				(justify right)
-			)
-		)
 		(pin "{RS485_MAIN}" bidirectional
-			(at 80.01 59.69 0)
+			(at 80.01 63.5 0)
 			(effects
 				(font
