File: LRUs/Pad Control Unit/Electrical/Main Controller Board/KICAD PROJECT/master_gse_pcb_project/misc.kicad_sch (KiCad schematic)
At the start: 25 parts, among them J25 61202021721, J26 61200621721, J27 09242206824, U32 TPD6E05U06RVZ, U33 TPD6E05U06RVZ

Commit message: Committ latest changes
Parts:
- removed C157, C158: 10uF, Capacitor_Tantalum_SMD:CP_EIA-3216-18_Kemet-A, symbol Device:C_Polarized_Small_US
- added C166, C167: 10uF, Capacitor_SMD:C_0805_2012Metric, symbol Device:C_Small_US
- J29: renamed from J27; footprint Connector_DIN:DIN41612_B3_2x10_Female_Vertical_THT -> Connector_PinSocket_2.54mm:PinSocket_2x10_P2.54mm_Vertical; symbol Connector_Generic:Conn_02x10_Row_Letter_First -> Connector_Generic:Conn_02x10_Odd_Even
- renumbered C156 to C165, C159 to C168, J25 to J27, J26 to J28, R174 to R184, R175 to R185, R176 to R186, R177 to R187, R178 to R188, R179 to R189, R180 to R190, R181 to R191, R182 to R192, R183 to R193, U32 to U33, U33 to U34
Connections:
- net +3V3: now also C166.1, C167.1
- net +3V3_INTF: now also J29.4 (Pin_4), J29.8 (Pin_8); no longer J29.a2 (Pin_a2), J29.a4 (Pin_a4)
- net +5V_INTF: now also J29.1 (Pin_1), J29.5 (Pin_5); no longer J29.b1 (Pin_b1), J29.b3 (Pin_b3)
- net GND: now also J29.10 (Pin_10), J29.11 (Pin_11), J29.14 (Pin_14), J29.15 (Pin_15), J29.18 (Pin_18), J29.19 (Pin_19), J29.2 (Pin_2), J29.3 (Pin_3), J29.6 (Pin_6), J29.7 (Pin_7), C166.2, C167.2; no longer J29.a1 (Pin_a1), J29.a3 (Pin_a3), J29.a5 (Pin_a5), J29.a7 (Pin_a7), J29.a9 (Pin_a9), J29.b10 (Pin_b10), J29.b2 (Pin_b2), J29.b4 (Pin_b4), J29.b6 (Pin_b6), J29.b8 (Pin_b8)
- net I2C1_SCL: now also J29.20 (Pin_20); no longer J29.a10 (Pin_a10)
- net I2C1_SDA: now also J29.17 (Pin_17); no longer J29.b9 (Pin_b9)
- net INTF_1: now also J29.9 (Pin_9); no longer J29.b5 (Pin_b5)
- net INTF_2: now also J29.12 (Pin_12); no longer J29.a6 (Pin_a6)
- net INTF_3: now also J29.13 (Pin_13); no longer J29.b7 (Pin_b7)
- net INTF_4: now also J29.16 (Pin_16); no longer J29.a8 (Pin_a8)

Commit message: Commit da changes
Parts:
- added FID1, FID2, FID3: Fiducial, Fiducial:Fiducial_1mm_Mask3mm, symbol Mechanical:Fiducial
- added H8: M3 Mount, MountingHole:MountingHole_3.2mm_M3_DIN965_Pad, symbol Mechanical:MountingHole_Pad
- C165, C168: Footprint_Size (none) -> 0402
- C166, C167: Footprint_Size (none) -> 0805
- R184, R185, R186, R187, R188, R189, R190, R191, R192, R193: Footprint_Size (none) -> 0603
- U33, U34: Footprint_Size (none) -> USON-14; VR (none) -> 5.5V
Connections:
- net GND: now also H8.1
Other:
- moved on the sheet: H2, H3, H4, H5, H6, H7, J29, U33
