File: LRUs/Pad Control Unit/Electrical/Main Controller Board/KICAD PROJECT/master_gse_pcb_project/power_distribution.kicad_sch (KiCad schematic)
At the start: 6 parts, among them J1 Conn_01x02_Pin, J2 RAPC722X, J3 Conn_01x02_Pin

Commit message: Commit valve board updates
Parts:
- FB1, FB2: Footprint_Size (none) -> 0603; Imp (none) -> 120Ω@100MHz
- J1: value Conn_01x02_Pin -> XT-60
- J3: value Conn_01x02_Pin -> 01x02_PinHeader; Footprint_Size (none) -> 2.54mm
- R1: Footprint_Size (none) -> 0603
Other:
- moved on the sheet: R1

Commit message: Commit da changes
Changed lines of the file:
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@@
 	(title_block
 		(title "Power Distribution")
-		(date "2026-08-27")
+		(date "2026-08-30")
 		(rev "A")
 	)
@@
 	(text "Place near PTs"
 		(exclude_from_sim no)
-		(at 210.566 43.688 0)
+		(at 210.566 41.656 0)
 		(effects
 			(font
@@
 		(dnp no)
 		(property "Reference" "FB1"
-			(at 204.978 45.466 90)
+			(at 208.788 43.942 90)
 			(show_name no)
 			(do_not_autoplace no)
@@
 		(property "Value" "120R"
 			(at 212.598 45.466 90)
+			(hide yes)
 			(show_name no)
 			(do_not_autoplace no)
@@
 		(dnp no)
 		(property "Reference" "FB2"
-			(at 222.758 82.296 90)
+			(at 226.568 80.772 90)
 			(show_name no)
 			(do_not_autoplace no)
@@
 		(property "Value" "120R"
 			(at 230.378 82.296 90)
-			(show_name no)
-			(do_not_autoplace no)
+			(hide yes)
+			(show_name no)
+			(do_not_autoplace no)
