File: LRUs/Pad Control Unit/Electrical/Main Controller Board/KICAD PROJECT/master_gse_pcb_project/pt1.kicad_sch (KiCad schematic)
At the start: 29 parts, among them J19 B5B-XH-A, Q15 SS8550, U28 HX711

Commit message: Committ latest changes
Parts:
- removed C119, C124, C126: 10uF, Capacitor_Tantalum_SMD:CP_EIA-3216-18_Kemet-A, symbol Device:C_Polarized_Small_US
- added C128, C133, C135: 10uF, Capacitor_SMD:C_0805_2012Metric, symbol Device:C_Small_US
- renumbered C118 to C127, C120 to C129, C121 to C130, C122 to C131, C123 to C132, C125 to C134, C127 to C136, D38 to D37, D39 to D38, J19 to J21, JP3 to JP2, JP4 to JP3, JP5 to JP4, JP6 to JP5, R144 to R154, R145 to R155, R146 to R156, R147 to R157, R148 to R158, R149 to R159, R150 to R160, TP39 to TP48, TP40 to TP49, U28 to U29
Connections:
- net +3V3A: now also C128.1
- net +5V: now also C133.1
- net GND: now also C128.2, C133.2, C135.2
- net PT1_E_PRE+: now also C135.1
- net PT1_3WIRE_OUT renamed PT_3WIRE_OUT
- net PT1_DOUT renamed PT_DOUT
- net PT1_SCK renamed PT_SCK

Commit message: Commit da changes
Parts:
- removed C127: 100nF, Capacitor_SMD:C_0402_1005Metric, symbol Device:C_Small_US
- added C137: 100nF, Capacitor_SMD:C_0402_1005Metric, symbol Device:C_Small_US
- C128, C133, C135: Footprint_Size (none) -> 0805
- C129, C131, C132, C134, C136: Footprint_Size (none) -> 0402
- C130: Footprint_Size (none) -> 7343
- L4, R154, R155, R156, R157, R158, R159, R160: Footprint_Size (none) -> 0603
- Q15: Footprint_Size (none) -> SOT-23; Vce (none) -> 25V
Connections:
- net GND: now also C137.2
- net PT_3WIRE_OUT: now also C137.1
Other:
- moved on the sheet: L4
