File: LRUs/Pad Control Unit/Electrical/Main Controller Board/KICAD PROJECT/master_gse_pcb_project/rf.kicad_sch (KiCad schematic)
At the start: 7 parts, among them J11 Conn_02x04_Odd_Even, J12 Conn_Coaxial, U22 RFM69HW

Commit message: Committ latest changes
Parts:
- removed C80: 10uF, Capacitor_Tantalum_SMD:CP_EIA-3216-18_Kemet-A, symbol Device:C_Polarized_Small_US
- added C89: 10uF, Capacitor_SMD:C_0805_2012Metric, symbol Device:C_Small_US
- H1: now not fitted
- renumbered C81 to C90, C82 to C91, J11 to J13, J12 to J14, U22 to U23
Connections:
- net +3V3_RADIO: now also C89.1
- net GND: now also C89.2
Other:
- note removed: "Placeholder shield mount"

Commit message: Commit da changes
Parts:
- C89, C90: Footprint_Size (none) -> 0805
- C91: Footprint_Size (none) -> 0402
- J13: value Conn_02x04_Odd_Even -> 02x04_PinHeader; Footprint_Size (none) -> 2.54mm
- J14: value Conn_Coaxial -> SMA; Impedance (none) -> 50Ω
Connections:
- net ANT: now reaches J14.1 (In), U23.10 (ANA)
Changed lines of the file:
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@@
 	(title_block
 		(title "LoRa Radio")
-		(date "2026-08-27")
+		(date "2026-08-30")
 		(rev "A")
 	)
@@
 	(label "RF_INT"
 		(at 60.96 99.06 180)
+		(effects
+			(font
+				(size 1.27 1.27)
+			)
+			(justify right bottom)
+		)
+	)
+	(label "ANT"
+		(at 172.72 83.82 180)
 		(effects
 			(font
@@
 		(in_pos_files yes)
 		(dnp no)
-		(fields_autoplaced yes)
 		(property "Reference" "U23"
-			(at 150.7333 76.2 0)
+			(at 137.922 80.01 0)
 			(show_name no)
 			(do_not_autoplace no)
@@
 		)
 		(property "Value" "RFM69HW"
-			(at 150.7333 78.74 0)
+			(at 138.176 103.124 0)
 			(show_name no)
 			(do_not_autoplace no)
@@
 		(dnp no)
 		(property "Reference" "C91"
-			(at 138.684 61.214 0)
+			(at 139.446 61.214 0)
 			(show_name no)
 			(do_not_autoplace no)
@@
 		)
 		(property "Value" "100nF"
-			(at 139.446 63.754 0)
+			(at 139.446 62.992 0)
 			(show_name no)
 			(do_not_autoplace no)
@@
 		)
 		(property "Vmax" "50V"
-			(at 140.716 66.04 0)
+			(at 141.224 64.77 0)
 			(show_name no)
 			(do_not_autoplace no)
@@
 			(at 137.16 63.5 0)
 			(hide yes)
+			(show_name no)
+			(do_not_autoplace no)
+			(effects
+				(font
+					(size 1.27 1.27)
+				)
+			)
+		)
+		(property "Footprint_Size" "0402"
+			(at 141.732 66.548 0)
 			(show_name no)
 			(do_not_autoplace no)
@@
 		(in_pos_files yes)
 		(dnp no)
-		(fields_autoplaced yes)
 		(property "Reference" "J14"
-			(at 201.93 82.8431 0)
+			(at 201.168 82.042 0)
 			(show_name no)
 			(do_not_autoplace no)
@@
 			)
 		)
-		(property "Value" "Conn_Coaxial"
-			(at 201.93 85.3831 0)
+		(property "Value" "SMA"
+			(at 201.168 83.8591 0)
 			(show_name no)
 			(do_not_autoplace no)
@@
 			(at 198.12 83.82 0)
 			(hide yes)
+			(show_name no)
+			(do_not_autoplace no)
+			(effects
+				(font
+					(size 1.27 1.27)
+				)
+			)
+		)
+		(property "Impedance" "50Ω"
+			(at 203.2 85.598 0)
+			(show_name no)
+			(do_not_autoplace no)
+			(effects
+				(font
+					(size 1.27 1.27)
+				)
+			)
+		)
+		(property "Footprint_Size" ""
+			(at 198.12 83.82 0)
 			(show_name no)
 			(do_not_autoplace no)
@@
 		(in_pos_files yes)
 		(dnp no)
-		(fields_autoplaced yes)
 		(property "Reference" "J13"
-			(at 106.68 116.84 0)
-			(show_name no)
-			(do_not_autoplace no)
-			(effects
-				(font
-					(size 1.27 1.27)
-				)
-			)
-		)
-		(property "Value" "Conn_02x04_Odd_Even"
-			(at 106.68 119.38 0)
+			(at 106.68 116.078 0)
+			(show_name no)
+			(do_not_autoplace no)
+			(effects
+				(font
+					(size 1.27 1.27)
+				)
+			)
+		)
+		(property "Value" "02x04_PinHeader"
+			(at 106.68 118.364 0)
 			(show_name no)
 			(do_not_autoplace no)
@@
 			(at 105.41 125.73 0)
 			(hide yes)
+			(show_name no)
+			(do_not_autoplace no)
+			(effects
+				(font
+					(size 1.27 1.27)
+				)
+			)
+		)
+		(property "Footprint_Size" "2.54mm"
+			(at 106.934 120.396 0)
 			(show_name no)
 			(do_not_autoplace no)
@@
 		(dnp no)
 		(property "Reference" "C90"
-			(at 127.254 61.214 0)
+			(at 127.508 61.214 0)
 			(show_name no)
 			(do_not_autoplace no)
@@
 		)
 		(property "Value" "1uF"
-			(at 128.778 63.754 0)
+			(at 127.762 62.992 0)
 			(show_name no)
 			(do_not_autoplace no)
@@
 		)
 		(property "Vmax" "50V"
-			(at 128.778 66.294 0)
+			(at 129.54 64.77 0)
 			(show_name no)
 			(do_not_autoplace no)
@@
 			(at 125.73 63.5 0)
 			(hide yes)
+			(show_name no)
+			(do_not_autoplace no)
+			(effects
+				(font
+					(size 1.27 1.27)
+				)
+			)
+		)
+		(property "Footprint_Size" "0805"
+			(at 130.048 66.548 0)
 			(show_name no)
 			(do_not_autoplace no)
@@
 		(dnp no)
 		(property "Reference" "C89"
-			(at 115.062 61.214 0)
+			(at 115.316 61.214 0)
 			(show_name no)
 			(do_not_autoplace no)
@@
 		)
 		(property "Value" "10uF"
-			(at 115.57 63.5 0)
+			(at 115.316 62.992 0)
 			(show_name no)
 			(do_not_autoplace no)
@@
 		)
 		(property "Vmax" "16V"
-			(at 117.094 65.786 0)
-			(show_name no)
-			(do_not_autoplace no)
+			(at 117.094 64.77 0)
+			(show_name no)
+			(do_not_autoplace no)
+			(effects
+				(font
+					(size 1.27 1.27)
+				)
+			)
+		)
+		(property "Footprint_Size" "0805"
+			(at 117.856 66.548 0)
+			(show_name no)
+			(do_not_autoplace no)
