File: LRUs/Pad Control Unit/Electrical/Main Controller Board/KICAD PROJECT/master_gse_pcb_project/stm32_controller.kicad_sch (KiCad schematic)
At the start: 65 parts, among them J6 Conn_ST_STDC14, Q10 AO3400A, Q7 AO3400A, Q8 AO3400A, Q9 AO3400A, SW1 SW_SPDT, SW2 SW_Push, U13 STM32L496ZGTx, Y1 8MHz, Y2 32KHz

Commit message: Committ latest changes
Parts:
- added TP16, TP27, TP28: TestPoint, TestPoint:TestPoint_Pad_D2.0mm, symbol Connector:TestPoint
- renumbered D19 to D17, D20 to D18, D21 to D19, D22 to D20, J6 to J9, TP16 to TP17, TP17 to TP18, TP18 to TP19, TP19 to TP20, TP20 to TP21, TP21 to TP22, TP22 to TP23, TP23 to TP24, TP24 to TP25, TP25 to TP26
Connections:
- net AUX_DE: no longer names the net of U13.47 (PB1)
- net AUX_DE: now also TP27.1
- net AUX_RX renamed ADC_RDY
- net AUX_TX: no longer names the net of U13.44 (PC4)
- net AUX_TX: now also TP28.1
- net ~{AUX_RE}: no longer names the net of U13.132 (PG15)
- net ~{AUX_RE}: now also TP16.1
Other:
- note removed: "USART3"

Commit message: Committttt
Parts:
- C42, C43, C44, C45, C46, C47, C49, C50, C51, C52, C53, C54, C55, C56, C57, C58, C63, C64: Footprint_Size (none) -> 0402
- C48, C60, C61: Footprint_Size (none) -> 0805
- C59: Footprint_Size (none) -> 1206
- C62, D17, D18, D19, D20, FB4, R72, R73, R74, R75, R76, R77, R78, R79, R80, R81, R82, R83, R84, R85, R86, R87: Footprint_Size (none) -> 0603
- Q10, Q7, Q8, Q9: Footprint_Size (none) -> SOT-23
- U13: value STM32L496ZGTx -> STM32L496ZGT6
- Y1: Footprint_Size (none) -> SMD_3225
- Y2: Footprint_Size (none) -> SMD_3215
Other:
- moved on the sheet: C63, Y2

Commit message: Commit da changes
Parts:
- BZ1: footprint footprints:MURATA_ELECTRONICS_NORTH_AMERICA_PKM22EPPH2002-B0_0 -> Buzzer_Beeper:Buzzer_Murata_PKMCS0909E; Pitch 10mm -> 9mmx9mm
- D17, D18, D19, D20: Vf 2V -> 3.1V
Connections:
- net OSC32_OUT: now reaches C63.1, U13.9 (PC15), Y2.2
- net BUZZ_MCU: now reaches R74.1, R75.2, U13.68 (PE15)
- net OSC32_IN: now reaches C64.1, U13.8 (PC14), Y2.1
- net BUZZ_P: now reaches BZ1.1 (+), R74.2
Changed lines of the file:
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@@
 	(title_block
 		(title "STM32 Microcontroller")
-		(date "2026-08-27")
+		(date "2026-08-30")
 		(rev "A")
 	)
@@
 	(wire
 		(pts
-			(xy 120.65 237.49) (xy 120.65 243.84)
-		)
-		(stroke
-			(width 0)
-			(type default)
-		)
-	)
-	(wire
-		(pts
 			(xy 354.33 60.96) (xy 354.33 57.15)
 		)
@@
 	(wire
 		(pts
-			(xy 109.22 232.41) (xy 119.38 232.41)
+			(xy 101.6 232.41) (xy 119.38 232.41)
 		)
 		(stroke
@@
 	(wire
 		(pts
-			(xy 109.22 237.49) (xy 120.65 237.49)
+			(xy 101.6 237.49) (xy 120.65 237.49)
 		)
 		(stroke
@@
 	(wire
 		(pts
+			(xy 120.65 237.49) (xy 120.65 243.84)
+		)
+		(stroke
+			(width 0)
+			(type default)
+		)
+	)
+	(wire
+		(pts
 			(xy 152.4 168.91) (xy 165.1 168.91)
 		)
@@
 	(wire
 		(pts
-			(xy 233.68 204.47) (xy 226.06 204.47)
+			(xy 245.11 204.47) (xy 226.06 204.47)
 		)
 		(stroke
@@
 		)
 	)
+	(label "OSC32_OUT"
+		(at 238.76 209.55 180)
+		(effects
+			(font
+				(size 1.27 1.27)
+			)
+			(justify right bottom)
+		)
+	)
 	(label "D4"
 		(at 227.33 240.03 0)
@@
 		)
 	)
+	(label "BUZZ_MCU"
+		(at 152.4 232.41 0)
+		(effects
+			(font
+				(size 1.27 1.27)
+			)
+			(justify left bottom)
+		)
+	)
 	(label "OUT_3"
 		(at 323.85 93.98 0)
@@
 		)
 	)
+	(label "BUZZ_P"
+		(at 106.68 232.41 0)
+		(effects
+			(font
+				(size 1.27 1.27)
+			)
+			(justify left bottom)
+		)
+	)
 	(label "RF_MISO"
 		(at 237.49 173.99 180)
@@
 		)
 	)
+	(label "OSC32_IN"
+		(at 238.76 207.01 180)
+		(effects
+			(font
+				(size 1.27 1.27)
+			)
+			(justify right bottom)
+		)
+	)
 	(label "INTF_3"
 		(at 326.39 124.46 0)
@@
 	(hierarchical_label "~{TC4_FAULT}"
 		(shape input)
-		(at 233.68 204.47 0)
+		(at 245.11 204.47 0)
 		(effects
 			(font
@@
 		(dnp no)
 		(property "Reference" "FB4"
-			(at 180.848 32.766 90)
+			(at 184.658 31.242 90)
 			(show_name no)
 			(do_not_autoplace no)
@@
 		(property "Value" "120R"
 			(at 188.468 32.766 90)
+			(hide yes)
 			(show_name no)
 			(do_not_autoplace no)
@@
 	)
 	(symbol
+		(lib_id "Device:Buzzer")
+		(at 99.06 234.95 0)
+		(mirror y)
+		(unit 1)
+		(body_style 1)
+		(exclude_from_sim no)
+		(in_bom yes)
+		(on_board yes)
+		(in_pos_files yes)
+		(dnp no)
+		(property "Reference" "BZ1"
+			(at 99.06 224.028 0)
+			(show_name no)
+			(do_not_autoplace no)
+			(effects
+				(font
+					(size 1.27 1.27)
+				)
+			)
+		)
+		(property "Value" "Buzzer"
+			(at 99.06 226.568 0)
+			(show_name no)
+			(do_not_autoplace no)
+			(effects
+				(font
+					(size 1.27 1.27)
+				)
+			)
+		)
+		(property "Footprint" "Buzzer_Beeper:Buzzer_Murata_PKMCS0909E"
+			(at 99.695 232.41 90)
+			(hide yes)
+			(show_name no)
+			(do_not_autoplace no)
+			(effects
+				(font
+					(size 1.27 1.27)
+				)
+			)
+		)
+		(property "Datasheet" ""
+			(at 99.695 232.41 90)
+			(hide yes)
+			(show_name no)
+			(do_not_autoplace no)
+			(effects
+				(font
+					(size 1.27 1.27)
+				)
+			)
+		)
+		(property "Description" "Buzzer, polarized"
+			(at 99.06 234.95 0)
+			(hide yes)
+			(show_name no)
+			(do_not_autoplace no)
+			(effects
+				(font
+					(size 1.27 1.27)
+				)
+			)
+		)
+		(property "JLCPCB Part #" ""
+			(at 99.06 234.95 0)
+			(hide yes)
+			(show_name no)
+			(do_not_autoplace no)
+			(effects
+				(font
+					(size 1.27 1.27)
+				)
+			)
+		)
+		(property "Pitch" "9mmx9mm"
+			(at 99.0531 229.108 0)
+			(show_name no)
+			(do_not_autoplace no)
+			(effects
+				(font
+					(size 1.27 1.27)
+				)
+			)
+		)
+		(property "Footprint_Size" ""
+			(at 99.06 234.95 0)
+			(show_name no)
+			(do_not_autoplace no)
+			(effects
+				(font
+					(size 1.27 1.27)
+				)
+			)
+		)
+		(pin "1"
+		)
+		(pin "2"
+		)
+		(instances
+			(project "master_gse_pcb_project"
+				(path "/5dea7f1e-c3ae-4a7c-865b-d3606d04c094/3a85163a-eaab-44e7-b566-82b4544e5347"
+					(reference "BZ1")
+					(unit 1)
+				)
+			)
+		)
+	)
+	(symbol
 		(lib_id "Device:R_Small_US")
 		(at 297.18 233.68 0)
@@
 	)
 	(symbol
-		(lib_id "Device:Buzzer")
-		(at 106.68 234.95 0)
-		(mirror y)
-		(unit 1)
-		(body_style 1)
-		(exclude_from_sim no)
-		(in_bom yes)
-		(on_board yes)
-		(in_pos_files yes)
-		(dnp no)
-		(property "Reference" "BZ1"
-			(at 106.68 224.028 0)
-			(show_name no)
-			(do_not_autoplace no)
-			(effects
-				(font
-					(size 1.27 1.27)
-				)
-			)
-		)
-		(property "Value" "Buzzer"
-			(at 106.68 226.568 0)
-			(show_name no)
-			(do_not_autoplace no)
-			(effects
-				(font
-					(size 1.27 1.27)
-				)
-			)
-		)
-		(property "Footprint" "footprints:MURATA_ELECTRONICS_NORTH_AMERICA_PKM22EPPH2002-B0_0"
-			(at 107.315 232.41 90)
-			(hide yes)
-			(show_name no)
-			(do_not_autoplace no)
-			(effects
-				(font
-					(size 1.27 1.27)
-				)
-			)
-		)
-		(property "Datasheet" ""
-			(at 107.315 232.41 90)
-			(hide yes)
-			(show_name no)
-			(do_not_autoplace no)
-			(effects
-				(font
-					(size 1.27 1.27)
-				)
-			)
-		)
-		(property "Description" "Buzzer, polarized"
-			(at 106.68 234.95 0)
-			(hide yes)
-			(show_name no)
-			(do_not_autoplace no)
-			(effects
-				(font
-					(size 1.27 1.27)
-				)
-			)
-		)
-		(property "JLCPCB Part #" ""
-			(at 106.68 234.95 0)
-			(hide yes)
-			(show_name no)
-			(do_not_autoplace no)
-			(effects
-				(font
-					(size 1.27 1.27)
-				)
-			)
-		)
-		(property "Pitch" "10mm"
-			(at 106.6731 229.108 0)
-			(show_name no)
-			(do_not_autoplace no)
-			(effects
-				(font
-					(size 1.27 1.27)
-				)
-			)
-		)
-		(pin "1"
-		)
-		(pin "2"
-		)
-		(instances
-			(project "master_gse_pcb_project"
-				(path "/5dea7f1e-c3ae-4a7c-865b-d3606d04c094/3a85163a-eaab-44e7-b566-82b4544e5347"
-					(reference "BZ1")
-					(unit 1)
-				)
-			)
-		)
-	)
-	(symbol
 		(lib_id "power:GND")
 		(at 91.44 121.92 90)
@@
 			)
 		)
-		(property "Vf" "2V"
-			(at 336.55 196.342 90)
+		(property "Vf" "3.1V"
+			(at 337.566 196.342 90)
 			(show_name no)
 			(do_not_autoplace no)
@@
 			)
 		)
-		(property "Vf" "2V"
-			(at 312.42 196.342 90)
+		(property "Vf" "3.1V"
+			(at 313.182 196.342 90)
 			(show_name no)
 			(do_not_autoplace no)
@@
 			)
 		)
-		(property "Vf" "2V"
-			(at 361.95 196.342 90)
+		(property "Vf" "3.1V"
+			(at 362.966 196.342 90)
 			(show_name no)
 			(do_not_autoplace no)
@@
 			)
 		)
-		(property "Vf" "2V"
-			(at 386.08 196.342 90)
+		(property "Vf" "3.1V"
+			(at 387.096 196.342 90)
 			(show_name no)
 			(do_not_autoplace no)
