File: LRUs/Pad Control Unit/Electrical/Main Controller Board/KICAD PROJECT/master_gse_pcb_project/usb_c.kicad_sch (KiCad schematic)
At the start: 20 parts, among them J5 GSB1C41110SSHR, U12 AMS1117-3.3

Commit message: Committ latest changes
Parts:
- removed C37, C40, C41: 10uF, Capacitor_Tantalum_SMD:CP_EIA-3216-18_Kemet-A, symbol Device:C_Polarized_Small_US
- added C37, C40, C41: 10uF, Capacitor_SMD:C_0805_2012Metric, symbol Device:C_Small_US
- renumbered D13 to D11, D14 to D12, D15 to D13, D16 to D14, D17 to D15, D18 to D16, J5 to J8
Connections:
- net 3V3_USB: now also C40.1, C41.1
- net GND: now also C37.2, C40.2, C41.2
- net VBUS: now also C37.1

Commit message: Commit da changes
Parts:
- C37, C38, C39, C40, C41: Footprint_Size (none) -> 0805
- D11, D12, D13, D14, D15: Footprint_Size (none) -> X2SON2
- D16: Footprint_Size (none) -> 0603; Vf 2V -> 3.1V
- FB3: Footprint_Size (none) -> 0603; Imp (none) -> 120Ω@100MHz
- R66, R67, R68, R69, R70, R71: Footprint_Size (none) -> 0603
Connections:
- net CC1: now reaches D12.1 (K), J8.A5 (CC1), R69.1
- net CC2: now reaches D14.1 (K), J8.B5 (CC2), R68.1
- net USB_SHIELD: now reaches FB3.1, J8.SH1 (SHIELD), J8.SH2 (SHIELD__1), J8.SH3 (SHIELD__2), J8.SH4 (SHIELD__3)
Other:
- moved on the sheet: C37, C38, D11, D12, D16, J8, R66, R68, R70, R71, U12
