File: LRUs/Valve Control Unit/Electrical/Valve Power Board/valve_control_pcb/RS_485.kicad_sch (KiCad schematic)
At the start: 28 parts, among them J12 Conn_01x04, U22 74LVC1G17, U23 SN6505BDBV, U24 ISO1450BDWR, U25 AMS1117-5.0

Commit message: Commit valve board updates
Parts:
- removed C75: 1uF, Capacitor_SMD:C_0805_2012Metric, symbol Device:C_Small_US
- removed C76, C78: 100nF, Capacitor_SMD:C_0402_1005Metric, symbol Device:C_Small_US
- removed C77, C79, C80, C81: 10uF, Capacitor_SMD:C_0805_2012Metric, symbol Device:C_Small_US
- removed D30, D31: MBR0520LT, Diode_SMD:D_SOD-123, symbol Diode:MBR0520LT
- removed D32: SM712_SOT23, Package_TO_SOT_SMD:SOT-23, symbol Diode:SM712_SOT23
- removed J12: Conn_01x04, Connector_Molex:Molex_Micro-Fit_3.0_43650-0415_1x04_P3.00mm_Vertical, symbol Connector_Generic:Conn_01x04
- removed JP1: SolderJumper_2_Bridged, Jumper:SolderJumper-2_P1.3mm_Bridged_RoundedPad1.0x1.5mm, symbol Jumper:SolderJumper_2_Bridged
- removed R129: 10k, Resistor_SMD:R_0603_1608Metric, symbol Device:R_Small_US
- removed R130, R131: 10, Resistor_SMD:R_0402_1005Metric, symbol Device:R_Small_US
- removed R132: 0, Resistor_SMD:R_1206_3216Metric, symbol Device:R_Small_US
- removed R133: 120, Resistor_SMD:R_0402_1005Metric, symbol Device:R_Small_US
- removed TP100, TP101, TP96, TP97, TP98, TP99: TestPoint, TestPoint:TestPoint_Pad_D2.0mm, symbol Connector:TestPoint
- removed TR1: 750315371, Transformer_SMD:Transformer_Wuerth_750315371, symbol Transformer:Wuerth_750315371
- removed U22: 74LVC1G17, Package_TO_SOT_SMD:SOT-23-5_HandSoldering, symbol 74xGxx:74LVC1G17
- removed U23: SN6505BDBV, Package_TO_SOT_SMD:SOT-23-6, symbol Power_Management:SN6505BDBV
- removed U24: ISO1450BDWR, footprints:SOIC127P1030X265-16N, symbol symbols:ISO1450BDWR
- removed U25: AMS1117-5.0, Package_TO_SOT_SMD:SOT-223-3_TabPin2, symbol Regulator_Linear:AMS1117-5.0
Connections:
- no-connect marks 1 -> 0
Other:
- note removed: "3.3V level shift"
- note removed: "420kHz switching"
- note removed: "Galvanic Power Isolation"
- note removed: "LDO if turn ratio increases"
