File: LRUs/Valve Control Unit/Electrical/Valve Power Board/valve_control_pcb/stm32_microcontroller.kicad_sch (KiCad schematic)
At the start: 56 parts, among them J9 Conn_ST_STDC14, Q10 AO3400A, Q7 AO3400A, Q8 AO3400A, Q9 AO3400A, SW1 SW_SPDT, SW2 SW_Push, U11 W25Q128JVS, U12 STM32L496ZGTx, Y1 8MHz, Y2 32KHz

Commit message: Update valve
Parts:
- removed U11: W25Q128JVS, Package_SO:SOIC-8_5.3x5.3mm_P1.27mm, symbol Memory_Flash:W25Q128JVS
- added C101: 100nF, Capacitor_SMD:C_0402_1005Metric, symbol Device:C_Small_US
- added U30: W25Q128JVE, Package_SON:WSON-8-1EP_8x6mm_P1.27mm_EP3.4x4.3mm, symbol Memory_Flash:W25Q128JVE
- BZ1: footprint footprints:MURATA_ELECTRONICS_NORTH_AMERICA_PKM22EPPH2002-B0_0 -> Buzzer_Beeper:Buzzer_Murata_PKMCS0909E
Connections:
- net +3V3: now also C101.1, U30.8 (VCC)
- net GND: now also C101.2, U30.4 (GND), U30.9 (EP)
- net USB_VBUS_DET: now reaches U12.101 (PA9)
- net D_N: now reaches U12.103 (PA11)
- net D_P: now reaches U12.104 (PA12)
- net SDMMC1_D2: now reaches U12.111 (PC10)
- net SDMMC1_D3: now reaches U12.112 (PC11)
- net SDMMC1_CK: now reaches U12.113 (PC12)
- net SDMMC1_CMD: now reaches U12.116 (PD2)
- net I2C1_SDA: now reaches U12.128 (PG13)
- net I2C1_SCL: now reaches U12.129 (PG14)
- net QUADSPI_BK1_IO3: now reaches U12.18 (PF6)
- net QUADSPI_BK1_IO3: now also U30.7 (~{HOLD}/~{RESET}/IO_{3})
- net QUADSPI_BK1_IO2: now reaches U12.19 (PF7)
- net QUADSPI_BK1_IO2: now also U30.3 (~{WP}/IO_{2})
- net QUADSPI_BK1_IO0: now reaches U12.20 (PF8)
- net QUADSPI_BK1_IO0: now also U30.5 (DI/IO_{0})
- net QUADSPI_BK1_IO1: now reaches U12.21 (PF9)
- net QUADSPI_BK1_IO1: now also U30.2 (DO/IO_{1})
- net QUADSPI_CLK: now reaches U12.22 (PF10)
- net QUADSPI_CLK: now also U30.6 (CLK)
- net ~{QUADSPI_BK1_NCS}: now reaches U12.36 (PA2)
- net ~{QUADSPI_BK1_NCS}: now also U30.1 (~{CS})
- net SDMMC1_D0: now reaches U12.98 (PC8)
- net SDMMC1_D1: now reaches U12.99 (PC9)
Other:
- moved on the sheet: SW1

Commit message: Commit valve board updates
Parts:
- removed BZ1: Buzzer, Buzzer_Beeper:Buzzer_Murata_PKMCS0909E, symbol Device:Buzzer
- removed C101, C27, C28, C29, C30, C31, C32, C34, C36, C38, C39, C40, C41, C42, C43: 100nF, Capacitor_SMD:C_0402_1005Metric, symbol Device:C_Small_US
- removed C33, C45, C46: 1uF, Capacitor_SMD:C_0805_2012Metric, symbol Device:C_Small_US
- removed C35, C37: 20pF, Capacitor_SMD:C_0402_1005Metric, symbol Device:C_Small_US
- removed C44: 4.7uF, Capacitor_SMD:C_1206_3216Metric, symbol Device:C_Small_US
- removed C47: 10nF, Capacitor_SMD:C_0603_1608Metric, symbol Device:C_Small_US
- removed C48, C49: 10pF, Capacitor_SMD:C_0402_1005Metric, symbol Device:C_Small_US
- removed D25, D26, D27, D28: WHITE, LED_SMD:LED_0603_1608Metric, symbol Device:LED
- removed FB1: 120R, Inductor_SMD:L_0603_1608Metric, symbol Device:FerriteBead_Small
- removed J9: Conn_ST_STDC14, Connector_PinHeader_1.27mm:PinHeader_2x07_P1.27mm_Vertical, symbol Connector:Conn_ST_STDC14
- removed Q10, Q7, Q8, Q9: AO3400A, Package_TO_SOT_SMD:SOT-23, symbol Transistor_FET:AO3400A
- removed R100, R105, R96, R98: 4.7k, Resistor_SMD:R_0603_1608Metric, symbol Device:R_Small_US
- removed R101, R102, R103, R106: 0, Resistor_SMD:R_0603_1608Metric, symbol Device:R_Small_US
- removed R104, R95, R97, R99: 47k, Resistor_SMD:R_0603_1608Metric, symbol Device:R_Small_US
- removed R91: 390, Resistor_SMD:R_0603_1608Metric, symbol Device:R_Small_US
- removed R92: 10k, Resistor_SMD:R_0603_1608Metric, symbol Device:R_Small_US
- removed R93: 100, Resistor_SMD:R_0603_1608Metric, symbol Device:R_Small_US
- removed R94: 1M, Resistor_SMD:R_0603_1608Metric, symbol Device:R_Small_US
- removed SW1: SW_SPDT, Button_Switch_THT:SW_Slide_SPDT_Straight_CK_OS102011MS2Q, symbol Switch:SW_SPDT
- removed SW2: SW_Push, Button_Switch_SMD:SW_Push_SPST_NO_Alps_SKRK, symbol Switch:SW_Push
- removed U12: STM32L496ZGTx, Package_QFP:LQFP-144_20x20mm_P0.5mm, symbol MCU_ST_STM32L4:STM32L496ZGTx
- removed U30: W25Q128JVE, Package_SON:WSON-8-1EP_8x6mm_P1.27mm_EP3.4x4.3mm, symbol Memory_Flash:W25Q128JVE
- removed Y1: 8MHz, Crystal:Crystal_SMD_3225-4Pin_3.2x2.5mm, symbol Device:Crystal_GND24
- removed Y2: 32KHz, Crystal:Crystal_SMD_3215-2Pin_3.2x1.5mm, symbol Device:Crystal
Connections:
- no-connect marks 1 -> 0
Other:
- note removed: "Buses"
- note removed: "D1"
- note removed: "D2"
- note removed: "D3"
- note removed: "D4"
- note removed: "Debugging and Status LEDs"
- note removed: "ST-Link"
- note removed: "Supply & Analog Supply Filtering"
