File: LRUs/Valve Control Unit/Electrical/Valve Power Board/valve_control_pcb/valve_control_pcb.kicad_pcb (KiCad board)
At the start: 6 copper layers, 186 x 126 mm, 470 parts, among them J1 0436500215, J10 Conn_01x02_Pin, J11 01x02_PinHeader, J12 Conn_01x04, J13 Conn_Coaxial, J14 Conn_Coaxial, J2 0436500215, J3 0436500215, J4 0436500215, J5 0436500215, J6 0436500215, J7 0768290110, J8 Conn_02x10_Odd_Even, J9 Conn_ST_STDC14, Q1 SiR882ADP, Q10 AO3400A, Q11 SiR882ADP, Q12 SiR882ADP, Q2 SiR882ADP, Q3 SiR882ADP, Q4 SiR882ADP, Q5 SiR882ADP, Q6 SiR882ADP, Q7 AO3400A, Q8 AO3400A, Q9 AO3400A, SW1 SW_SPDT, SW2 SW_Push, U1 TPS27SA08CPWPR, U10 TMP1075DSG, U11 W25Q128JVS, U12 STM32L496ZGTx, U13 AMS1117-3.3, U14 TPS62933P, U15 TPS2116DRL, U16 TPS22810DBV, U17 AMS1117-3.3, U18 TPS22810DBV, U19 TMP1075DSG, U2 TPS27SA08CPWPR, U20 TMP1075DSG, U21 TMP1075DSG, U22 74LVC1G17, U23 SN6505BDBV, U24 ISO1450BDWR, U25 AMS1117-5.0, U27 LM5145RGYR, U28 TMP1075DSG, U29 TMP1075DSG, U3 TPS27SA08CPWPR, U4 TPS27SA08CPWPR, U5 TPS27SA08CPWPR, U6 TPS27SA08CPWPR, U7 TPD6E05U06RVZ, U8 TPD6E05U06RVZ, U9 PCA9306DC, Y1 8MHz, Y2 32KHz

Commit message: Update valve
Parts:
- added C101: 100nF, Capacitor_SMD:C_0402_1005Metric, F.Cu at (90.2, 200.5)
- added C102: 10uF, Capacitor_SMD:C_0805_2012Metric, F.Cu at (77.0, 193.5)
- added C103: 1uF, Capacitor_SMD:C_0805_2012Metric, F.Cu at (77.0, 196.5)
- added C104: 1uF, Capacitor_SMD:C_0805_2012Metric, F.Cu at (77.0, 199.5)
- added C105: 10uF, Capacitor_SMD:C_0805_2012Metric, F.Cu at (77.0, 202.5)
- added C106: 10uF, Capacitor_SMD:C_0805_2012Metric, F.Cu at (77.0, 205.5)
- added C107: 10uF, Capacitor_SMD:C_0805_2012Metric, F.Cu at (77.0, 208.6)
- added C110: 100nF, Capacitor_SMD:C_0402_1005Metric, F.Cu at (72.9, 216.6)
- added D38: WHITE, LED_SMD:LED_0603_1608Metric, F.Cu at (69.9, 222.0)
- added FB3: 120R, Inductor_SMD:L_0603_1608Metric, F.Cu at (76.8, 211.3)
- added J16: Micro_SD_Card_Det2, Connector_Card:microSD_HC_Hirose_DM3AT-SF-PEJM5, F.Cu at (102.0, 136.2)
- added R159: 2.2k, Resistor_SMD:R_0603_1608Metric, F.Cu at (76.8, 213.8)
- added R160: 2.2k, Resistor_SMD:R_0603_1608Metric, F.Cu at (76.8, 216.3)
- added R161: 5.1k, Resistor_SMD:R_0603_1608Metric, F.Cu at (76.8, 218.8)
- added R162: 5.1k, Resistor_SMD:R_0603_1608Metric, F.Cu at (76.8, 221.4)
- added R163: 100k, Resistor_SMD:R_0603_1608Metric, F.Cu at (76.8, 223.9)
- added R164: 200k, Resistor_SMD:R_0603_1608Metric, F.Cu at (80.8, 211.3)
- added R165: 0, Resistor_SMD:R_0603_1608Metric, F.Cu at (118.0, 139.5)
- added R166: 0, Resistor_SMD:R_0603_1608Metric, F.Cu at (118.0, 138.0)
- added R167: 0, Resistor_SMD:R_0603_1608Metric, F.Cu at (118.0, 136.5)
- added R168: 0, Resistor_SMD:R_0603_1608Metric, F.Cu at (118.0, 130.5)
- added R169: 10k, Resistor_SMD:R_0603_1608Metric, F.Cu at (80.8, 223.9)
- added R170: 0, Resistor_SMD:R_0603_1608Metric, F.Cu at (118.0, 132.0)
- added R171: 0, Resistor_SMD:R_0603_1608Metric, F.Cu at (118.0, 133.5)
- added R173: 22, Resistor_SMD:R_0603_1608Metric, F.Cu at (118.0, 135.0)
- added U30: W25Q128JVE, Package_SON:WSON-8-1EP_8x6mm_P1.27mm_EP3.4x4.3mm, F.Cu at (94.0, 195.8)
- added U31: AMS1117-3.3, Package_TO_SOT_SMD:SOT-223-3_TabPin2, F.Cu at (62.9, 219.8)
- added U32: TPD6E05U06RVZ, Package_SON:Texas_R-PUSON-N14, F.Cu at (113.3, 135.0)
- BZ1: footprint footprints:MURATA_ELECTRONICS_NORTH_AMERICA_PKM22EPPH2002-B0_0 -> Buzzer_Beeper:Buzzer_Murata_PKMCS0909E
- R93, R94: moved to F.Cu
- moved BZ1 84.7 mm to (109.5, 105.5)
- moved R94 43.2 mm to (111.0, 113.3), turned to -90 degrees
- moved R93 41.5 mm to (109.5, 113.3), turned to 90 degrees
- moved Q10 6.93 mm to (115.0, 122.9)
- moved D25 6.93 mm to (106.7, 118.0)
- moved D26 6.93 mm to (108.6, 118.0)
- moved D27 6.93 mm to (110.5, 118.0)
- moved R105 6.93 mm to (112.4, 114.0)
- moved R96 6.93 mm to (106.7, 114.0)
- moved R98 6.93 mm to (108.6, 114.0)
- moved D28 6.93 mm to (112.4, 118.0)
- moved R100 6.93 mm to (110.5, 114.0)
- moved Q7 6.93 mm to (104.2, 122.9)
- moved Q9 6.93 mm to (111.4, 122.9)
- moved R95 6.93 mm to (104.1, 126.3)
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Connections:
- R106 pad 2: /Root/stm32_microcontroller/SD_DET -> SD_DET
- U12 pad 101: unconnected-(U12-PA9-Pad101) -> USB_VBUS_DET
- U12 pad 103: unconnected-(U12-PA11-Pad103) -> D_N
- U12 pad 104: unconnected-(U12-PA12-Pad104) -> D_P
- U12 pad 111: unconnected-(U12-PC10-Pad111) -> SDMMC1_D2
- U12 pad 112: unconnected-(U12-PC11-Pad112) -> SDMMC1_D3
- U12 pad 113: unconnected-(U12-PC12-Pad113) -> SDMMC1_CK
- U12 pad 116: unconnected-(U12-PD2-Pad116) -> SDMMC1_CMD
- U12 pad 128: unconnected-(U12-PG13-Pad128) -> I2C1_SDA
- U12 pad 129: unconnected-(U12-PG14-Pad129) -> I2C1_SCL
- U12 pad 18: unconnected-(U12-PF6-Pad18) -> /Root/stm32_microcontroller/QUADSPI_BK1_IO3
- U12 pad 19: unconnected-(U12-PF7-Pad19) -> /Root/stm32_microcontroller/QUADSPI_BK1_IO2
- U12 pad 20: unconnected-(U12-PF8-Pad20) -> /Root/stm32_microcontroller/QUADSPI_BK1_IO0
- U12 pad 21: unconnected-(U12-PF9-Pad21) -> /Root/stm32_microcontroller/QUADSPI_BK1_IO1
- U12 pad 22: unconnected-(U12-PF10-Pad22) -> /Root/stm32_microcontroller/QUADSPI_CLK
- U12 pad 36: unconnected-(U12-PA2-Pad36) -> /Root/stm32_microcontroller/~{QUADSPI_BK1_NCS}
- U12 pad 98: unconnected-(U12-PC8-Pad98) -> SDMMC1_D0
- U12 pad 99: unconnected-(U12-PC9-Pad99) -> SDMMC1_D1
Routing:
- net GND: vias 568 -> 560

Commit message: Commit valve board updates
Parts:
- removed C104: 1uF, Capacitor_SMD:C_0805_2012Metric
- removed C105, C106: 10uF, Capacitor_SMD:C_0805_2012Metric
- added C108: 10uF, Capacitor_SMD:C_0805_2012Metric, F.Cu at (-22.2, 124.9)
- added C109: 10uF, Capacitor_SMD:C_0805_2012Metric, F.Cu at (-22.2, 127.9)
- added C111: 10uF, Capacitor_SMD:C_0805_2012Metric, F.Cu at (-17.7, 121.8)
- added C112: 10uF, Capacitor_SMD:C_0805_2012Metric, F.Cu at (-17.7, 124.9)
- added C113: 10uF, Capacitor_SMD:C_0805_2012Metric, F.Cu at (-17.7, 127.9)
- added C25: 4.7uF, Capacitor_SMD:C_1206_3216Metric, F.Cu at (8.36, 87.5)
- added C60: 10uF, Capacitor_Tantalum_SMD:CP_EIA-3216-18_Kemet-A, F.Cu at (8.18, 79.1)
- added C76: 100nF, Capacitor_SMD:C_0402_1005Metric, F.Cu at (5.12, 121.0)
- added C77: 4.7uF, Capacitor_SMD:C_1206_3216Metric, F.Cu at (8.36, 90.8)
- added C78: 100nF, Capacitor_SMD:C_0402_1005Metric, F.Cu at (5.12, 122.9)
- added D39: RED, LED_SMD:LED_0603_1608Metric, F.Cu at (8.48, 101.6)
- added D40: RED, LED_SMD:LED_0603_1608Metric, F.Cu at (8.48, 104.2)
- added H12: MountingHole_Pad, MountingHole:MountingHole_3.2mm_M3_ISO14580_Pad, F.Cu at (-9.29, 129.5)
- added J25: B2B-XH-A, Connector_JST:JST_XH_B2B-XH-A_1x02_P2.50mm_Vertical, F.Cu at (-2.29, 119.4)
- added J26: B2B-XH-A, Connector_JST:JST_XH_B2B-XH-A_1x02_P2.50mm_Vertical, F.Cu at (-2.29, 127.2)
- added Q19: AO3400A, Package_TO_SOT_SMD:SOT-23, F.Cu at (9.02, 118.3)
- added Q20: AO3400A, Package_TO_SOT_SMD:SOT-23, F.Cu at (9.02, 122.7)
- added R129: 10k, Resistor_SMD:R_0603_1608Metric, F.Cu at (-22.8, 101.5)
- added R134: 1M, Resistor_SMD:R_0603_1608Metric, F.Cu at (75.7, 152.1)
- added R135: 100k, Resistor_SMD:R_0603_1608Metric, F.Cu at (75.7, 154.6)
- added R137: 47k, Resistor_SMD:R_0603_1608Metric, F.Cu at (-22.8, 104.0)
- added R139: 0, Resistor_SMD:R_0603_1608Metric, F.Cu at (75.7, 157.1)
- added R172: 200k, Resistor_SMD:R_0603_1608Metric, F.Cu at (-18.8, 101.5)
- added R174: 0, Resistor_SMD:R_0603_1608Metric, F.Cu at (-18.8, 104.0)
- added R175: 0, Resistor_SMD:R_0603_1608Metric, F.Cu at (-18.8, 106.5)
- added R176: 0, Resistor_SMD:R_0603_1608Metric, F.Cu at (-18.8, 109.0)
- added R177: 0, Resistor_SMD:R_0603_1608Metric, F.Cu at (-18.8, 111.6)
- added R178: 0, Resistor_SMD:R_0603_1608Metric, F.Cu at (-18.8, 114.1)
- added R179: 0, Resistor_SMD:R_0603_1608Metric, F.Cu at (-18.8, 116.6)
- added R180: 0, Resistor_SMD:R_0603_1608Metric, F.Cu at (-18.8, 119.1)
- added R181: 0, Resistor_SMD:R_0603_1608Metric, F.Cu at (-14.8, 99.0)
- added R182: 2.2k, Resistor_SMD:R_0603_1608Metric, F.Cu at (-14.8, 101.5)
- added R183: 2.2k, Resistor_SMD:R_0603_1608Metric, F.Cu at (-14.8, 104.0)
- added R184: 100, Resistor_SMD:R_0603_1608Metric, F.Cu at (-14.8, 106.5)
- added R185: 100, Resistor_SMD:R_0603_1608Metric, F.Cu at (-14.8, 109.0)
- added R186: 0, Resistor_SMD:R_0603_1608Metric, F.Cu at (21.4, 157.1)
- added R187: 0, Resistor_SMD:R_0603_1608Metric, F.Cu at (42.7, 96.8)
- added R188: 0, Resistor_SMD:R_0603_1608Metric, F.Cu at (42.7, 133.5)
- added R189: 0, Resistor_SMD:R_0603_1608Metric, F.Cu at (-14.2, 158.1)
- added R190: 0, Resistor_SMD:R_0603_1608Metric, F.Cu at (77.6, 96.8)
- added R191: 0, Resistor_SMD:R_0603_1608Metric, F.Cu at (77.6, 133.5)
- added R192: 10k, Resistor_SMD:R_0402_1005Metric, F.Cu at (18.0, 153.8)
- added R193: 10k, Resistor_SMD:R_0402_1005Metric, F.Cu at (33.6, 80.5)
- added R194: 10k, Resistor_SMD:R_0402_1005Metric, F.Cu at (33.6, 117.1)
- added R195: 10k, Resistor_SMD:R_0402_1005Metric, F.Cu at (-23.4, 141.7)
- added R196: 10k, Resistor_SMD:R_0402_1005Metric, F.Cu at (68.5, 80.5)
- added R197: 10k, Resistor_SMD:R_0402_1005Metric, F.Cu at (68.5, 117.1)
- added R198: 10k, Resistor_SMD:R_0402_1005Metric, F.Cu at (18.0, 155.8)
- added R199: 10k, Resistor_SMD:R_0402_1005Metric, F.Cu at (33.6, 82.5)
- added R200: 10k, Resistor_SMD:R_0402_1005Metric, F.Cu at (33.6, 119.1)
- added R201: 10k, Resistor_SMD:R_0402_1005Metric, F.Cu at (-23.4, 143.7)
- added R202: 10k, Resistor_SMD:R_0402_1005Metric, F.Cu at (68.5, 82.5)
- added R203: 10k, Resistor_SMD:R_0402_1005Metric, F.Cu at (68.5, 119.1)
- added R204: 90.9k, Resistor_SMD:R_0402_1005Metric, F.Cu at (18.0, 157.8)
- added R205: 90.9k, Resistor_SMD:R_0402_1005Metric, F.Cu at (33.6, 84.5)
- added R206: 90.9k, Resistor_SMD:R_0402_1005Metric, F.Cu at (33.6, 121.1)
- added R207: 90.9k, Resistor_SMD:R_0402_1005Metric, F.Cu at (-23.4, 145.7)
- added R208: 90.9k, Resistor_SMD:R_0402_1005Metric, F.Cu at (68.5, 84.5)
- added R209: 90.9k, Resistor_SMD:R_0402_1005Metric, F.Cu at (68.5, 121.1)
- added R210: 90.9k, Resistor_SMD:R_0402_1005Metric, F.Cu at (18.0, 159.8)
- added R211: 90.9k, Resistor_SMD:R_0402_1005Metric, F.Cu at (33.6, 86.5)
- added R212: 90.9k, Resistor_SMD:R_0402_1005Metric, F.Cu at (33.6, 123.1)
- added R213: 90.9k, Resistor_SMD:R_0402_1005Metric, F.Cu at (-23.4, 147.7)
- added R214: 90.9k, Resistor_SMD:R_0402_1005Metric, F.Cu at (68.5, 86.5)
- added R215: 90.9k, Resistor_SMD:R_0402_1005Metric, F.Cu at (68.5, 123.1)
- added R87: 47k, Resistor_SMD:R_0603_1608Metric, F.Cu at (-26.8, 106.5)
- added R88: 4.7k, Resistor_SMD:R_0603_1608Metric, F.Cu at (-26.8, 109.0)
- added R89: 4.7k, Resistor_SMD:R_0603_1608Metric, F.Cu at (-26.8, 111.6)
- added TP102: TestPoint, TestPoint:TestPoint_Pad_D2.0mm, F.Cu at (-26.8, 79.5)
- added TP103: TestPoint, TestPoint:TestPoint_Pad_D2.0mm, F.Cu at (-26.8, 83.6)
- added TP104: TestPoint, TestPoint:TestPoint_Pad_D2.0mm, F.Cu at (-26.8, 87.6)
- added TP105: TestPoint, TestPoint:TestPoint_Pad_D2.0mm, F.Cu at (-26.8, 91.7)
- added TP106: TestPoint, TestPoint:TestPoint_Pad_D2.0mm, F.Cu at (-26.8, 95.7)
- added TP107: TestPoint, TestPoint:TestPoint_Pad_D2.0mm, F.Cu at (-22.8, 79.5)
- added TP108: TestPoint, TestPoint:TestPoint_Pad_D2.0mm, F.Cu at (-22.8, 83.6)
- added TP109: TestPoint, TestPoint:TestPoint_Pad_D2.0mm, F.Cu at (-22.8, 87.6)
- added TP110: TestPoint, TestPoint:TestPoint_Pad_D2.0mm, F.Cu at (-22.8, 91.7)
- added TP111: TestPoint, TestPoint:TestPoint_Pad_D2.0mm, F.Cu at (50.4, 152.8)
- added TP112: TestPoint, TestPoint:TestPoint_Pad_D2.0mm, F.Cu at (50.4, 156.9)
- added TP113: TestPoint, TestPoint:TestPoint_Pad_D2.0mm, F.Cu at (50.4, 160.9)
- added TP114: TestPoint, TestPoint:TestPoint_Pad_D2.0mm, F.Cu at (50.4, 165.0)
- added TP115: TestPoint, TestPoint:TestPoint_Pad_D2.0mm, F.Cu at (54.4, 152.8)
- added TP116: TestPoint, TestPoint:TestPoint_Pad_D2.0mm, F.Cu at (54.4, 156.9)
- added TP117: TestPoint, TestPoint:TestPoint_Pad_D1.0mm, F.Cu at (58.0, 152.3)
- added TP118: TestPoint, TestPoint:TestPoint_Pad_D2.0mm, F.Cu at (54.4, 160.9)
- added TP119: TestPoint, TestPoint:TestPoint_Pad_D1.0mm, F.Cu at (58.0, 155.4)
- added TP120: TestPoint, TestPoint:TestPoint_Pad_D1.0mm, F.Cu at (58.0, 158.4)
- added TP121: TestPoint, TestPoint:TestPoint_Pad_D1.0mm, F.Cu at (58.0, 161.5)
- added TP122: TestPoint, TestPoint:TestPoint_Pad_D1.0mm, F.Cu at (61.0, 152.3)
- added TP123: TestPoint, TestPoint:TestPoint_Pad_D1.0mm, F.Cu at (61.0, 155.4)
- added TP124: TestPoint, TestPoint:TestPoint_Pad_D1.0mm, F.Cu at (61.0, 158.4)
- added TP125: TestPoint, TestPoint:TestPoint_Pad_D1.0mm, F.Cu at (61.0, 161.5)
- added TP126: TestPoint, TestPoint:TestPoint_Pad_D1.0mm, F.Cu at (64.1, 152.3)
- added TP127: TestPoint, TestPoint:TestPoint_Pad_D1.0mm, F.Cu at (64.1, 155.4)
- added TP128: TestPoint, TestPoint:TestPoint_Pad_D1.0mm, F.Cu at (64.1, 158.4)
- added TP129: TestPoint, TestPoint:TestPoint_Pad_D1.0mm, F.Cu at (69.1, 152.3)
- added TP130: TestPoint, TestPoint:TestPoint_Pad_D1.0mm, F.Cu at (69.1, 155.4)
- added TP131: TestPoint, TestPoint:TestPoint_Pad_D1.0mm, F.Cu at (69.1, 158.4)
- added TP132: TestPoint, TestPoint:TestPoint_Pad_D1.0mm, F.Cu at (69.1, 161.5)
- added TP133: TestPoint, TestPoint:TestPoint_Pad_D1.0mm, F.Cu at (69.1, 164.5)
- added TP134: TestPoint, TestPoint:TestPoint_Pad_D1.0mm, F.Cu at (72.2, 152.3)
- added TP135: TestPoint, TestPoint:TestPoint_Pad_D1.0mm, F.Cu at (72.2, 155.4)
- added TP136: TestPoint, TestPoint:TestPoint_Pad_D1.0mm, F.Cu at (72.2, 158.4)
- added TP137: TestPoint, TestPoint:TestPoint_Pad_D1.0mm, F.Cu at (72.2, 161.5)
- added TP138: TestPoint, TestPoint:TestPoint_Pad_D1.0mm, F.Cu at (72.2, 164.5)
- added TP139: TestPoint, TestPoint:TestPoint_Pad_D1.0mm, F.Cu at (-4.24, 99.3)
- added TP140: TestPoint, TestPoint:TestPoint_Pad_D1.0mm, F.Cu at (-4.24, 102.3)
- added TP141: TestPoint, TestPoint:TestPoint_Pad_D1.0mm, F.Cu at (-4.24, 105.4)
- added TP142: TestPoint, TestPoint:TestPoint_Pad_D1.0mm, F.Cu at (-4.24, 108.4)
- added TP143: TestPoint, TestPoint:TestPoint_Pad_D1.0mm, F.Cu at (-4.24, 111.5)
- added TP144: TestPoint, TestPoint:TestPoint_Pad_D1.0mm, F.Cu at (-4.24, 114.5)
- added TP145: TestPoint, TestPoint:TestPoint_Pad_D1.0mm, F.Cu at (-1.19, 99.3)
- added TP146: TestPoint, TestPoint:TestPoint_Pad_D2.0mm, F.Cu at (-22.8, 95.7)
- added TP147: TestPoint, TestPoint:TestPoint_Pad_D1.0mm, F.Cu at (-1.19, 102.3)
- added TP148: TestPoint, TestPoint:TestPoint_Pad_D1.0mm, F.Cu at (-1.19, 105.4)
- added TP149: TestPoint, TestPoint:TestPoint_Pad_D1.0mm, F.Cu at (-1.19, 108.4)
- added TP150: TestPoint, TestPoint:TestPoint_Pad_D1.0mm, F.Cu at (-1.19, 111.5)
- added TP151: TestPoint, TestPoint:TestPoint_Pad_D1.0mm, F.Cu at (31.2, 140.9)
- added TP152: TestPoint, TestPoint:TestPoint_Pad_D1.0mm, F.Cu at (-25.8, 162.5)
- added TP153: TestPoint, TestPoint:TestPoint_Pad_D1.0mm, F.Cu at (-1.19, 114.5)
- added TP154: TestPoint, TestPoint:TestPoint_Pad_D1.0mm, F.Cu at (1.86, 99.3)
- added TP155: TestPoint, TestPoint:TestPoint_Pad_D1.0mm, F.Cu at (1.86, 102.3)
- added TP156: TestPoint, TestPoint:TestPoint_Pad_D1.0mm, F.Cu at (1.86, 105.4)
- added TP157: TestPoint, TestPoint:TestPoint_Pad_D1.0mm, F.Cu at (1.86, 108.4)
- added TP158: TestPoint, TestPoint:TestPoint_Pad_D1.0mm, F.Cu at (1.86, 111.5)
- added TP159: TestPoint, TestPoint:TestPoint_Pad_D1.0mm, F.Cu at (1.86, 114.5)
- added TP160: TestPoint, TestPoint:TestPoint_Pad_D1.0mm, F.Cu at (4.92, 99.3)
- added TP161: TestPoint, TestPoint:TestPoint_Pad_D1.0mm, F.Cu at (4.92, 102.3)
- added TP162: TestPoint, TestPoint:TestPoint_Pad_D2.0mm, F.Cu at (-18.7, 79.5)
- added TP163: TestPoint, TestPoint:TestPoint_Pad_D2.0mm, F.Cu at (-18.7, 83.6)
- added TP164: TestPoint, TestPoint:TestPoint_Pad_D2.0mm, F.Cu at (-18.7, 87.6)
- added TP165: TestPoint, TestPoint:TestPoint_Pad_D2.0mm, F.Cu at (-18.7, 91.7)
- added TP166: TestPoint, TestPoint:TestPoint_Pad_D2.0mm, F.Cu at (-18.7, 95.7)
- added TP167: TestPoint, TestPoint:TestPoint_Pad_D2.0mm, F.Cu at (-14.7, 79.5)
- added TP168: TestPoint, TestPoint:TestPoint_Pad_D2.0mm, F.Cu at (-14.7, 83.6)
- added TP169: TestPoint, TestPoint:TestPoint_Pad_D2.0mm, F.Cu at (-14.7, 87.6)
- added TP170: TestPoint, TestPoint:TestPoint_Pad_D2.0mm, F.Cu at (-14.7, 91.7)
- added TP171: TestPoint, TestPoint:TestPoint_Pad_D2.0mm, F.Cu at (-14.7, 95.7)
- added TP172: TestPoint, TestPoint:TestPoint_Pad_D2.0mm, F.Cu at (-10.6, 79.5)
- added TP173: TestPoint, TestPoint:TestPoint_Pad_D2.0mm, F.Cu at (-10.6, 83.6)
- added TP174: TestPoint, TestPoint:TestPoint_Pad_D2.0mm, F.Cu at (-10.6, 87.6)
- added TP175: TestPoint, TestPoint:TestPoint_Pad_D1.0mm, F.Cu at (31.0, 152.3)
- added TP176: TestPoint, TestPoint:TestPoint_Pad_D1.0mm, F.Cu at (-7.08, 152.9)
- added TP177: TestPoint, TestPoint:TestPoint_Pad_D1.0mm, F.Cu at (31.0, 164.9)
- added TP178: TestPoint, TestPoint:TestPoint_Pad_D1.0mm, F.Cu at (-7.08, 140.3)
- added TP179: TestPoint, TestPoint:TestPoint_Pad_D1.0mm, F.Cu at (15.0, 166.5)
- added TP180: TestPoint, TestPoint:TestPoint_Pad_D1.0mm, F.Cu at (-7.08, 165.4)
- added TP181: TestPoint, TestPoint:TestPoint_Pad_D1.0mm, F.Cu at (31.0, 155.4)
- added TP182: TestPoint, TestPoint:TestPoint_Pad_D1.0mm, F.Cu at (-7.08, 155.9)
- added TP183: TestPoint, TestPoint:TestPoint_Pad_D1.0mm, F.Cu at (31.0, 168.0)
- added TP184: TestPoint, TestPoint:TestPoint_Pad_D1.0mm, F.Cu at (-7.08, 143.3)
- added TP185: TestPoint, TestPoint:TestPoint_Pad_D1.0mm, F.Cu at (15.0, 169.6)
- added TP186: TestPoint, TestPoint:TestPoint_Pad_D1.0mm, F.Cu at (-7.08, 168.5)
- added TP187: TestPoint, TestPoint:TestPoint_Pad_D1.0mm, F.Cu at (34.1, 152.3)
- added TP188: TestPoint, TestPoint:TestPoint_Pad_D1.0mm, F.Cu at (-4.04, 152.9)
- added TP189: TestPoint, TestPoint:TestPoint_Pad_D1.0mm, F.Cu at (34.1, 164.9)
- added TP190: TestPoint, TestPoint:TestPoint_Pad_D1.0mm, F.Cu at (-4.04, 140.3)
- added TP191: TestPoint, TestPoint:TestPoint_Pad_D1.0mm, F.Cu at (18.0, 166.5)
- added TP192: TestPoint, TestPoint:TestPoint_Pad_D1.0mm, F.Cu at (-4.04, 165.4)
- added TP193: TestPoint, TestPoint:TestPoint_Pad_D2.0mm, F.Cu at (-10.6, 91.7)
- added TP194: TestPoint, TestPoint:TestPoint_Pad_D2.0mm, F.Cu at (-10.6, 95.7)
- added TP195: TestPoint, TestPoint:TestPoint_Pad_D2.0mm, F.Cu at (-6.58, 79.5)
- added TP196: TestPoint, TestPoint:TestPoint_Pad_D2.0mm, F.Cu at (-6.58, 83.6)
- added TP197: TestPoint, TestPoint:TestPoint_Pad_D2.0mm, F.Cu at (-6.58, 87.6)
- added TP198: TestPoint, TestPoint:TestPoint_Pad_D2.0mm, F.Cu at (-6.58, 91.7)
- added TP199: TestPoint, TestPoint:TestPoint_Pad_D2.0mm, F.Cu at (-6.58, 95.7)
- added TP200: TestPoint, TestPoint:TestPoint_Pad_D1.0mm, F.Cu at (-25.8, 165.5)
- added TP201: TestPoint, TestPoint:TestPoint_Pad_D1.0mm, F.Cu at (66.1, 101.2)
- added TP202: TestPoint, TestPoint:TestPoint_Pad_D1.0mm, F.Cu at (66.1, 104.3)
- added TP203: TestPoint, TestPoint:TestPoint_Pad_D1.0mm, F.Cu at (66.1, 137.9)
- added TP204: TestPoint, TestPoint:TestPoint_Pad_D1.0mm, F.Cu at (34.1, 155.4)
- added TP205: TestPoint, TestPoint:TestPoint_Pad_D1.0mm, F.Cu at (-4.04, 155.9)
- added TP206: TestPoint, TestPoint:TestPoint_Pad_D1.0mm, F.Cu at (34.1, 168.0)
- added TP207: TestPoint, TestPoint:TestPoint_Pad_D1.0mm, F.Cu at (-4.04, 143.3)
- added TP208: TestPoint, TestPoint:TestPoint_Pad_D1.0mm, F.Cu at (18.0, 169.6)
- added TP209: TestPoint, TestPoint:TestPoint_Pad_D1.0mm, F.Cu at (-4.04, 168.5)
- added TP210: TestPoint, TestPoint:TestPoint_Pad_D1.0mm, F.Cu at (37.1, 152.3)
- added TP211: TestPoint, TestPoint:TestPoint_Pad_D1.0mm, F.Cu at (-0.98, 152.9)
- added TP212: TestPoint, TestPoint:TestPoint_Pad_D1.0mm, F.Cu at (37.1, 164.9)
- added TP213: TestPoint, TestPoint:TestPoint_Pad_D1.0mm, F.Cu at (-0.98, 140.3)
- added TP214: TestPoint, TestPoint:TestPoint_Pad_D1.0mm, F.Cu at (21.1, 166.5)
- added TP215: TestPoint, TestPoint:TestPoint_Pad_D1.0mm, F.Cu at (-0.98, 165.4)
- added TP216: TestPoint, TestPoint:TestPoint_Pad_D1.0mm, F.Cu at (37.1, 155.4)
- added TP217: TestPoint, TestPoint:TestPoint_Pad_D1.0mm, F.Cu at (-0.98, 155.9)
- added TP218: TestPoint, TestPoint:TestPoint_Pad_D1.0mm, F.Cu at (37.1, 168.0)
- added TP219: TestPoint, TestPoint:TestPoint_Pad_D1.0mm, F.Cu at (-0.98, 143.3)
- added TP220: TestPoint, TestPoint:TestPoint_Pad_D1.0mm, F.Cu at (21.1, 169.6)
- added TP221: TestPoint, TestPoint:TestPoint_Pad_D1.0mm, F.Cu at (-0.98, 168.5)
- added TP222: TestPoint, TestPoint:TestPoint_Pad_D1.0mm, F.Cu at (66.1, 140.9)
- added TP223: TestPoint, TestPoint:TestPoint_Pad_D1.0mm, F.Cu at (4.92, 105.4)
- added TP224: TestPoint, TestPoint:TestPoint_Pad_D1.0mm, F.Cu at (4.92, 108.4)
- added U28: INA821IDRG, Package_SON:WSON-8-1EP_3x3mm_P0.5mm_EP1.45x2.4mm, F.Cu at (73.0, 86.5)
- added U29: INA821IDRG, Package_SON:WSON-8-1EP_3x3mm_P0.5mm_EP1.45x2.4mm, F.Cu at (73.0, 123.2)
- added U33: TMP1075DSG, Package_SON:Texas_DSG0008A_WSON-8-1EP_2x2mm_P0.5mm_EP0.9x1.6mm, F.Cu at (31.5, 171.4)
- added U34: TMP1075DSG, Package_SON:Texas_DSG0008A_WSON-8-1EP_2x2mm_P0.5mm_EP0.9x1.6mm, F.Cu at (-6.58, 146.7)
- added U35: TMP1075DSG, Package_SON:Texas_DSG0008A_WSON-8-1EP_2x2mm_P0.5mm_EP0.9x1.6mm, F.Cu at (15.5, 173.0)
- added U36: TMP1075DSG, Package_SON:Texas_DSG0008A_WSON-8-1EP_2x2mm_P0.5mm_EP0.9x1.6mm, F.Cu at (-6.58, 171.9)
- added U37: AD7689BCP, Package_CSP:LFCSP-20-1EP_4x4mm_P0.5mm_EP2.1x2.1mm, B.Cu at (6.00, 154.1)
- C102: value 10uF -> 100nF; footprint Capacitor_SMD:C_0805_2012Metric -> Capacitor_SMD:C_0402_1005Metric
- C103, C54: value 1uF -> 100nF; footprint Capacitor_SMD:C_0805_2012Metric -> Capacitor_SMD:C_0402_1005Metric
- C51: value 10uF -> 100nF; footprint Capacitor_Tantalum_SMD:CP_EIA-3216-18_Kemet-A -> Capacitor_SMD:C_0402_1005Metric
- C56: value 10uF -> 1uF; footprint Capacitor_Tantalum_SMD:CP_EIA-3216-18_Kemet-A -> Capacitor_SMD:C_0805_2012Metric
- C66, C73, C74, R126, R127, R128, R15, R16, R25, R27, R29, R30, R39, R41, R43, R44, R53, R55, R57, R58, R67, R69, R71, R72, R81, R83, TP16, TP17, TP18, TP19, TP20, TP21, TP22, TP23, TP25, TP26, TP27, TP28, TP31, TP32, TP33, TP34, TP35, TP36, TP37, TP38, TP40, TP41, TP42, TP43, TP46, TP47, TP48, TP49, TP50, TP51, TP52, TP53, TP55, TP56, TP57, TP58, TP61, TP62, TP63, TP64, TP65, TP66, TP67, TP68, TP70, TP71, TP72, TP73, TP76, TP77, TP78, TP79, TP80, TP81, TP82, TP83, TP85, TP86, TP87, TP88: moved to F.Cu
- J1, J2, J3, J4, J5, J6: value 0436500215 -> 0039299047; footprint Connector_Molex:Molex_Micro-Fit_3.0_43650-0215_1x02_P3.00mm_Vertical -> Connector_Molex:Molex_Mini-Fit_Jr_5566-04A2_2x02_P4.20mm_Vertical
- J8: value Conn_02x10_Odd_Even -> IDC-Header_2x10
- R136: value 27k -> 22k
- TP100, TP101, TP96, TP97, TP98, TP99: moved to B.Cu
- TP13: footprint TestPoint:TestPoint_Pad_D2.0mm -> TestPoint:TestPoint_Pad_D1.0mm; moved to F.Cu
- TP14, TP29, TP30, TP44, TP45, TP59, TP60, TP74, TP75, TP89, TP90, TP91, TP92, TP93, TP94, TP95: footprint TestPoint:TestPoint_Pad_D2.0mm -> TestPoint:TestPoint_Pad_D1.0mm
- U10: value TMP1075DSG -> INA821IDRG; footprint Package_SON:WSON-8-1EP_2x2mm_P0.5mm_EP0.9x1.6mm_ThermalVias -> Package_SON:WSON-8-1EP_3x3mm_P0.5mm_EP1.45x2.4mm
- U11: value W25Q128JVS -> TMP1075DSG; footprint Package_SO:SOIC-8_5.3x5.3mm_P1.27mm -> Package_SON:Texas_DSG0008A_WSON-8-1EP_2x2mm_P0.5mm_EP0.9x1.6mm; moved to F.Cu
- U12: value STM32L496ZGTx -> STM32L496ZGT6
- U13: value AMS1117-3.3 -> TMP1075DSG; footprint Package_TO_SOT_SMD:SOT-223-3_TabPin2 -> Package_SON:Texas_DSG0008A_WSON-8-1EP_2x2mm_P0.5mm_EP0.9x1.6mm
- U19, U20, U21: value TMP1075DSG -> INA821IDRG; footprint Package_SON:WSON-8-1EP_2x2mm_P0.5mm_EP0.9x1.6mm_ThermalVias -> Package_SON:WSON-8-1EP_3x3mm_P0.5mm_EP1.45x2.4mm; moved to F.Cu
- U26: value ~ -> TPS259830
- moved R54 439.8 mm to (-23.4, 139.7)
- moved C16 425.8 mm to (-22.2, 153.1)
- moved R56 425.5 mm to (-14.2, 155.6)
- moved R40 418.7 mm to (33.6, 115.2)
- moved C12 403.1 mm to (34.7, 128.5)
- moved R42 402.9 mm to (42.7, 131.0)
- moved R26 388.6 mm to (33.6, 78.5)
- moved TP60 384.5 mm to (-25.8, 159.4)
- moved R28 367.9 mm to (42.7, 94.3)
- moved C8 367.6 mm to (34.7, 91.8)
- moved TP45 348.3 mm to (31.2, 134.8)
- moved TP30 333.9 mm to (31.2, 98.2)
- moved TP90 321.6 mm to (66.1, 134.8)
- moved R82 312.5 mm to (68.5, 115.2)
- moved R68 311.5 mm to (68.5, 78.5)
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Connections:
- net /Root/RS_485/A_RX_MAIN_N renamed /RS-485/A_RX_MAIN_N
- net /Root/RS_485/A_RX_MAIN_P renamed /RS-485/A_RX_MAIN_P
- net /Root/RS_485/RX_MAIN_N renamed /RS-485/RX_MAIN_N
- net /Root/RS_485/RX_MAIN_P renamed /RS-485/RX_MAIN_P
- net /Root/stm32_microcontroller/BOOT renamed /STM32/BOOT
- net /Root/stm32_microcontroller/JTDI renamed /STM32/JTDI
- net /Root/stm32_microcontroller/JTDO renamed /STM32/JTDO
- net /Root/stm32_microcontroller/NRST renamed /STM32/NRST
- net /Root/stm32_microcontroller/QUADSPI_BK1_IO0 renamed /STM32/QUADSPI_BK1_IO0
- net /Root/stm32_microcontroller/QUADSPI_BK1_IO1 renamed /STM32/QUADSPI_BK1_IO1
- net /Root/stm32_microcontroller/QUADSPI_BK1_IO2 renamed /STM32/QUADSPI_BK1_IO2
- net /Root/stm32_microcontroller/QUADSPI_BK1_IO3 renamed /STM32/QUADSPI_BK1_IO3
- net /Root/stm32_microcontroller/QUADSPI_CLK renamed /STM32/QUADSPI_CLK
- net /Root/stm32_microcontroller/VDDA renamed /STM32/VDDA
- net /Root/stm32_microcontroller/~{QUADSPI_BK1_NCS} renamed /STM32/~{QUADSPI_BK1_NCS}
- C102 pad 1: /USB-C/VBUS -> +3V3
- C103 pad 1: /USB-C/VBUS -> Net-(U37-REFIN)
- C107 pad 1: +3V3_SD -> +3V3
- C110 pad 1: +3V3_SD -> +3V3
- C51 pad 1: VBUS -> Net-(U24-VCC2)
- C51 pad 2: GND -> ISOGND
- C54 pad 1: VBUS -> +5V
- C55 pad 1: Net-(U13-VO) -> 3V3_USB
- C56 pad 1: Net-(U13-VO) -> /USB-C/V5P0_USB
- C96 pad 1: /Valves/12V_main/VOUT_MAIN -> +12V
- C97 pad 1: /Valves/12V_main/VOUT_MAIN -> +12V
- J13 pad 1: /Valves/12V_main/VOUT_MAIN -> +12V
- J16 pad 4: +3V3_SD -> +3V3
- J9 pad 4: /Root/stm32_microcontroller/SWDIO -> /STM32/SWDIO
- J9 pad 6: /Root/stm32_microcontroller/SWCLK -> /STM32/SWCLK
- L2 pad 2: /Valves/12V_main/VOUT_MAIN -> +12V
- Q10 pad 1: /Root/stm32_microcontroller/D4 -> /STM32/D4
- Q7 pad 1: /Root/stm32_microcontroller/D1 -> /STM32/D1
- Q8 pad 1: /Root/stm32_microcontroller/D2 -> /STM32/D2
- Q9 pad 1: /Root/stm32_microcontroller/D3 -> /STM32/D3
- R101 pad 2: /Root/stm32_microcontroller/EFUSE_PGOOD -> VALVE2.LSW_LATCH
- R102 pad 1: /Root/stm32_microcontroller/MAIN_TX -> MAIN_TX
- R103 pad 1: /Root/stm32_microcontroller/MAIN_RX -> MAIN_RX
- R104 pad 1: /Root/stm32_microcontroller/D4 -> /STM32/D4
- R106 pad 2: SD_DET -> /STM32/JTDI_STM32
- R114 pad 2: /System Power/5V_MAIN_PG -> 5V_MAIN_PG
- R117 pad 2: /System Power/3V3_STATUS -> 3V3_STATUS
- R155 pad 2: /Valves/12V_main/VOUT_MAIN -> +12V
- R159 pad 1: /USB-C/VBUS -> /USB-C/V5P0_USB
- R163 pad 2: /USB-C/VBUS -> /USB-C/V5P0_USB
- R169 pad 1: +3V3_SD -> +3V3
- R93 pad 1: Net-(U12-PE15) -> Net-(BZ1-+)
- R93 pad 2: Net-(BZ1-+) -> Net-(U12-PB10)
- R94 pad 2: Net-(U12-PE15) -> Net-(U12-PB10)
- R95 pad 1: /Root/stm32_microcontroller/D1 -> /STM32/D1
- R97 pad 1: /Root/stm32_microcontroller/D2 -> /STM32/D2
- R99 pad 1: /Root/stm32_microcontroller/D3 -> /STM32/D3
- TP28 pad 1: /Valves/Valve 2/12V_OUT+ -> VALVE2_LSW_SNS
- TP29 pad 1: /Valves/Valve 2/12V_OUT- -> /Valves/Valve 2/12V_OUT+
- TP30 pad 1: VALVE2_LSW_SNS -> /Valves/Valve 2/12V_OUT-
- TP43 pad 1: /Valves/Valve 3/12V_OUT+ -> VALVE3_LSW_SNS
- TP44 pad 1: /Valves/Valve 3/12V_OUT- -> /Valves/Valve 3/12V_OUT+
- TP45 pad 1: VALVE3_LSW_SNS -> /Valves/Valve 3/12V_OUT-
- TP58 pad 1: /Valves/Valve 4/12V_OUT+ -> VALVE4_LSW_SNS
- TP59 pad 1: /Valves/Valve 4/12V_OUT- -> /Valves/Valve 4/12V_OUT+
- TP60 pad 1: VALVE4_LSW_SNS -> /Valves/Valve 4/12V_OUT-
- TP73 pad 1: /Valves/Valve 5/12V_OUT+ -> VALVE5_LSW_SNS
- TP74 pad 1: /Valves/Valve 5/12V_OUT- -> /Valves/Valve 5/12V_OUT+
- TP75 pad 1: VALVE5_LSW_SNS -> /Valves/Valve 5/12V_OUT-
- TP88 pad 1: /Valves/Valve 6/12V_OUT+ -> VALVE6_LSW_SNS
- TP89 pad 1: /Valves/Valve 6/12V_OUT- -> /Valves/Valve 6/12V_OUT+
- TP90 pad 1: VALVE6_LSW_SNS -> /Valves/Valve 6/12V_OUT-
- TP91 pad 1: VBUS -> /Valves/Valve 1/VSENSE_N
- TP92 pad 1: /System Power/VEN -> /Valves/Valve 1/VSENSE_P
- TP93 pad 1: /System Power/VFB -> /Valves/Valve 2/VSENSE_N
- TP94 pad 1: /System Power/VOUT -> /Valves/Valve 2/VSENSE_P
- TP95 pad 1: /System Power/5V_MAIN_PG -> /Valves/Valve 3/VSENSE_N
- U10 pad 1: I2C1_SDA -> /Valves/Valve 1/VSENSE_DIV_N
- U10 pad 2: I2C1_SCL -> /Valves/Valve 1/GAIN1
- U10 pad 3: TEMP_ALERT1 -> /Valves/Valve 1/GAIN2
- U10 pad 4: GND -> /Valves/Valve 1/VSENSE_DIV_P
- U10 pad 7: GND -> VALVE1_KELVIN_SNS
- U10 pad 8: +3V3 -> +5V
- U11 pad 1: unconnected-(U11-~{CS}-Pad1) -> I2C1_SDA
- U11 pad 2: unconnected-(U11-DO/IO_{1}-Pad2) -> I2C1_SCL
- U11 pad 3: unconnected-(U11-~{WP}/IO_{2}-Pad3) -> TEMP_ALERT1
- U11 pad 4: unconnected-(U11-GND-Pad4) -> GND
- U11 pad 5: unconnected-(U11-DI/IO_{0}-Pad5) -> GND
- U11 pad 6: unconnected-(U11-CLK-Pad6) -> GND
- U11 pad 7: unconnected-(U11-~{HOLD}/~{RESET}/IO_{3}-Pad7) -> GND
- U11 pad 8: unconnected-(U11-VCC-Pad8) -> +3V3
- U12 pad 1: unconnected-(U12-PE2-Pad1) -> VALVE4_LSS_EN
- U12 pad 10: unconnected-(U12-PF0-Pad10) -> VALVE4.LSW_LATCH
- U12 pad 100: unconnected-(U12-PA8-Pad100) -> Net-(U12-PA8)
- U12 pad 102: unconnected-(U12-PA10-Pad102) -> Net-(U12-PA10)
- U12 pad 105: unconnected-(U12-PA13-Pad105) -> /STM32/SWDIO
- U12 pad 109: unconnected-(U12-PA14-Pad109) -> /STM32/SWCLK
- U12 pad 11: unconnected-(U12-PF1-Pad11) -> VALVE4.~{LSW_ST}
- U12 pad 110: unconnected-(U12-PA15-Pad110) -> /STM32/JTDI_STM32
- U12 pad 114: unconnected-(U12-PD0-Pad114) -> VALVE1_LSS_EN
- U12 pad 115: unconnected-(U12-PD1-Pad115) -> VALVE1_HSS_EN
- U12 pad 117: unconnected-(U12-PD3-Pad117) -> VALVE1.LSW_SEL1
- U12 pad 118: unconnected-(U12-PD4-Pad118) -> VALVE1.LSW_SEL2
- U12 pad 119: unconnected-(U12-PD5-Pad119) -> VALVE1.LSW_DIA_EN
- U12 pad 12: unconnected-(U12-PF2-Pad12) -> FAN2_TOGGLE
- U12 pad 122: unconnected-(U12-PD6-Pad122) -> VALVE1.LSW_LATCH
- U12 pad 123: unconnected-(U12-PD7-Pad123) -> VALVE1.~{LSW_ST}
- U12 pad 124: unconnected-(U12-PG9-Pad124) -> VALVE2_LSS_EN
- U12 pad 125: unconnected-(U12-PG10-Pad125) -> VALVE2_HSS_EN
- U12 pad 126: unconnected-(U12-PG11-Pad126) -> VALVE2.LSW_SEL1
- U12 pad 127: unconnected-(U12-PG12-Pad127) -> VALVE2.LSW_SEL2
- U12 pad 13: unconnected-(U12-PF3-Pad13) -> FAN1_TOGGLE
- U12 pad 132: unconnected-(U12-PG15-Pad132) -> VALVE2.LSW_DIA_EN
- U12 pad 133: unconnected-(U12-PB3-Pad133) -> VALVE2.LSW_LATCH
- U12 pad 134: unconnected-(U12-PB4-Pad134) -> VALVE2.~{LSW_ST}
- U12 pad 135: unconnected-(U12-PB5-Pad135) -> VALVE3_LSS_EN
- U12 pad 136: unconnected-(U12-PB6-Pad136) -> VALVE3_HSS_EN
- U12 pad 137: unconnected-(U12-PB7-Pad137) -> VALVE3.LSW_SEL1
- U12 pad 139: unconnected-(U12-PB8-Pad139) -> VALVE3.LSW_SEL2
- U12 pad 14: unconnected-(U12-PF4-Pad14) -> V-12P0_MAIN_PG
- U12 pad 140: unconnected-(U12-PB9-Pad140) -> VALVE3.LSW_DIA_EN
- U12 pad 141: unconnected-(U12-PE0-Pad141) -> VALVE3.LSW_LATCH
- U12 pad 142: unconnected-(U12-PE1-Pad142) -> VALVE3.~{LSW_ST}
- U12 pad 15: unconnected-(U12-PF5-Pad15) -> 3V3_STATUS
- U12 pad 2: unconnected-(U12-PE3-Pad2) -> VALVE4_HSS_EN
- U12 pad 26: unconnected-(U12-PC0-Pad26) -> VALVE6_LSW_SNS
- U12 pad 27: unconnected-(U12-PC1-Pad27) -> VALVE5_LSW_SNS
- U12 pad 28: unconnected-(U12-PC2-Pad28) -> VALVE4_LSW_SNS
- U12 pad 29: unconnected-(U12-PC3-Pad29) -> VALVE3_LSW_SNS
- U12 pad 3: unconnected-(U12-PE4-Pad3) -> VALVE4.LSW_SEL1
- U12 pad 34: unconnected-(U12-PA0-Pad34) -> VALVE2_LSW_SNS
- U12 pad 35: unconnected-(U12-PA1-Pad35) -> VALVE1_LSW_SNS
- U12 pad 37: unconnected-(U12-PA3-Pad37) -> Net-(U12-PA3)
- U12 pad 4: unconnected-(U12-PE5-Pad4) -> VALVE4.LSW_SEL2
- U12 pad 40: unconnected-(U12-PA4-Pad40) -> Net-(U12-PA4)
- U12 pad 41: unconnected-(U12-PA5-Pad41) -> Net-(U12-PA5)
- U12 pad 42: unconnected-(U12-PA6-Pad42) -> Net-(U12-PA6)
- U12 pad 43: unconnected-(U12-PA7-Pad43) -> Net-(U12-PA7)
- U12 pad 44: unconnected-(U12-PC4-Pad44) -> MAIN_TX
- U12 pad 45: unconnected-(U12-PC5-Pad45) -> MAIN_RX
- U12 pad 46: unconnected-(U12-PB0-Pad46) -> Net-(U12-PB0)
- U12 pad 47: unconnected-(U12-PB1-Pad47) -> MAIN_DE
- U12 pad 48: unconnected-(U12-PB2-Pad48) -> ~{MAIN_RE}
- U12 pad 49: unconnected-(U12-PF11-Pad49) -> Net-(U12-PF11)
- U12 pad 5: unconnected-(U12-PE6-Pad5) -> VALVE4.LSW_DIA_EN
- U12 pad 50: unconnected-(U12-PF12-Pad50) -> Net-(U12-PF12)
- U12 pad 53: unconnected-(U12-PF13-Pad53) -> VALVE5.~{LSW_ST}
- U12 pad 54: unconnected-(U12-PF14-Pad54) -> VALVE5.LSW_LATCH
- U12 pad 55: unconnected-(U12-PF15-Pad55) -> VALVE5.LSW_DIA_EN
- U12 pad 56: unconnected-(U12-PG0-Pad56) -> VALVE5.LSW_SEL2
- U12 pad 57: unconnected-(U12-PG1-Pad57) -> VALVE5.LSW_SEL1
- U12 pad 58: unconnected-(U12-PE7-Pad58) -> VALVE5_HSS_EN
- U12 pad 59: unconnected-(U12-PE8-Pad59) -> VALVE5_LSS_EN
- U12 pad 60: unconnected-(U12-PE9-Pad60) -> VALVE6.~{LSW_ST}
- U12 pad 63: unconnected-(U12-PE10-Pad63) -> VALVE6.LSW_LATCH
- U12 pad 64: unconnected-(U12-PE11-Pad64) -> VALVE6.LSW_DIA_EN
- U12 pad 65: unconnected-(U12-PE12-Pad65) -> VALVE6.LSW_SEL2
- U12 pad 66: unconnected-(U12-PE13-Pad66) -> VALVE6.LSW_SEL1
- U12 pad 67: unconnected-(U12-PE14-Pad67) -> VALVE6_HSS_EN
- U12 pad 68: Net-(U12-PE15) -> VALVE6_LSS_EN
- U12 pad 69: unconnected-(U12-PB10-Pad69) -> Net-(U12-PB10)
- U12 pad 7: unconnected-(U12-PC13-Pad7) -> Net-(U12-PC13)
- U12 pad 70: unconnected-(U12-PB11-Pad70) -> Net-(U12-PB11)
- U12 pad 73: unconnected-(U12-PB12-Pad73) -> PIN20_STM32
- U12 pad 74: unconnected-(U12-PB13-Pad74) -> PIN17_STM32
- U12 pad 75: unconnected-(U12-PB14-Pad75) -> PIN16_STM32
- U12 pad 76: unconnected-(U12-PB15-Pad76) -> PIN13_STM32
- U12 pad 77: unconnected-(U12-PD8-Pad77) -> PIN12_STM32
- U12 pad 78: unconnected-(U12-PD9-Pad78) -> PIN9_STM32
- U12 pad 79: /Root/stm32_microcontroller/D4 -> PIN8_STM32
- U12 pad 80: /Root/stm32_microcontroller/D3 -> PIN5_STM32
- U12 pad 81: /Root/stm32_microcontroller/D2 -> /STM32/D4
- U12 pad 82: /Root/stm32_microcontroller/D1 -> /STM32/D3
- U12 pad 85: unconnected-(U12-PD14-Pad85) -> /STM32/D2
- U12 pad 86: unconnected-(U12-PD15-Pad86) -> /STM32/D1
- U12 pad 87: unconnected-(U12-PG2-Pad87) -> Net-(U12-PG2)
- U12 pad 88: unconnected-(U12-PG3-Pad88) -> Net-(U12-PG3)
- U12 pad 89: unconnected-(U12-PG4-Pad89) -> Net-(U12-PG4)
- U12 pad 90: unconnected-(U12-PG5-Pad90) -> Net-(U12-PG5)
- U12 pad 91: unconnected-(U12-PG6-Pad91) -> Net-(U12-PG6)
- U12 pad 92: unconnected-(U12-PG7-Pad92) -> Net-(U12-PG7)
- U12 pad 93: unconnected-(U12-PG8-Pad93) -> Net-(U12-PG8)
- U12 pad 96: unconnected-(U12-PC6-Pad96) -> Net-(U12-PC6)
- U12 pad 97: unconnected-(U12-PC7-Pad97) -> SD_DET
- U13 pad 1: GND -> I2C1_SDA
- U13 pad 2: Net-(U13-VO) -> I2C1_SCL
- U13 pad 3: VBUS -> TEMP_ALERT2
- U14 pad 7: /System Power/5V_MAIN_PG -> 5V_MAIN_PG
- U15 pad 6: Net-(U13-VO) -> 3V3_USB
- U15 pad 8: /System Power/3V3_STATUS -> 3V3_STATUS
- U19 pad 1: I2C1_SDA -> /Valves/Valve 2/VSENSE_DIV_N
- U19 pad 2: I2C1_SCL -> /Valves/Valve 2/GAIN1
- U19 pad 3: TEMP_ALERT2 -> /Valves/Valve 2/GAIN2
- U19 pad 4: GND -> /Valves/Valve 2/VSENSE_DIV_P
- U19 pad 7: +3V3 -> VALVE2_KELVIN_SNS
- U19 pad 8: +3V3 -> +5V
- U20 pad 1: I2C1_SDA -> /Valves/Valve 3/VSENSE_DIV_N
- U20 pad 2: I2C1_SCL -> /Valves/Valve 3/GAIN1
- U20 pad 3: TEMP_ALERT3 -> /Valves/Valve 3/GAIN2
- U20 pad 4: GND -> /Valves/Valve 3/VSENSE_DIV_P
- U20 pad 6: +3V3 -> GND
- U20 pad 7: GND -> VALVE3_KELVIN_SNS
- U20 pad 8: +3V3 -> +5V
- U21 pad 1: I2C1_SDA -> /Valves/Valve 4/VSENSE_DIV_N
- U21 pad 2: I2C1_SCL -> /Valves/Valve 4/GAIN1
- U21 pad 3: TEMP_ALERT4 -> /Valves/Valve 4/GAIN2
- U21 pad 4: GND -> /Valves/Valve 4/VSENSE_DIV_P
- U21 pad 6: +3V3 -> GND
- U21 pad 7: +3V3 -> VALVE4_KELVIN_SNS
- U21 pad 8: +3V3 -> +5V
- U22 pad 4: /Root/RS_485/MAIN_RX -> MAIN_RX
- U24 pad 4: /Root/RS_485/~{MAIN_RE} -> ~{MAIN_RE}
- U24 pad 5: /Root/RS_485/MAIN_TX -> MAIN_TX
- U24 pad 6: /Root/RS_485/MAIN_DE -> MAIN_DE
- U26 pad 1: /Valves/12V_main/VOUT_MAIN -> +12V
- U26 pad 16: /Valves/12V_main/VOUT_MAIN -> +12V
- U26 pad 2: /Valves/12V_main/VOUT_MAIN -> +12V
- U26 pad 25: /Valves/12V_main/VOUT_MAIN -> +12V
- U26 pad 27: /Valves/12V_main/VOUT_MAIN -> +12V
- U26 pad 28: /Valves/12V_main/VOUT_MAIN -> +12V
- U26 pad 29: /Valves/12V_main/VOUT_MAIN -> +12V
- U26 pad 3: /Valves/12V_main/VOUT_MAIN -> +12V
- U26 pad 30: /Valves/12V_main/VOUT_MAIN -> +12V
- U26 pad 31: /Valves/12V_main/VOUT_MAIN -> +12V
- U26 pad 32: /Valves/12V_main/VOUT_MAIN -> +12V
- U31 pad 3: /USB-C/VBUS -> /USB-C/V5P0_USB
- U9 pad 5: /Connectors/I2C_SDA -> I2C_SDA
- U9 pad 6: /Connectors/I2C_SCL -> I2C_SCL
Routing:
- net VALVE6_LSS_EN: track 23.8 -> 0.00 mm
- net VALVE4_LSS_EN: track 23.8 -> 0.00 mm
- net VALVE3_LSS_EN: track 23.8 -> 0.00 mm
- net VALVE5_LSS_EN: track 23.8 -> 0.00 mm
- net VALVE2_LSS_EN: track 23.8 -> 0.00 mm
- net VALVE5_HSS_EN: track 21.6 -> 0.00 mm, vias 1 -> 0
- net VALVE6_HSS_EN: track 21.6 -> 0.00 mm, vias 1 -> 0
- net VALVE2_HSS_EN: track 21.6 -> 0.00 mm, vias 1 -> 0
- net VALVE4_HSS_EN: track 21.6 -> 0.00 mm, vias 1 -> 0
- net VALVE3_HSS_EN: track 21.6 -> 0.00 mm, vias 1 -> 0
- net VALVE1_LSS_EN: track 23.8 -> 11.1 mm
- net VALVE1_HSS_EN: track 27.6 -> 16.5 mm
- net /Valves/Valve 4/LFET_GATE: track 9.50 -> 0.00 mm, vias 1 -> 0
- net /Valves/Valve 3/LFET_GATE: track 9.50 -> 0.00 mm, vias 1 -> 0
- net /Valves/Valve 2/LFET_GATE: track 9.50 -> 0.00 mm, vias 1 -> 0
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- removed copper zone on F.Cu, net /Valves/Valve 1/12V_OUT+
- removed copper zone on F.Cu, net /Valves/Valve 1/12V_OUT-
- removed copper zone on F.Cu, net /Valves/Valve 2/12V_OUT+
- removed copper zone on F.Cu, net /Valves/Valve 2/12V_OUT-
- removed copper zone on F.Cu, net /Valves/Valve 3/12V_OUT+
- removed copper zone on F.Cu, net /Valves/Valve 3/12V_OUT-
- removed copper zone on F.Cu, net /Valves/Valve 4/12V_OUT+
- removed copper zone on F.Cu, net /Valves/Valve 4/12V_OUT-
- removed copper zone on F.Cu, net /Valves/Valve 5/12V_OUT+
- removed copper zone on F.Cu, net /Valves/Valve 5/12V_OUT-
- removed copper zone on F.Cu, net /Valves/Valve 6/12V_OUT+
- removed copper zone on F.Cu, net /Valves/Valve 6/12V_OUT-
Other:
- board size 186 x 126 mm -> 256 x 166 mm
- board text removed: "VALVE 2"
- board text removed: "VALVE 3"
- board text removed: "VALVE 4"
- board text removed: "VALVE 5"
- board text removed: "VALVE 6"
