File: LRUs/Valve Control Unit/Electrical/Valve Power Board/valve_control_pcb/valve_control_pcb.kicad_pcb (KiCad board)
At the start: 6 copper layers, 256 x 166 mm, 724 parts, among them J1 0039299047, J10 0768290106, J11 Conn_01x02_Pin, J12 0436500415, J13 Conn_Coaxial, J14 Conn_Coaxial, J15 GSB1C41110SSHR, J16 Micro_SD_Card_Det2, J17 01x02_PinHeader, J18 XT-60, J19 B4B-XH-A, J2 0039299047, J20 1x2 Screw Terminal, J21 1x2 Screw Terminal, J22 0768290106, J25 B2B-XH-A, J26 B2B-XH-A, J27 B2B-XH-A, J3 0039299047, J4 0039299047, J5 0768290102, J8 IDC-Header_2x10, J9 Conn_ST_STDC14, K1 J107F1CS205VDC.45, Q1 SIR5108DP-T1-RE3-HXY, Q10 AO3400A, Q11 SIR5108DP-T1-RE3-HXY, Q12 SIR5108DP-T1-RE3-HXY, Q13 AO3400A, Q14 STD52P3LLH6, Q15 AO3400A, Q16 AO3400A, Q17 SiR882ADP, Q18 SiR882ADP, Q19 AO3400A, Q2 SIR5108DP-T1-RE3-HXY, Q20 AO3400A, Q21 SiR882ADP, Q22 SiR882ADP, Q3 SIR5108DP-T1-RE3-HXY, Q4 SIR5108DP-T1-RE3-HXY, Q5 AO3400A, Q6 AO3400A, Q7 AO3400A, Q8 AO3400A, Q9 AO3400A, SW1 SW_SPDT, SW2 SW_Push, U1 TPS27SA08CPWPR, U10 ADS124S08IPBSR, U11 TMP1075DSGR, U12 STM32L496ZGT6, U13 TMP1075DSGR, U14 UCC27524D, U15 UCC27524D, U17 AMS1117-3.3, U18 TPS2116DRL, U19 TPS62933P, U2 TPS27SA08CPWPR, U20 TPS22810DBV, U21 TPS22810DBV, U22 74LVC1G17, U23 SN6505BDBVR, U24 ISO1450BDWR, U25 AMS1117-5.0, U26 TPS259830, U27 LM5145RGYR, U28 TPS259830ONRGER, U3 TPS27SA08CPWPR, U30 W25Q128JVE, U31 AMS1117-3.3, U32 TPD6E05U06RVZ, U33 TMP1075DSGR, U34 TMP1075DSGR, U35 TMP1075DSGR, U36 TMP1075DSGR, U4 TPS27SA08CPWPR, U5 LTC4359-MS8, U6 LTC4359-MS8, U7 TPD6E05U06RVZ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

Commit message: Commit updates
Parts:
- C135, C141, C143: footprint Capacitor_SMD:C_0402_1005Metric -> valve_pcb_footprints:C_0402_1005Metric
- C136, C137: footprint Capacitor_SMD:C_0603_1608Metric -> valve_pcb_footprints:C_0603_1608Metric
- R11, R13, R244, R245, R247, R25, R252, R253, R258, R259, R260, R261, R262, R263, R264, R265, R266, R267, R268, R269, R27, R270, R271, R272, R273, R274, R275, R276, R277, R278, R41, R53, R55: footprint Resistor_SMD:R_0603_1608Metric -> valve_pcb_footprints:R_0603_1608Metric
- R39: footprint Capacitor_SMD:C_0603_1608Metric -> valve_pcb_footprints:R_0603_1608Metric
Routing:
- net GND: vias 845 -> 857
