File: LRUs/Valve Control Unit/Electrical/Valve Power Board/valve_control_pcb/valve_control_pcb.kicad_pcb (KiCad board)
At the start: 6 copper layers, 256 x 166 mm, 723 parts, among them J1 01x02_PinHeader, J10 XT-60, J11 B4B-XH-A, J12 0768290102, J13 0039299047, J14 Conn_ST_STDC14, J15 Micro_SD_Card_Det2, J16 GSB1C41110SSHR, J17 0436500415, J18 B2B-XH-A, J19 B2B-XH-A, J2 Conn_01x02_Pin, J20 0768290102, J21 0768290102, J22 0768290106, J23 0768290106, J24 IDC-Header_2x10, J3 Conn_Coaxial, J4 Conn_Coaxial, J5 B2B-XH-A, J6 0039299047, J7 0039299047, J8 0039299047, J9 0039299047, K1 J107F1CS205VDC.45, Q1 AO3400A, Q10 SIR5108DP, Q11 AO3400A, Q12 STD52P3LLH6, Q13 AO3400A, Q14 AO3400A, Q15 AO3400A, Q16 AO3400A, Q17 AO3400A, Q18 AO3400A, Q19 AO3400A, Q2 AO3400A, Q20 AO3400A, Q3 SIR5108DP, Q4 SIR5108DP, Q5 SIR5108DP, Q6 SIR5108DP, Q7 SIR5108DP, Q8 SIR5108DP, Q9 SIR5108DP, SW1 SW_SPDT, SW2 SW_Push, U1 TPS62933P, U10 UCC27524D, U11 UCC27524D, U12 TPS27SA08CPWPR, U13 TPS27SA08CPWPR, U14 TPS27SA08CPWPR, U15 TPS27SA08CPWPR, U16 TPS259830ONRGER, U17 ADS124S08IPBSR, U18 W25Q128JVE, U19 STM32L496ZGT6, U2 TPS22810DBV, U20 TPD6E05U06RVZ, U21 AMS1117-3.3, U22 SN6505BDBVR, U23 ISO1450BDWR, U24 AMS1117-5.0, U25 TMP1075DSGR, U26 TMP1075DSGR, U27 TMP1075DSGR, U28 TMP1075DSGR, U29 TMP1075DSGR, U3 AMS1117-3.3, U30 TMP1075DSGR, U31 PCA9306DC1Z, U32 TPD6E05U06RVZ, U33 TPD6E05U06RVZ, U4 TPS2116DRL, U5 TPS22810DBV, U6 LM74700, U7 LM74700, U8 LM5145RGYR, U9 TPS259830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

Commit message: Commit
Routing:
- net GND: track 32.9 -> 24.1 mm, vias 873 -> 895
- net TEMP_ALERT2: track 133.4 -> 127.5 mm
