File: LRUs/Valve Control Unit/Electrical/Valve Power Board/valve_control_pcb/valve_control_pcb.kicad_sch (KiCad schematic)
At the start: 0 parts

Commit message: Commit valve board updates
Other:
- removed sheet RS_485
Changed lines of the file:
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@@
-		)
-	)
-	(sheet
-		(at 86.36 213.36)
-		(size 43.18 17.78)
-		(exclude_from_sim no)
-		(in_bom yes)
-		(on_board yes)
-		(dnp no)
-		(fields_autoplaced yes)
-		(stroke
-			(width 0.1524)
-			(type solid)
-		)
-		(fill
-			(color 0 0 0 0)
-		)
-		(property "Sheetname" "RS_485"
-			(at 86.36 212.6484 0)
-			(show_name no)
-			(do_not_autoplace no)
-			(effects
-				(font
-					(size 1.27 1.27)
-				)
-				(justify left bottom)
-			)
-		)
-		(property "Sheetfile" "RS_485.kicad_sch"
-			(at 86.36 231.7246 0)
-			(show_name no)
-			(do_not_autoplace no)
-			(effects
-				(font
-					(size 1.27 1.27)
-				)
-				(justify left top)
-			)
-		)
-		(pin "{RS485_MAIN}" bidirectional
-			(at 129.54 217.17 0)
-			(effects
-				(font
-					(size 1.27 1.27)
-				)
-				(justify right)
-			)
-		)
-		(instances
-			(project "valve_control_pcb"
-				(path "/fc15abd0-0409-4213-a92e-28e770df5352"
-					(page "17")
-				)
-			)
 		)
 	)
