File: LRUs/Valve Control Unit/Electrical/Valve Power Board/valve_control_pcb/12V_main.kicad_sch (KiCad schematic)
At the start: 33 parts, among them J13 Conn_Coaxial, J14 Conn_Coaxial, Q11 SiR882ADP, Q12 SiR882ADP, U27 LM5145RGYR

Commit message: Commit valve board updates
Parts:
- added TP111, TP112, TP113, TP114, TP115, TP116, TP118: TestPoint, TestPoint:TestPoint_Pad_D2.0mm, symbol Connector:TestPoint
- added TP117, TP119, TP120, TP121, TP122, TP123, TP124, TP125, TP126, TP127, TP128: TestPoint, TestPoint:TestPoint_Pad_D1.0mm, symbol Connector:TestPoint
Connections:
- net 12V_MAIN_PGOOD: now also TP124.1
- net GND: now also TP122.1, TP123.1
- net VIN: now also TP125.1
- net VOUT_MAIN: now also TP117.1
- net at C93.1, C98.2, R150.1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: now also TP111.1, TP112.1
- net at R144.2, U27.2 (RT): now also TP115.1
- net at C92.1, U27.17 (BST): now also TP118.1
- net at C92.2, L2.1, Q11.1 (S)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: now also TP119.1
- net at R148.2, U27.8 (SYNCIN): now also TP113.1
- net at R145.1, R146.2, U27.1 (EN_UVLO): now also TP116.1
- net at C95.2, R151.2: now also TP120.1
- net at C88.1, U27.3 (SS_TRK): now also TP114.1
- net at C90.1, R147.1, U27.20 (VIN): now also TP126.1
- net at Q12.4 (G), U27.13 (LO): now also TP128.1
- net at C94.2, C95.1, U27.4 (COMP): now also TP121.1
- net at Q11.4 (G), U27.18 (HO): now also TP127.1
Other:
- note added: "12V MAIN"
- note added: "5.7mΩ * 12A = 67mW"
- title: (none) -> 12V MAIN
- moved on the sheet: C88, R144

Commit message: Committttt
Parts:
- J13, J14: Impedance 50 -> 50Ω
Connections:
- net FB: now reaches C93.1, C98.2, R150.1, R152.1, R153.2, TP111.1, TP112.1, U27.5 (FB)
- net BST: now reaches C92.1, TP118.1, U27.17 (BST)
- net SW: now reaches C92.2, L2.1, Q11.1 (S), Q11.2 (S), Q11.3 (S), Q12.5 (D), R149.1, TP119.1, U27.19 (SW)
- net HO: now reaches Q11.4 (G), TP127.1, U27.18 (HO)
- net ILIM: now reaches C91.1, R149.2, U27.11 (ILIM)
- net LO: now reaches Q12.4 (G), TP128.1, U27.13 (LO)
- net COMP: now reaches C94.2, C95.1, TP121.1, U27.4 (COMP)
Other:
- note removed: "5.7mΩ * 12A = 67mW"
- moved on the sheet: R149
Changed lines of the file:
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@@
 		)
 	)
-	(text "5.7mΩ * 12A = 67mW"
-		(exclude_from_sim no)
-		(at 209.296 74.168 0)
-		(effects
-			(font
-				(size 1.27 1.27)
-			)
-		)
-	)
 	(junction
 		(at 156.21 110.49)
@@
 	)
 	(junction
-		(at 157.48 86.36)
-		(diameter 0)
-		(color 0 0 0 0)
-	)
-	(junction
 		(at 246.38 82.55)
 		(diameter 0)
@@
 	)
 	(junction
-		(at 227.33 109.22)
+		(at 179.07 86.36)
 		(diameter 0)
 		(color 0 0 0 0)
 	)
 	(junction
-		(at 76.2 66.04)
+		(at 157.48 86.36)
 		(diameter 0)
 		(color 0 0 0 0)
 	)
 	(junction
-		(at 179.07 86.36)
+		(at 227.33 109.22)
+		(diameter 0)
+		(color 0 0 0 0)
+	)
+	(junction
+		(at 76.2 66.04)
 		(diameter 0)
 		(color 0 0 0 0)
@@
 	(wire
 		(pts
-			(xy 76.2 97.79) (xy 109.22 97.79)
+			(xy 154.94 86.36) (xy 157.48 86.36)
 		)
 		(stroke
@@
 	(wire
 		(pts
-			(xy 157.48 137.16) (xy 158.75 137.16)
+			(xy 76.2 97.79) (xy 109.22 97.79)
 		)
 		(stroke
@@
 	(wire
 		(pts
-			(xy 215.9 91.44) (xy 215.9 90.17)
+			(xy 157.48 137.16) (xy 158.75 137.16)
 		)
 		(stroke
@@
 	(wire
 		(pts
-			(xy 54.61 66.04) (xy 66.04 66.04)
+			(xy 215.9 91.44) (xy 215.9 90.17)
 		)
 		(stroke
@@
 	(wire
 		(pts
-			(xy 157.48 146.05) (xy 157.48 144.78)
+			(xy 54.61 66.04) (xy 66.04 66.04)
 		)
 		(stroke
@@
 	(wire
 		(pts
-			(xy 81.28 78.74) (xy 81.28 81.28)
+			(xy 157.48 146.05) (xy 157.48 144.78)
 		)
 		(stroke
@@
 	(wire
 		(pts
-			(xy 233.68 92.71) (xy 233.68 90.17)
+			(xy 81.28 78.74) (xy 81.28 81.28)
 		)
 		(stroke
@@
 	(wire
 		(pts
-			(xy 179.07 60.96) (xy 179.07 48.26)
+			(xy 233.68 92.71) (xy 233.68 90.17)
 		)
 		(stroke
@@
 	(wire
 		(pts
-			(xy 154.94 86.36) (xy 157.48 86.36)
+			(xy 179.07 60.96) (xy 179.07 48.26)
 		)
 		(stroke
@@
 	(wire
 		(pts
-			(xy 156.21 100.33) (xy 171.45 100.33)
-		)
-		(stroke
-			(width 0)
-			(type default)
-		)
-	)
-	(wire
-		(pts
 			(xy 102.87 68.58) (xy 102.87 66.04)
 		)
@@
 	(wire
 		(pts
+			(xy 154.94 100.33) (xy 171.45 100.33)
+		)
+		(stroke
+			(width 0)
+			(type default)
+		)
+	)
+	(wire
+		(pts
 			(xy 259.08 76.2) (xy 259.08 77.47)
 		)
@@
 		)
 	)
-	(polyline
-		(pts
-			(xy 194.31 77.47) (xy 194.31 78.74)
-		)
-		(stroke
-			(width 0)
-			(type default)
-		)
-	)
 	(wire
 		(pts
-			(xy 154.94 100.33) (xy 156.21 100.33)
-		)
-		(stroke
-			(width 0)
-			(type default)
-		)
-	)
-	(wire
-		(pts
-			(xy 157.48 86.36) (xy 168.91 86.36)
+			(xy 157.48 86.36) (xy 170.18 86.36)
 		)
 		(stroke
@@
 	(wire
 		(pts
-			(xy 173.99 86.36) (xy 179.07 86.36)
+			(xy 175.26 86.36) (xy 179.07 86.36)
 		)
 		(stroke
@@
 		)
 	)
-	(polyline
-		(pts
-			(xy 194.31 78.74) (xy 195.58 78.74)
-		)
-		(stroke
-			(width 0)
-			(type default)
-		)
-	)
 	(wire
 		(pts
@@
 		)
 	)
-	(polyline
+	(wire
 		(pts
-			(xy 194.31 78.74) (xy 198.12 74.93)
+			(xy 200.66 80.01) (xy 200.66 82.55)
 		)
 		(stroke
@@
 		)
 	)
-	(wire
-		(pts
-			(xy 200.66 80.01) (xy 200.66 82.55)
+	(label "LO"
+		(at 154.94 100.33 0)
+		(effects
+			(font
+				(size 1.27 1.27)
+			)
+			(justify left bottom)
 		)
-		(stroke
-			(width 0)
-			(type default)
+	)
+	(label "COMP"
+		(at 157.48 129.54 0)
+		(effects
+			(font
+				(size 1.27 1.27)
+			)
+			(justify left bottom)
+		)
+	)
+	(label "HO"
+		(at 157.48 66.04 0)
+		(effects
+			(font
+				(size 1.27 1.27)
+			)
+			(justify left bottom)
+		)
+	)
+	(label "SW"
+		(at 154.94 78.74 0)
+		(effects
+			(font
+				(size 1.27 1.27)
+			)
+			(justify left bottom)
+		)
+	)
+	(label "BST"
+		(at 154.94 71.12 0)
+		(effects
+			(font
+				(size 1.27 1.27)
+			)
+			(justify left bottom)
+		)
+	)
+	(label "FB"
+		(at 157.48 110.49 0)
+		(effects
+			(font
+				(size 1.27 1.27)
+			)
+			(justify left bottom)
+		)
+	)
+	(label "ILIM"
+		(at 154.94 86.36 0)
+		(effects
+			(font
+				(size 1.27 1.27)
+			)
+			(justify left bottom)
 		)
 	)
@@
 			)
 		)
-		(property "Impedance" "50"
-			(at 263.906 73.152 0)
+		(property "Impedance" "50Ω"
+			(at 264.668 73.152 0)
 			(show_name no)
 			(do_not_autoplace no)
@@
 			)
 		)
-		(property "Impedance" "50"
-			(at 263.906 94.742 0)
+		(property "Impedance" "50Ω"
+			(at 264.668 94.742 0)
 			(show_name no)
 			(do_not_autoplace no)
@@
 	(symbol
 		(lib_id "Device:R_Small_US")
-		(at 171.45 86.36 270)
+		(at 172.72 86.36 270)
 		(unit 1)
 		(body_style 1)
@@
 		(dnp no)
 		(property "Reference" "R149"
-			(at 169.926 85.09 90)
+			(at 171.196 85.09 90)
 			(show_name no)
 			(do_not_autoplace no)
@@
 		)
 		(property "Value" "680"
-			(at 176.53 85.09 90)
+			(at 177.8 85.09 90)
 			(show_name no)
 			(do_not_autoplace no)
@@
 		)
 		(property "Footprint" "Resistor_SMD:R_0603_1608Metric"
-			(at 171.45 86.36 0)
+			(at 172.72 86.36 0)
 			(hide yes)
 			(show_name no)
@@
 		)
 		(property "Datasheet" ""
-			(at 171.45 86.36 0)
+			(at 172.72 86.36 0)
 			(hide yes)
 			(show_name no)
@@
 		)
 		(property "Description" "680 1% 0603 Resistor"
-			(at 171.45 86.36 0)
+			(at 172.72 86.36 0)
 			(hide yes)
 			(show_name no)
@@
 		)
 		(property "Tolerance" "1%"
-			(at 168.656 87.884 90)
+			(at 169.926 87.884 90)
 			(show_name no)
 			(do_not_autoplace no)
@@
 		)
 		(property "JLCPCB Part #" "C23228"
-			(at 171.45 86.36 0)
+			(at 172.72 86.36 0)
 			(hide yes)
 			(show_name no)
@@
 		)
 		(property "Footprint_Size" "0603"
-			(at 175.26 87.884 90)
+			(at 176.53 87.884 90)
 			(show_name no)
 			(do_not_autoplace no)

Commit message: Commit da changes
Parts:
- removed TP111, TP118: TestPoint, TestPoint:TestPoint_Pad_D2.0mm, symbol Connector:TestPoint
- removed TP127, TP128: TestPoint, TestPoint:TestPoint_Pad_D1.0mm, symbol Connector:TestPoint
- added D43: GREEN, LED_SMD:LED_0805_2012Metric, symbol Device:LED
- added R120: 10k, valve_pcb_footprints:R_0603_1608Metric, symbol Device:R_Small_US
- added R246: 10, valve_pcb_footprints:R_0402_1005Metric_GSE, symbol Device:R_Small_US
- C87: footprint Capacitor_SMD:C_1206_3216Metric -> valve_pcb_footprints:C_1206_3216Metric
- C88, C93, C94, C98: footprint Capacitor_SMD:C_0603_1608Metric -> valve_pcb_footprints:C_0603_1608Metric
- C89: footprint Capacitor_SMD:C_0603_1608Metric -> valve_pcb_footprints:C_0603_1608Metric; JLCPCB Part # C12530 -> C43922
- C90, C92: footprint Capacitor_SMD:C_0402_1005Metric -> valve_pcb_footprints:C_0402_1005Metric
- C91, C95: footprint Capacitor_SMD:C_0402_1005Metric -> valve_pcb_footprints:C_0402_1005Metric; JLCPCB Part # C307331 -> C32949
- J13, J14: JLCPCB Part # (none) -> C2894919
- Q11, Q12: value SiR882ADP -> SIR5108DP-T1-RE3-HXY; footprint Package_SO:PowerPAK_SO-8_Single -> valve_pcb_footprints:PowerPAK_SO-8_Single
- R144, R147, R148, R149, R150, R151, R152, R153, R154, R155, R156: footprint Resistor_SMD:R_0603_1608Metric -> valve_pcb_footprints:R_0603_1608Metric
- R145: footprint Resistor_SMD:R_0603_1608Metric -> valve_pcb_footprints:R_0603_1608Metric; JLCPCB Part # C4184 -> C23231
- R146: footprint Resistor_SMD:R_0603_1608Metric -> valve_pcb_footprints:R_0603_1608Metric; JLCPCB Part # C4184 -> C25981
- TP112, TP113, TP114, TP115, TP116: footprint TestPoint:TestPoint_Pad_D2.0mm -> TestPoint:TestPoint_Pad_D1.0mm
- U27: JLCPCB Part # (none) -> C485912
Connections:
- net BST: now also R246.2; no longer C92.1
- net GND: now also D43.1 (K)
- net VOUT_MAIN: now also R120.1
- net VIN_S: now reaches C90.1, R147.1, TP126.1, U27.20 (VIN)
- net RT: now reaches R144.2, TP115.1, U27.2 (RT)
- net EN_UVLO: now reaches R145.1, R146.2, TP116.1, U27.1 (EN_UVLO)
- net VCC: now reaches C89.1, R148.1, U27.14 (VCC)
- net SYNCIN: now reaches R148.2, TP113.1, U27.8 (SYNCIN)
- net SS_TRK: now reaches C88.1, TP114.1, U27.3 (SS_TRK)
- new net: C92.1, R246.1
- new net: D43.2 (A), R120.2
Other:
- moved on the sheet: C89, C90, C92, C97, C98, J13, J14, Q11, Q12, R148, R152, R153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

Commit message: Major changes
Parts:
- Q11, Q12: value SIR5108DP-T1-RE3-HXY -> SIR5108DP; JLCPCB Part # C553986 -> C53262900
Changed lines of the file:
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@@
 	(title_block
 		(title "12V MAIN")
-		(date "2026-10-07")
+		(date "2026-10-08")
 		(rev "A")
 	)
@@
 			)
 		)
-		(property "Value" "SIR5108DP-T1-RE3-HXY"
-			(at 196.596 99.314 0)
+		(property "Value" "SIR5108DP"
+			(at 189.484 99.314 0)
 			(show_name no)
 			(do_not_autoplace no)
@@
 			)
 		)
-		(property "JLCPCB Part #" "C553986"
+		(property "JLCPCB Part #" "C53262900"
 			(at 179.07 100.33 90)
 			(hide yes)
@@
 			)
 		)
-		(property "Value" "SIR5108DP-T1-RE3-HXY"
-			(at 196.596 65.024 0)
+		(property "Value" "SIR5108DP"
+			(at 189.738 65.024 0)
 			(show_name no)
 			(do_not_autoplace no)
@@
 			)
 		)
-		(property "JLCPCB Part #" "C553986"
+		(property "JLCPCB Part #" "C53262900"
 			(at 179.07 66.04 90)
 			(hide yes)

Commit message: Small updates
Parts:
- removed D43: GREEN, LED_SMD:LED_0805_2012Metric, symbol Device:LED
- added D21: RED, LED_SMD:LED_0603_1608Metric, symbol Device:LED
Connections:
- net GND: now also D21.1 (K)
- net at R120.2: now also D21.2 (A)
Changed lines of the file:
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@@
+	)
+	(symbol
+		(lib_id "Device:LED")
+		(at 262.89 123.19 90)
+		(unit 1)
+		(body_style 1)
+		(exclude_from_sim no)
+		(in_bom yes)
+		(on_board yes)
+		(in_pos_files yes)
+		(dnp no)
+		(property "Reference" "D21"
+			(at 265.43 121.158 90)
+			(show_name no)
+			(do_not_autoplace no)
+			(effects
+				(font
+					(size 1.27 1.27)
+				)
+				(justify right)
+			)
+		)
+		(property "Value" "RED"
+			(at 265.43 122.936 90)
+			(show_name no)
+			(do_not_autoplace no)
+			(effects
+				(font
+					(size 1.27 1.27)
+				)
+				(justify right)
+			)
+		)
+		(property "Footprint" "LED_SMD:LED_0603_1608Metric"
+			(at 262.89 123.19 0)
+			(hide yes)
+			(show_name no)
+			(do_not_autoplace no)
+			(effects
+				(font
+					(size 1.27 1.27)
+				)
+			)
+		)
+		(property "Datasheet" ""
+			(at 262.89 123.19 0)
+			(hide yes)
+			(show_name no)
+			(do_not_autoplace no)
+			(effects
+				(font
+					(size 1.27 1.27)
+				)
+			)
+		)
+		(property "Description" "KT-0603R Red LED"
+			(at 262.89 123.19 0)
+			(hide yes)
+			(show_name no)
+			(do_not_autoplace no)
+			(effects
+				(font
+					(size 1.27 1.27)
+				)
+			)
+		)
+		(property "Sim.Pins" "1=K 2=A"
+			(at 262.89 123.19 0)
+			(hide yes)
+			(show_name no)
+			(do_not_autoplace no)
+			(effects
+				(font
+					(size 1.27 1.27)
+				)
+			)
+		)
+		(property "Vf" "2V"
+			(at 266.7 124.714 90)
+			(show_name no)
+			(do_not_autoplace no)
+			(effects
+				(font
+					(size 1.27 1.27)
+				)
+			)
+		)
+		(property "JLCPCB Part #" "C2286"
+			(at 262.89 123.19 90)
+			(hide yes)
+			(show_name no)
+			(do_not_autoplace no)
+			(effects
+				(font
+					(size 1.27 1.27)
+				)
+			)
+		)
+		(property "Footprint_Size" "0603"
+			(at 267.97 126.492 90)
+			(show_name no)
+			(do_not_autoplace no)
+			(effects
+				(font
+					(size 1.27 1.27)
+				)
+			)
+		)
+		(pin "1"
+		)
+		(pin "2"
+		)
+		(instances
+			(project "valve_control_pcb"
+				(path "/d4e8203a-d76f-4c3b-b909-1a52c35190e7/6bd93a81-61dc-4f80-83b3-8d2a24dec243"
+					(reference "D21")
+					(unit 1)
+					(variant
+						(name "My VARIANT DARNIT")
+					)
+				)
+			)
+		)
 	)
 	(symbol
@@
 					(unit 1)
 					(variant
-						(name "My VARIANT DARNIT")
-					)
-				)
-			)
-		)
-	)
-	(symbol
-		(lib_id "Device:LED")
-		(at 262.89 123.19 90)
-		(unit 1)
-		(body_style 1)
-		(exclude_from_sim no)
-		(in_bom yes)
-		(on_board yes)
-		(in_pos_files yes)
-		(dnp no)
-		(property "Reference" "D43"
-			(at 265.43 121.412 90)
-			(show_name no)
-			(do_not_autoplace no)
-			(effects
-				(font
-					(size 1.27 1.27)
-				)
-				(justify right)
-			)
-		)
-		(property "Value" "GREEN"
-			(at 265.43 123.19 90)
-			(show_name no)
-			(do_not_autoplace no)
-			(effects
-				(font
-					(size 1.27 1.27)
-				)
-				(justify right)
-			)
-		)
-		(property "Footprint" "LED_SMD:LED_0805_2012Metric"
-			(at 262.89 123.19 0)
-			(hide yes)
-			(show_name no)
-			(do_not_autoplace no)
-			(effects
-				(font
-					(size 1.27 1.27)
-				)
-			)
-		)
-		(property "Datasheet" ""
-			(at 262.89 123.19 0)
-			(hide yes)
-			(show_name no)
-			(do_not_autoplace no)
-			(effects
-				(font
-					(size 1.27 1.27)
-				)
-			)
-		)
-		(property "Description" "KT-0603R Red LED"
-			(at 262.89 123.19 0)
-			(hide yes)
-			(show_name no)
-			(do_not_autoplace no)
-			(effects
-				(font
-					(size 1.27 1.27)
-				)
-			)
-		)
-		(property "Sim.Pins" "1=K 2=A"
-			(at 262.89 123.19 0)
-			(hide yes)
-			(show_name no)
-			(do_not_autoplace no)
-			(effects
-				(font
-					(size 1.27 1.27)
-				)
-			)
-		)
-		(property "Vf" "3.1V"
-			(at 267.716 124.968 90)
-			(show_name no)
-			(do_not_autoplace no)
-			(effects
-				(font
-					(size 1.27 1.27)
-				)
-			)
-		)
-		(property "JLCPCB Part #" "C2297"
-			(at 262.89 123.19 90)
-			(hide yes)
-			(show_name no)
-			(do_not_autoplace no)
-			(effects
-				(font
-					(size 1.27 1.27)
-				)
-			)
-		)
-		(property "Footprint_Size" "0805"
-			(at 267.97 126.746 90)
-			(show_name no)
-			(do_not_autoplace no)
-			(effects
-				(font
-					(size 1.27 1.27)
-				)
-			)
-		)
-		(pin "1"
-		)
-		(pin "2"
-		)
-		(instances
-			(project "valve_control_pcb"
-				(path "/d4e8203a-d76f-4c3b-b909-1a52c35190e7/6bd93a81-61dc-4f80-83b3-8d2a24dec243"
-					(reference "D43")
-					(unit 1)
-					(variant

Commit message: Fixes
Added hops, fixed the planes, and fixed minor issues
Parts:
- renumbered C85 to C23, C86 to C24, C87 to C25, C88 to C26, C89 to C27, C90 to C28, C91 to C29, C93 to C30, C94 to C31, C92 to C32, C95 to C33, C96 to C34, C97 to C35, C98 to C36, D21 to D5, J13 to J3, J14 to J4, Q11 to Q5, Q12 to Q6, R144 to R26, R145 to R27, R146 to R28, R147 to R29, R148 to R30, R246 to R31, R149 to R32, R150 to R33, R151 to R34, R152 to R35, R153 to R36, R154 to R37, R155 to R38, R156 to R39, R120 to R40, TP125 to TP10, TP124 to TP11, TP115 to TP12, TP114 to TP13, TP116 to TP14, TP113 to TP15, TP126 to TP16, TP121 to TP17, TP122 to TP18, TP123 to TP19, TP112 to TP20, TP119 to TP21, TP120 to TP22, TP117 to TP23, U27 to U8
