File: LRUs/Valve Control Unit/Electrical/Valve Power Board/valve_control_pcb/TMP1075.kicad_sch (KiCad schematic)
At the start: 3 parts, among them U10 TMP1075DSG

Commit message: Commit valve board updates
Parts:
- removed U10: TMP1075DSG, Package_SON:WSON-8-1EP_2x2mm_P0.5mm_EP0.9x1.6mm_ThermalVias, symbol Sensor_Temperature:TMP1075DSG
- added TP175, TP181, TP187, TP204, TP210, TP216: TestPoint, TestPoint:TestPoint_Pad_D1.0mm, symbol Connector:TestPoint
- added U11: TMP1075DSG, Package_SON:Texas_DSG0008A_WSON-8-1EP_2x2mm_P0.5mm_EP0.9x1.6mm, symbol Sensor_Temperature:TMP1075DSG
Connections:
- net +3V3: now also TP187.1, U11.8 (V+)
- net A0: now also TP204.1, U11.7 (A0)
- net A1: now also TP210.1, U11.6 (A1)
- net A2: now also TP216.1, U11.5 (A2)
- net ALERT: now also TP175.1, U11.3 (ALERT)
- net GND: now also TP181.1, U11.4 (GND), U11.9 (EP)
- net SCL: now also U11.2 (SCL)
- net SDA: now also U11.1 (SDA)
Other:
- note added: "TMP1075"
- title: (none) -> TMP1075

Commit message: Commit da changes
Parts:
- C26: footprint Capacitor_SMD:C_0402_1005Metric -> valve_pcb_footprints:C_0402_1005Metric
- R90: footprint Resistor_SMD:R_0603_1608Metric -> valve_pcb_footprints:R_0603_1608Metric
- U11: value TMP1075DSG -> TMP1075DSGR; Footprint_Size (none) -> WSON-8-EP(2x2); JLCPCB Part # (none) -> C2870250
Other:
- moved on the sheet: C26, R90, TP175, TP181, TP187, TP204, TP210, TP216, U11

Commit message: Fixes
Added hops, fixed the planes, and fixed minor issues
Parts:
- renumbered C26 to C127, R90 to R215, TP204 to TP149, TP210 to TP150, TP216 to TP151, TP181 to TP152, TP187 to TP153, TP175 to TP154, U11 to U25
