File: LRUs/Valve Control Unit/Electrical/Valve Power Board/valve_control_pcb/adc.kicad_sch (KiCad schematic)
At the start: 8 parts, among them U37 AD7689BCP

Commit message: Committttt
Parts:
- removed U37: AD7689BCP, Package_CSP:LFCSP-20-1EP_4x4mm_P0.5mm_EP2.1x2.1mm, symbol Analog_ADC:AD7689xCP
- added C104, C105, C106, C114, C115, C116, C117, C118, C119: 100nF, Capacitor_SMD:C_0402_1005Metric, symbol Device:C_Small_US
- added C120: 4.7uF, Capacitor_SMD:C_1206_3216Metric, symbol Device:C_Small_US
- added R186, R187, R192, R195, R198, R201, R204, R207, R210, R213, R216, R219: 15k, Resistor_SMD:R_0402_1005Metric, symbol Device:R_Small_US
- added R188, R189, R193, R196, R199, R202, R205, R208, R211, R214, R217, R220: 90.9k, Resistor_SMD:R_0402_1005Metric, symbol Device:R_Small_US
- added R190, R191, R194, R197, R200, R203, R206, R209, R212, R215, R218, R221: 1k, Resistor_SMD:R_0603_1608Metric, symbol Device:R_Small_US
- added R222: 0, Resistor_SMD:R_0603_1608Metric, symbol Device:R_Small_US
- added TP225, TP226: TestPoint, TestPoint:TestPoint_Pad_D1.0mm, symbol Connector:TestPoint
- added U10: ADS124S08IPBSR, valve_pcb_footprints:QFP50P700X700X120-32N, symbol valve_pcb_symbols:ADS124S08IPBSR
- C112, C113: value 10uF -> 100nF; footprint Capacitor_SMD:C_0805_2012Metric -> Capacitor_SMD:C_0402_1005Metric; Footprint_Size 0805 -> 0402; JLCPCB Part # C95841 -> C307331; Vmax 16V -> 50V
- C78: value 100nF -> 1uF; footprint Capacitor_SMD:C_0402_1005Metric -> Capacitor_SMD:C_0805_2012Metric; Footprint_Size 0402 -> 0805; JLCPCB Part # C307331 -> C28323
Connections:
- net +3V3: now also U10.15 (IOVDD), U10.16 (DVDD)
- net +5V: now also U10.26 (AVDD); no longer C112.1
- net GND: now also C104.2, C105.2, C106.2, C114.2, C115.2, C116.2, C117.2, C118.2, C119.2, C120.2, R188.1, R189.1, R193.1, R196.1, R199.1, R202.1, R205.1, R208.1, R211.1, R214.1, R217.1, R220.1, R222.1, U10.14 (DGND), U10.24 (REFCOM), U10.27 (AVSS), U10.28 (AVSS-SW)
- net VALVE3_VSENSE_FILT_N: now reaches C113.1
- net VALVE3_VSENSE_FILT_N: now also R203.1, U10.2 (AIN5)
- net VALVE1_VSENSE_FILT_P: now reaches C103.1
- net VALVE1_VSENSE_FILT_P: now also R190.1, U10.7 (AIN0)
- net CLK: now reaches TP223.1
- net CLK: now also R222.2, U10.17 (CLK)
- net REFN0: now reaches TP224.1
- net REFN0: now also U10.29 (REFN0)
- new net ADC_MISO: U10.12 (DOUT/~{DRDY})
- new net ADC_MOSI: U10.10 (DIN)
- new net ADC_SCLK: U10.11 (SCLK)
- new net ADC_START: U10.8 (START/SYNC)
- new net AINCOM: TP226.1, U10.1 (AINCOM)
- new net REFOUT: C120.1, U10.23 (REFOUT)
- new net REFP0: TP225.1, U10.30 (REFP0)
- new net VALVE1_VSENSE_DIV_N: R187.1, R189.2, R191.2
- new net VALVE1_VSENSE_DIV_P: R186.1, R188.2, R190.2
- new net VALVE1_VSENSE_FILT_N: C104.1, R191.1, U10.6 (AIN1)
- new net VALVE1_VSENSE_N: R187.2
- new net VALVE1_VSENSE_P: R186.2
- new net VALVE2_VSENSE_DIV_N: R195.1, R196.2, R197.2
- new net VALVE2_VSENSE_DIV_P: R192.1, R193.2, R194.2
- new net VALVE2_VSENSE_FILT_N: C106.1, R197.1, U10.4 (AIN3)
- new net VALVE2_VSENSE_FILT_P: C105.1, R194.1, U10.5 (AIN2)
- new net VALVE2_VSENSE_N: R195.2
- new net VALVE2_VSENSE_P: R192.2
- new net VALVE3_VSENSE_DIV_N: R201.1, R202.2, R203.2
- new net VALVE3_VSENSE_DIV_P: R198.1, R199.2, R200.2
- new net VALVE3_VSENSE_FILT_P: C112.1, R200.1, U10.3 (AIN4)
- new net VALVE3_VSENSE_N: R201.2
- new net VALVE3_VSENSE_P: R198.2
- new net VALVE4_VSENSE_DIV_N: R207.1, R208.2, R209.2
- new net VALVE4_VSENSE_DIV_P: R204.1, R205.2, R206.2
- new net VALVE4_VSENSE_FILT_N: C115.1, R209.1, U10.31 (REFN1/AIN7)
- new net VALVE4_VSENSE_FILT_P: C114.1, R206.1, U10.32 (REFP1/AIN6)
- new net VALVE4_VSENSE_N: R207.2
- new net VALVE4_VSENSE_P: R204.2
- new net VALVE5_VSENSE_DIV_N: R213.1, R214.2, R215.2
- new net VALVE5_VSENSE_DIV_P: R210.1, R211.2, R212.2
- new net VALVE5_VSENSE_FILT_N: C117.1, R215.1, U10.21 (GPIO1/AIN9)
- new net VALVE5_VSENSE_FILT_P: C116.1, R212.1, U10.22 (GPIO0/AIN8)
- new net VALVE5_VSENSE_N: R213.2
- new net VALVE5_VSENSE_P: R210.2
- new net VALVE6_VSENSE_DIV_N: R219.1, R220.2, R221.2
- new net VALVE6_VSENSE_DIV_P: R216.1, R217.2, R218.2
- new net VALVE6_VSENSE_FILT_N: C119.1, R221.1, U10.19 (GPIO3/AIN11)
- new net VALVE6_VSENSE_FILT_P: C118.1, R218.1, U10.20 (GPIO2/AIN10)
- new net VALVE6_VSENSE_N: R219.2
- new net VALVE6_VSENSE_P: R216.2
- new net ~{ADC_CS}: U10.9 (~{CS})
- new net ~{ADC_DRDY}: U10.13 (~{DRDY})
- new net ~{ADC_RESET}: U10.18 (~{RESET})
Other:
- note added: "ADC"
- note added: "VALVE 1"
- note added: "VALVE 2"
- note added: "VALVE 3"
- note added: "VALVE 4"
- note added: "VALVE 5"
- note added: "VALVE 6"
- note added: "VOLTAGE DIVIDER & FILTER"
- title: (none) -> ADC

Commit message: Commit da changes
Parts:
- added R228, R229, R230, R231, R232, R233, R234: 0, valve_pcb_footprints:R_0603_1608Metric, symbol Device:R_Small_US
- added TP159, TP227: TestPoint, TestPoint:TestPoint_Pad_D1.0mm, symbol Connector:TestPoint
- C102, C103, C104, C105, C106, C112, C113, C114, C115, C116, C117, C118, C119: footprint Capacitor_SMD:C_0402_1005Metric -> valve_pcb_footprints:C_0402_1005Metric
- C120: footprint Capacitor_SMD:C_1206_3216Metric -> valve_pcb_footprints:C_1206_3216Metric
- C78: footprint Capacitor_SMD:C_0805_2012Metric -> valve_pcb_footprints:C_0805_2012Metric
- R186, R187, R188, R189, R192, R193, R195, R196, R198, R199, R201, R202, R204, R205, R207, R208, R210, R211, R213, R214, R216, R217, R219, R220: footprint Resistor_SMD:R_0402_1005Metric -> valve_pcb_footprints:R_0402_1005Metric_GSE
- R190, R191, R194, R197, R200, R203, R206, R209, R212, R215, R218, R221: footprint Resistor_SMD:R_0603_1608Metric -> valve_pcb_footprints:R_0402_1005Metric_GSE; Footprint_Size 0603 -> 0402; JLCPCB Part # C21190 -> C11702
- R222: footprint Resistor_SMD:R_0603_1608Metric -> valve_pcb_footprints:R_0603_1608Metric
- U10: JLCPCB Part # (none) -> C2870171
Connections:
- net ADC_MISO: now also R233.1; no longer U10.12 (DOUT/~{DRDY})
- net ADC_MOSI: now also R232.1; no longer U10.10 (DIN)
- net ADC_SCLK: now also R228.1; no longer U10.11 (SCLK)
- net ADC_START: now also R230.1; no longer U10.8 (START/SYNC)
- net GND: now also TP227.1
- net REFOUT: now also TP159.1
- net ~{ADC_CS}: now also R229.1; no longer U10.9 (~{CS})
- net ~{ADC_DRDY}: now also R234.1; no longer U10.13 (~{DRDY})
- net ~{ADC_RESET}: now also R231.1; no longer U10.18 (~{RESET})
- new net MISO: R233.2, U10.12 (DOUT/~{DRDY})
- new net MOSI: R232.2, U10.10 (DIN)
- new net SCLK: R228.2, U10.11 (SCLK)
- new net START: R230.2, U10.8 (START/SYNC)
- new net ~{CS}: R229.2, U10.9 (~{CS})
- new net ~{DRDY}: R234.2, U10.13 (~{DRDY})
- new net ~{RESET}: R231.2, U10.18 (~{RESET})
Other:
- note added: "14"
- note added: "4"
- moved on the sheet: C120

Commit message: Major changes due to architecture
Added battery muxing for valve power, igniter system, and separate system battery for control electronics
Connections:
- net VALVE5_VSENSE_DIV_N renamed IGN_VSENSE_DIV_N
- net VALVE5_VSENSE_DIV_P renamed IGN_VSENSE_DIV_P
- net VALVE5_VSENSE_FILT_N renamed IGN_VSENSE_FILT_N
- net VALVE5_VSENSE_FILT_P renamed IGN_VSENSE_FILT_P
- net VALVE5_VSENSE_N renamed IGN_VSENSE_N
- net VALVE5_VSENSE_P renamed IGN_VSENSE_P
- net VALVE6_VSENSE_DIV_N renamed VBUS_VSENSE_DIV_N
- net VALVE6_VSENSE_DIV_P renamed VBUS_VSENSE_DIV_P
- net VALVE6_VSENSE_FILT_N renamed VBUS_VSENSE_FILT_N
- net VALVE6_VSENSE_FILT_P renamed VBUS_VSENSE_FILT_P
- net VALVE6_VSENSE_N renamed VBUS_VSENSE_N
- net VALVE6_VSENSE_P renamed VBUS_VSENSE_P
Other:
- note added: "18"
- note added: "9"
- note added: "IGNITER BATTERY INPUT"
- note added: "VALVE BATTERY INPUT"
- note removed: "VALVE 5"
- note removed: "VALVE 6"
Changed lines of the file:
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@@
+		)
+	)
+	(text "VALVE BATTERY INPUT"
+		(exclude_from_sim no)
+		(at 52.324 250.444 0)
+		(effects
+			(font
+				(size 2.54 2.54)
+				(thickness 0.3175)
+			)
 		)
 	)
@@
 		)
 	)
-	(text "4"
+	(text "IGNITER BATTERY INPUT"
 		(exclude_from_sim no)
-		(at 50.292 242.824 0)
-		(effects
-			(font
-				(size 1.27 1.27)
-				(color 11 113 0 1)
+		(at 53.594 209.804 0)
+		(effects
+			(font
+				(size 2.54 2.54)
+				(thickness 0.3175)
 			)
 		)
@@
 		)
 	)
-	(text "4"
-		(exclude_from_sim no)
-		(at 50.292 217.424 0)
-		(effects
-			(font
-				(size 1.27 1.27)
-				(color 11 113 0 1)
-			)
-		)
-	)
-	(text "4"
-		(exclude_from_sim no)
-		(at 50.292 258.064 0)
-		(effects
-			(font
-				(size 1.27 1.27)
-				(color 11 113 0 1)
-			)
-		)
-	)
 	(text "14"
 		(exclude_from_sim no)
@@
 		)
 	)
-	(text "VALVE 5"
+	(text "18"
 		(exclude_from_sim no)
-		(at 59.182 210.312 0)
-		(effects
-			(font
-				(size 2.54 2.54)
-				(thickness 0.3175)
+		(at 52.578 202.184 0)
+		(effects
+			(font
+				(size 1.27 1.27)
+				(color 11 113 0 1)
+			)
+		)
+	)
+	(text "18"
+		(exclude_from_sim no)
+		(at 52.578 217.678 0)
+		(effects
+			(font
+				(size 1.27 1.27)
+				(color 11 113 0 1)
+			)
+		)
+	)
+	(text "9"
+		(exclude_from_sim no)
+		(at 51.054 242.824 0)
+		(effects
+			(font
+				(size 1.27 1.27)
+				(color 11 113 0 1)
 			)
 		)
@@
 		)
 	)
-	(text "VALVE 6"
-		(exclude_from_sim no)
-		(at 59.182 250.698 0)
-		(effects
-			(font
-				(size 2.54 2.54)
-				(thickness 0.3175)
-			)
-		)
-	)
 	(text "4"
 		(exclude_from_sim no)
@@
 		)
 	)
+	(text "9"
+		(exclude_from_sim no)
+		(at 51.054 258.064 0)
+		(effects
+			(font
+				(size 1.27 1.27)
+				(color 11 113 0 1)
+			)
+		)
+	)
 	(text "14"
 		(exclude_from_sim no)
@@
 				(size 2.54 2.54)
 				(thickness 0.3175)
-			)
-		)
-	)
-	(text "4"
-		(exclude_from_sim no)
-		(at 50.292 202.184 0)
-		(effects
-			(font
-				(size 1.27 1.27)
-				(color 11 113 0 1)
 			)
 		)
@@
 	(wire
 		(pts
+			(xy 71.12 242.57) (xy 88.9 242.57)
+		)
+		(stroke
+			(width 0)
+			(type default)
+		)
+	)
+	(wire
+		(pts
 			(xy 299.72 144.78) (xy 335.28 144.78)
 		)
@@
 	(wire
 		(pts
+			(xy 71.12 257.81) (xy 88.9 257.81)
+		)
+		(stroke
+			(width 0)
+			(type default)
+		)
+	)
+	(wire
+		(pts
 			(xy 180.34 113.03) (xy 180.34 142.24)
 		)
@@
 	(wire
 		(pts
-			(xy 71.12 257.81) (xy 88.9 257.81)
-		)
-		(stroke
-			(width 0)
-			(type default)
-		)
-	)
-	(wire
-		(pts
 			(xy 316.23 137.16) (xy 316.23 138.43)
 		)
@@
 		(pts
 			(xy 185.42 154.94) (xy 259.08 154.94)
-		)
-		(stroke
-			(width 0)
-			(type default)
-		)
-	)
-	(wire
-		(pts
-			(xy 71.12 242.57) (xy 88.9 242.57)
 		)
 		(stroke
@@
 		)
 	)
-	(label "VALVE6_VSENSE_DIV_P"
+	(label "VBUS_VSENSE_DIV_P"
 		(at 110.49 242.57 0)
 		(effects
@@
 		)
 	)
-	(label "VALVE5_VSENSE_FILT_P"
+	(label "IGN_VSENSE_FILT_P"
 		(at 209.5085 152.4 0)
 		(effects
@@
 		)
 	)
-	(label "VALVE5_VSENSE_FILT_N"
+	(label "IGN_VSENSE_FILT_N"
 		(at 209.5085 154.94 0)
 		(effects
@@
 		)
 	)
-	(label "VALVE6_VSENSE_DIV_N"
+	(label "VBUS_VSENSE_DIV_N"
 		(at 110.49 257.81 0)
 		(effects
@@
 		)
 	)
-	(label "VALVE6_VSENSE_FILT_P"
+	(label "VBUS_VSENSE_FILT_P"
 		(at 209.55 157.48 0)
 		(effects
@@
 		)
 	)
-	(label "VALVE5_VSENSE_DIV_N"
+	(label "IGN_VSENSE_DIV_N"
 		(at 110.49 217.17 0)
 		(effects
@@
 		)
 	)
-	(label "VALVE5_VSENSE_DIV_P"
+	(label "IGN_VSENSE_DIV_P"
 		(at 110.49 201.93 0)
 		(effects
@@
 		)
 	)
-	(label "VALVE6_VSENSE_FILT_N"
+	(label "VBUS_VSENSE_FILT_N"
 		(at 209.55 160.02 0)
 		(effects
@@
 			)
 			(justify right bottom)
-		)
-	)
-	(global_label "VALVE6_VSENSE_P"
-		(shape input)
-		(at 71.12 242.57 180)
-		(fields_autoplaced yes)
-		(effects
-			(font
-				(size 1.27 1.27)
-			)
-			(justify right)
-		)
-		(property "Intersheetrefs" "${INTERSHEET_REFS}"
-			(at 51.1411 242.57 0)
-			(hide yes)
-			(show_name no)
-			(do_not_autoplace no)
-			(effects
-				(font
-					(size 1.27 1.27)
-				)
-				(justify right)
-			)
 		)
 	)
@@
 		)
 	)
+	(global_label "VBUS_VSENSE_N"
+		(shape input)
+		(at 71.12 257.81 180)
+		(fields_autoplaced yes)
+		(effects
+			(font
+				(size 1.27 1.27)
+			)
+			(justify right)
+		)
+		(property "Intersheetrefs" "${INTERSHEET_REFS}"
+			(at 52.8344 257.81 0)
+			(hide yes)
+			(show_name no)
+			(do_not_autoplace no)
+			(effects
+				(font
+					(size 1.27 1.27)
+				)
+				(justify right)
+			)
+		)
+	)
 	(global_label "VALVE1_VSENSE_N"
 		(shape input)
@@
 		)
 	)
-	(global_label "VALVE5_VSENSE_N"
+	(global_label "IGN_VSENSE_P"
 		(shape input)
-		(at 71.12 217.17 180)
+		(at 71.12 201.93 180)
 		(fields_autoplaced yes)
 		(effects
@@
 		)
 		(property "Intersheetrefs" "${INTERSHEET_REFS}"
-			(at 51.0806 217.17 0)
+			(at 54.5882 201.93 0)
 			(hide yes)
 			(show_name no)
@@
 		)
 	)
-	(global_label "VALVE6_VSENSE_N"
-		(shape input)
-		(at 71.12 257.81 180)
-		(fields_autoplaced yes)
-		(effects
-			(font
-				(size 1.27 1.27)
-			)
-			(justify right)
-		)
-		(property "Intersheetrefs" "${INTERSHEET_REFS}"
-			(at 51.0806 257.81 0)
-			(hide yes)
-			(show_name no)
-			(do_not_autoplace no)
-			(effects
-				(font
-					(size 1.27 1.27)
-				)
-				(justify right)
-			)
-		)
-	)
 	(global_label "VALVE2_VSENSE_N"
 		(shape input)
@@
 		)
 	)
+	(global_label "IGN_VSENSE_N"
+		(shape input)
+		(at 71.12 217.17 180)
+		(fields_autoplaced yes)
+		(effects
+			(font
+				(size 1.27 1.27)
+			)
+			(justify right)
+		)
+		(property "Intersheetrefs" "${INTERSHEET_REFS}"
+			(at 54.5277 217.17 0)
+			(hide yes)
+			(show_name no)
+			(do_not_autoplace no)
+			(effects
+				(font
+					(size 1.27 1.27)
+				)
+				(justify right)
+			)
+		)
+	)
 	(global_label "VALVE2_VSENSE_P"
 		(shape input)
@@
 		)
 	)
-	(global_label "VALVE5_VSENSE_P"
+	(global_label "VBUS_VSENSE_P"
 		(shape input)
-		(at 71.12 201.93 180)
+		(at 71.12 242.57 180)
 		(fields_autoplaced yes)
 		(effects
@@
 		)
 		(property "Intersheetrefs" "${INTERSHEET_REFS}"
-			(at 51.1411 201.93 0)
+			(at 52.8949 242.57 0)
 			(hide yes)
 			(show_name no)

Commit message: Major changes
Other:
- moved on the sheet: R216, R217, R219, R220
Changed lines of the file:
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@@
 	(title_block
 		(title "ADC")
-		(date "2026-10-07")
+		(date "2026-10-08")
 		(rev "A")
 	)
@@
 	)
 	(junction
-		(at 100.33 257.81)
+		(at 99.06 257.81)
 		(diameter 0)
 		(color 0 0 0 0)
@@
 	)
 	(junction
-		(at 100.33 242.57)
+		(at 99.06 242.57)
 		(diameter 0)
 		(color 0 0 0 0)
@@
 	(wire
 		(pts
-			(xy 71.12 242.57) (xy 88.9 242.57)
+			(xy 71.12 242.57) (xy 87.63 242.57)
 		)
 		(stroke
@@
 	(wire
 		(pts
-			(xy 100.33 257.81) (xy 140.97 257.81)
+			(xy 99.06 257.81) (xy 140.97 257.81)
 		)
 		(stroke
@@
 	(wire
 		(pts
-			(xy 100.33 251.46) (xy 100.33 252.73)
+			(xy 99.06 251.46) (xy 99.06 252.73)
 		)
 		(stroke
@@
 	(wire
 		(pts
-			(xy 100.33 266.7) (xy 100.33 267.97)
+			(xy 99.06 266.7) (xy 99.06 267.97)
 		)
 		(stroke
@@
 	(wire
 		(pts
-			(xy 100.33 261.62) (xy 100.33 257.81)
+			(xy 99.06 261.62) (xy 99.06 257.81)
 		)
 		(stroke
@@
 	(wire
 		(pts
-			(xy 71.12 257.81) (xy 88.9 257.81)
+			(xy 71.12 257.81) (xy 87.63 257.81)
 		)
 		(stroke
@@
 	(wire
 		(pts
-			(xy 93.98 257.81) (xy 100.33 257.81)
+			(xy 92.71 257.81) (xy 99.06 257.81)
 		)
 		(stroke
@@
 	(wire
 		(pts
-			(xy 100.33 246.38) (xy 100.33 242.57)
+			(xy 99.06 246.38) (xy 99.06 242.57)
 		)
 		(stroke
@@
 	(wire
 		(pts
-			(xy 100.33 242.57) (xy 140.97 242.57)
+			(xy 99.06 242.57) (xy 140.97 242.57)
 		)
 		(stroke
@@
 	(wire
 		(pts
-			(xy 93.98 242.57) (xy 100.33 242.57)
+			(xy 92.71 242.57) (xy 99.06 242.57)
 		)
 		(stroke
@@
 	)
 	(label "VBUS_VSENSE_DIV_P"
-		(at 110.49 242.57 0)
+		(at 109.22 242.57 0)
 		(effects
 			(font
@@
 	)
 	(label "VBUS_VSENSE_DIV_N"
-		(at 110.49 257.81 0)
+		(at 109.22 257.81 0)
 		(effects
 			(font
@@
 	(symbol
 		(lib_id "Device:R_Small_US")
-		(at 100.33 264.16 180)
+		(at 99.06 264.16 180)
 		(unit 1)
 		(body_style 1)
@@
 		(dnp no)
 		(property "Reference" "R220"
-			(at 101.6 261.112 0)
+			(at 100.33 261.112 0)
 			(show_name no)
 			(do_not_autoplace no)
@@
 		)
 		(property "Value" "90.9k"
-			(at 101.6 262.89 0)
+			(at 100.33 262.89 0)
 			(show_name no)
 			(do_not_autoplace no)
@@
 		)
 		(property "Footprint" "valve_pcb_footprints:R_0402_1005Metric_GSE"
-			(at 100.33 264.16 0)
+			(at 99.06 264.16 0)
 			(hide yes)
 			(show_name no)
@@
 		)
 		(property "Datasheet" ""
-			(at 100.33 264.16 0)
+			(at 99.06 264.16 0)
 			(hide yes)
 			(show_name no)
@@
 		)
 		(property "Description" "90.9k 0.1% 0402 Resistor"
-			(at 100.33 264.16 0)
+			(at 99.06 264.16 0)
 			(hide yes)
 			(show_name no)
@@
 		)
 		(property "Tolerance" "0.1%"
-			(at 103.886 264.668 0)
+			(at 102.616 264.668 0)
 			(show_name no)
 			(do_not_autoplace no)
@@
 		)
 		(property "JLCPCB Part #" "C852949"
-			(at 100.33 264.16 0)
+			(at 99.06 264.16 0)
 			(hide yes)
 			(show_name no)
@@
 		)
 		(property "Footprint_Size" "0402"
-			(at 104.14 266.446 0)
+			(at 102.87 266.446 0)
 			(show_name no)
 			(do_not_autoplace no)
@@
 	(symbol
 		(lib_id "power:GND")
-		(at 100.33 267.97 0)
+		(at 99.06 267.97 0)
 		(mirror y)
 		(unit 1)
@@
 		(fields_autoplaced yes)
 		(property "Reference" "#PWR0315"
-			(at 100.33 274.32 0)
+			(at 99.06 274.32 0)
 			(hide yes)
 			(show_name no)
@@
 		)
 		(property "Value" "GND"
-			(at 100.33 273.05 0)
+			(at 99.06 273.05 0)
 			(hide yes)
 			(show_name no)
@@
 		)
 		(property "Footprint" ""
-			(at 100.33 267.97 0)
+			(at 99.06 267.97 0)
 			(hide yes)
 			(show_name no)
@@
 		)
 		(property "Datasheet" ""
-			(at 100.33 267.97 0)
+			(at 99.06 267.97 0)
 			(hide yes)
 			(show_name no)
@@
 		)
 		(property "Description" "Power symbol creates a global label with name \"GND\" , ground"
-			(at 100.33 267.97 0)
+			(at 99.06 267.97 0)
 			(hide yes)
 			(show_name no)
@@
 	(symbol
 		(lib_id "Device:R_Small_US")
-		(at 91.44 257.81 270)
+		(at 90.17 257.81 270)
 		(unit 1)
 		(body_style 1)
@@
 		(dnp no)
 		(property "Reference" "R219"
-			(at 90.17 256.286 90)
+			(at 88.9 256.286 90)
 			(show_name no)
 			(do_not_autoplace no)
@@
 		)
 		(property "Value" "15k"
-			(at 96.52 256.286 90)
+			(at 95.25 256.286 90)
 			(show_name no)
 			(do_not_autoplace no)
@@
 		)
 		(property "Footprint" "valve_pcb_footprints:R_0402_1005Metric_GSE"
-			(at 91.44 257.81 0)
+			(at 90.17 257.81 0)
 			(hide yes)
 			(show_name no)
@@
 		)
 		(property "Datasheet" ""
-			(at 91.44 257.81 0)
+			(at 90.17 257.81 0)
 			(hide yes)
 			(show_name no)
@@
 		)
 		(property "Description" "10k 0.1% 0402 Resistor"
-			(at 91.44 257.81 0)
+			(at 90.17 257.81 0)
 			(hide yes)
 			(show_name no)
@@
 		)
 		(property "Tolerance" "0.1%"
-			(at 88.646 259.334 90)
+			(at 87.376 259.334 90)
 			(show_name no)
 			(do_not_autoplace no)
@@
 		)
 		(property "JLCPCB Part #" "C190095"
-			(at 91.44 257.81 0)
+			(at 90.17 257.81 0)
 			(hide yes)
 			(show_name no)
@@
 		)
 		(property "Footprint_Size" "0402"
-			(at 95.25 259.334 90)
+			(at 93.98 259.334 90)
 			(show_name no)
 			(do_not_autoplace no)
@@
 	(symbol
 		(lib_id "Device:R_Small_US")
-		(at 91.44 242.57 270)
+		(at 90.17 242.57 270)
 		(unit 1)
 		(body_style 1)
@@
 		(dnp no)
 		(property "Reference" "R216"
-			(at 90.17 241.046 90)
+			(at 88.9 241.046 90)
 			(show_name no)
 			(do_not_autoplace no)
@@
 		)
 		(property "Value" "15k"
-			(at 96.52 241.046 90)
+			(at 95.25 241.046 90)
 			(show_name no)
 			(do_not_autoplace no)
@@
 		)
 		(property "Footprint" "valve_pcb_footprints:R_0402_1005Metric_GSE"
-			(at 91.44 242.57 0)
+			(at 90.17 242.57 0)
 			(hide yes)
 			(show_name no)
@@
 		)
 		(property "Datasheet" ""
-			(at 91.44 242.57 0)
+			(at 90.17 242.57 0)
 			(hide yes)
 			(show_name no)
@@
 		)
 		(property "Description" "10k 0.1% 0402 Resistor"
-			(at 91.44 242.57 0)
+			(at 90.17 242.57 0)
 			(hide yes)
 			(show_name no)
@@
 		)
 		(property "Tolerance" "0.1%"
-			(at 88.646 244.094 90)
+			(at 87.376 244.094 90)
 			(show_name no)
 			(do_not_autoplace no)
@@
 		)
 		(property "JLCPCB Part #" "C190095"
-			(at 91.44 242.57 0)
+			(at 90.17 242.57 0)
 			(hide yes)
 			(show_name no)
@@
 		)
 		(property "Footprint_Size" "0402"
-			(at 95.25 244.094 90)
+			(at 93.98 244.094 90)
 			(show_name no)
 			(do_not_autoplace no)
@@
 	(symbol
 		(lib_id "Device:R_Small_US")
-		(at 100.33 248.92 180)
+		(at 99.06 248.92 180)
 		(unit 1)
 		(body_style 1)
@@
 		(dnp no)
 		(property "Reference" "R217"
-			(at 101.6 245.872 0)
+			(at 100.33 245.872 0)
 			(show_name no)
 			(do_not_autoplace no)
@@
 		)
 		(property "Value" "90.9k"
-			(at 101.6 247.65 0)
+			(at 100.33 247.65 0)
 			(show_name no)
 			(do_not_autoplace no)
@@
 		)
 		(property "Footprint" "valve_pcb_footprints:R_0402_1005Metric_GSE"
-			(at 100.33 248.92 0)
+			(at 99.06 248.92 0)
 			(hide yes)
 			(show_name no)
@@
 		)
 		(property "Datasheet" ""
-			(at 100.33 248.92 0)
+			(at 99.06 248.92 0)
 			(hide yes)
 			(show_name no)
@@
 		)
 		(property "Description" "90.9k 0.1% 0402 Resistor"
-			(at 100.33 248.92 0)
+			(at 99.06 248.92 0)
 			(hide yes)
 			(show_name no)
@@
 		)
 		(property "Tolerance" "0.1%"
-			(at 103.886 249.428 0)
+			(at 102.616 249.428 0)
 			(show_name no)
 			(do_not_autoplace no)
@@
 		)
 		(property "JLCPCB Part #" "C852949"
-			(at 100.33 248.92 0)
+			(at 99.06 248.92 0)
 			(hide yes)
 			(show_name no)
@@
 		)
 		(property "Footprint_Size" "0402"
-			(at 104.14 251.206 0)
+			(at 102.87 251.206 0)
 			(show_name no)
 			(do_not_autoplace no)
@@
 	(symbol
 		(lib_id "power:GND")
-		(at 100.33 252.73 0)
+		(at 99.06 252.73 0)
 		(mirror y)
 		(unit 1)
@@
 		(fields_autoplaced yes)
 		(property "Reference" "#PWR0314"
-			(at 100.33 259.08 0)
+			(at 99.06 259.08 0)
 			(hide yes)
 			(show_name no)
@@
 		)
 		(property "Value" "GND"
-			(at 100.33 257.81 0)
+			(at 99.06 257.81 0)
 			(hide yes)
 			(show_name no)
@@
 		)
 		(property "Footprint" ""
-			(at 100.33 252.73 0)
+			(at 99.06 252.73 0)
 			(hide yes)
 			(show_name no)
@@
 		)
 		(property "Datasheet" ""
-			(at 100.33 252.73 0)
+			(at 99.06 252.73 0)
 			(hide yes)
 			(show_name no)
@@
 		)
 		(property "Description" "Power symbol creates a global label with name \"GND\" , ground"
-			(at 100.33 252.73 0)
+			(at 99.06 252.73 0)
 			(hide yes)
 			(show_name no)

Commit message: Fixes
Added hops, fixed the planes, and fixed minor issues
Parts:
- renumbered C105 to C75, C106 to C76, C112 to C77, C113 to C78, C114 to C79, C115 to C80, C116 to C81, C117 to C82, C118 to C83, C119 to C84, C103 to C85, C104 to C86, C78 to C87, C102 to C88, C120 to C89, R210 to R136, R213 to R137, R216 to R138, R219 to R139, R186 to R140, R187 to R141, R192 to R142, R195 to R143, R198 to R144, R201 to R145, R204 to R146, R207 to R147, R211 to R148, R214 to R149, R217 to R150, R220 to R151, R188 to R152, R189 to R153, R193 to R154, R196 to R155, R199 to R156, R202 to R157, R205 to R158, R208 to R159, R194 to R160, R197 to R161, R200 to R162, R203 to R163, R206 to R164, R209 to R165, R212 to R166, R215 to R167, R218 to R168, R221 to R169, R190 to R170, R191 to R171, R222 to R172, R231 to R173, R230 to R174, R229 to R175, R228 to R176, R232 to R177, R233 to R178, R234 to R179, TP224 to TP110, TP225 to TP111, TP226 to TP112, TP227 to TP113, TP223 to TP114, TP159 to TP115, U10 to U17
