File: LRUs/Valve Control Unit/Electrical/Valve Power Board/valve_control_pcb/fans.kicad_sch (KiCad schematic)
At the start: 14 parts, among them J25 B2B-XH-A, J26 B2B-XH-A, Q19 AO3400A, Q20 AO3400A

Commit message: Committttt
Other:
- note added: "FANS"
- moved on the sheet: C25, C77, D39, D40, J25, J26, Q19, Q20, R137, R182, R183, R184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

Commit message: Commit da changes
Parts:
- C25, C77: footprint Capacitor_SMD:C_1206_3216Metric -> valve_pcb_footprints:C_1206_3216Metric
- R137, R182, R183, R184, R185, R87: footprint Resistor_SMD:R_0603_1608Metric -> valve_pcb_footprints:R_0603_1608Metric
Other:
- note added: "20"

Commit message: Fixes
Added hops, fixed the planes, and fixed minor issues
Parts:
- renumbered C77 to C133, C25 to C134, D39 to D43, D40 to D44, J25 to J18, J26 to J19, R182 to R221, R183 to R222, R184 to R223, R185 to R224, R87 to R225, R137 to R226
Changed lines of the file:
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@@
 		(in_pos_files yes)
 		(dnp no)
-		(property "Reference" "J26"
+		(property "Reference" "J19"
 			(at 197.612 102.87 0)
 			(show_name no)
@@
 			(project "valve_control_pcb"
 				(path "/b2606128-8980-4101-9648-1808c1b96e2b"
-					(reference "J26")
+					(reference "J19")
 					(unit 1)
 					(variant
@@
 		(dnp no)
 		(fields_autoplaced yes)
-		(property "Reference" "#PWR0368"
+		(property "Reference" "#PWR0305"
 			(at 172.72 58.42 0)
 			(hide yes)
@@
 			(project "valve_control_pcb"
 				(path "/b2606128-8980-4101-9648-1808c1b96e2b"
-					(reference "#PWR0368")
+					(reference "#PWR0305")
 					(unit 1)
 				)
@@
 		(in_pos_files yes)
 		(dnp no)
-		(property "Reference" "C25"
+		(property "Reference" "C134"
 			(at 175.768 107.442 0)
 			(show_name no)
@@
 			(project "valve_control_pcb"
 				(path "/b2606128-8980-4101-9648-1808c1b96e2b"
-					(reference "C25")
+					(reference "C134")
 					(unit 1)
 					(variant
@@
 		(dnp no)
 		(fields_autoplaced yes)
-		(property "Reference" "#PWR0370"
+		(property "Reference" "#PWR0307"
 			(at 173.99 120.65 0)
 			(hide yes)
@@
 			(project "valve_control_pcb"
 				(path "/b2606128-8980-4101-9648-1808c1b96e2b"
-					(reference "#PWR0370")
+					(reference "#PWR0307")
 					(unit 1)
 				)
@@
 		(in_pos_files yes)
 		(dnp no)
-		(property "Reference" "C77"
+		(property "Reference" "C133"
 			(at 174.498 45.212 0)
 			(show_name no)
@@
 			(project "valve_control_pcb"
 				(path "/b2606128-8980-4101-9648-1808c1b96e2b"
-					(reference "C77")
+					(reference "C133")
 					(unit 1)
 					(variant
@@
 		(in_pos_files yes)
 		(dnp no)
-		(property "Reference" "R184"
+		(property "Reference" "R223"
 			(at 154.432 60.96 90)
 			(show_name no)
@@
 			(project "valve_control_pcb"
 				(path "/b2606128-8980-4101-9648-1808c1b96e2b"
-					(reference "R184")
+					(reference "R223")
 					(unit 1)
 					(variant
@@
 		(dnp no)
 		(fields_autoplaced yes)
-		(property "Reference" "#PWR0366"
+		(property "Reference" "#PWR0303"
 			(at 143.51 153.67 0)
 			(hide yes)
@@
 			(project "valve_control_pcb"
 				(path "/b2606128-8980-4101-9648-1808c1b96e2b"
-					(reference "#PWR0366")
+					(reference "#PWR0303")
 					(unit 1)
 				)
@@
 		(in_pos_files yes)
 		(dnp no)
-		(property "Reference" "R183"
+		(property "Reference" "R222"
 			(at 147.32 129.54 0)
 			(show_name no)
@@
 			(project "valve_control_pcb"
 				(path "/b2606128-8980-4101-9648-1808c1b96e2b"
-					(reference "R183")
+					(reference "R222")
 					(unit 1)
 					(variant
@@
 		(dnp no)
 		(fields_autoplaced yes)
-		(property "Reference" "#PWR0365"
+		(property "Reference" "#PWR0302"
 			(at 139.7 91.44 0)
 			(hide yes)
@@
 			(project "valve_control_pcb"
 				(path "/b2606128-8980-4101-9648-1808c1b96e2b"
-					(reference "#PWR0365")
+					(reference "#PWR0302")
 					(unit 1)
 				)
@@
 		(dnp no)
 		(fields_autoplaced yes)
-		(property "Reference" "#PWR0371"
+		(property "Reference" "#PWR0308"
 			(at 184.15 91.44 0)
 			(hide yes)
@@
 			(project "valve_control_pcb"
 				(path "/b2606128-8980-4101-9648-1808c1b96e2b"
-					(reference "#PWR0371")
+					(reference "#PWR0308")
 					(unit 1)
 				)
@@
 		(in_pos_files yes)
 		(dnp no)
-		(property "Reference" "R137"
+		(property "Reference" "R226"
 			(at 173.736 127.762 0)
 			(show_name no)
@@
 			(project "valve_control_pcb"
 				(path "/b2606128-8980-4101-9648-1808c1b96e2b"
-					(reference "R137")
+					(reference "R226")
 					(unit 1)
 					(variant
@@
 		(in_pos_files yes)
 		(dnp no)
-		(property "Reference" "D40"
+		(property "Reference" "D44"
 			(at 146.05 139.192 90)
 			(show_name no)
@@
 			(project "valve_control_pcb"
 				(path "/b2606128-8980-4101-9648-1808c1b96e2b"
-					(reference "D40")
+					(reference "D44")
 					(unit 1)
 					(variant
@@
 		(dnp no)
 		(fields_autoplaced yes)
-		(property "Reference" "#PWR0369"
+		(property "Reference" "#PWR0306"
 			(at 173.99 106.68 0)
 			(hide yes)
@@
 			(project "valve_control_pcb"
 				(path "/b2606128-8980-4101-9648-1808c1b96e2b"
-					(reference "#PWR0369")
+					(reference "#PWR0306")
 					(unit 1)
 				)
@@
 		(dnp no)
 		(fields_autoplaced yes)
-		(property "Reference" "#PWR0367"
+		(property "Reference" "#PWR0304"
 			(at 172.72 44.45 0)
 			(hide yes)
@@
 			(project "valve_control_pcb"
 				(path "/b2606128-8980-4101-9648-1808c1b96e2b"
-					(reference "#PWR0367")
+					(reference "#PWR0304")
 					(unit 1)
 				)
@@
 		(in_pos_files yes)
 		(dnp no)
-		(property "Reference" "R185"
+		(property "Reference" "R224"
 			(at 154.432 123.19 90)
 			(show_name no)
@@
 			(project "valve_control_pcb"
 				(path "/b2606128-8980-4101-9648-1808c1b96e2b"
-					(reference "R185")
+					(reference "R224")
 					(unit 1)
 					(variant
@@
 		(dnp no)
 		(fields_autoplaced yes)
-		(property "Reference" "#PWR0372"
+		(property "Reference" "#PWR0309"
 			(at 184.15 153.67 0)
 			(hide yes)
@@
 			(project "valve_control_pcb"
 				(path "/b2606128-8980-4101-9648-1808c1b96e2b"
-					(reference "#PWR0372")
+					(reference "#PWR0309")
 					(unit 1)
 				)
@@
 		(in_pos_files yes)
 		(dnp no)
-		(property "Reference" "J25"
+		(property "Reference" "J18"
 			(at 197.612 40.64 0)
 			(show_name no)
@@
 			(project "valve_control_pcb"
 				(path "/b2606128-8980-4101-9648-1808c1b96e2b"
-					(reference "J25")
+					(reference "J18")
 					(unit 1)
 					(variant
@@
 		(in_pos_files yes)
 		(dnp no)
-		(property "Reference" "R182"
+		(property "Reference" "R221"
 			(at 143.51 67.31 0)
 			(show_name no)
@@
 			(project "valve_control_pcb"
 				(path "/b2606128-8980-4101-9648-1808c1b96e2b"
-					(reference "R182")
+					(reference "R221")
 					(unit 1)
 					(variant
@@
 		(in_pos_files yes)
 		(dnp no)
-		(property "Reference" "D39"
+		(property "Reference" "D43"
 			(at 142.24 76.962 90)
 			(show_name no)
@@
 			(project "valve_control_pcb"
 				(path "/b2606128-8980-4101-9648-1808c1b96e2b"
-					(reference "D39")
+					(reference "D43")
 					(unit 1)
 					(variant
@@
 		(in_pos_files yes)
 		(dnp no)
-		(property "Reference" "R87"
+		(property "Reference" "R225"
 			(at 173.736 65.532 0)
 			(show_name no)
@@
 			(project "valve_control_pcb"
 				(path "/b2606128-8980-4101-9648-1808c1b96e2b"
-					(reference "R87")
+					(reference "R225")
 					(unit 1)
 					(variant
