File: LRUs/Valve Control Unit/Electrical/Valve Power Board/valve_control_pcb/rs-485.kicad_sch (KiCad schematic)
At the start: 28 parts, among them J12 Conn_01x04, U22 74LVC1G17, U23 SN6505BDBV, U24 ISO1450BDWR, U25 AMS1117-5.0

Commit message: Committttt
Parts:
- U24: footprint footprints:SOIC127P1030X265-16N -> valve_pcb_footprints:SOIC127P1030X265-16N
Changed lines of the file:
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@@
 			)
 		)
-		(property "Footprint" "footprints:SOIC127P1030X265-16N"
+		(property "Footprint" "valve_pcb_footprints:SOIC127P1030X265-16N"
 			(at 135.89 137.16 0)
 			(hide yes)
@@
 				)
 				(justify bottom)
+			)
+		)
+		(property "JLCPCB Part #" ""
+			(at 135.89 137.16 0)
+			(hide yes)
+			(show_name no)
+			(do_not_autoplace no)
+			(effects
+				(font
+					(size 1.27 1.27)
+				)
+			)
+		)
+		(property "Footprint_Size" ""
+			(at 135.89 137.16 0)
+			(show_name no)
+			(do_not_autoplace no)
+			(effects
+				(font
+					(size 1.27 1.27)
+				)
 			)
 		)
@@
 	(sheet_instances
 		(path "/"
-			(page "16")
+			(page "17")
 		)
 	)

Commit message: Commit da changes
Parts:
- C108, C75, C79, C80, C81: footprint Capacitor_SMD:C_0805_2012Metric -> valve_pcb_footprints:C_0805_2012Metric
- C51, C54: footprint Capacitor_SMD:C_0402_1005Metric -> valve_pcb_footprints:C_0402_1005Metric
- D30, D31: value MBR0520LT -> MBR0520LT1G
- J12: value Conn_01x04 -> 0436500415; footprint Connector_Molex:Molex_Micro-Fit_3.0_43650-0415_1x04_P3.00mm_Vertical -> valve_pcb_footprints:Molex_Micro-Fit_3.0_43650-0415_1x04_P3.00mm_Vertical; Footprint_Size (none) -> 3mm
- R129: footprint Resistor_SMD:R_0603_1608Metric -> valve_pcb_footprints:R_0603_1608Metric
- R130, R131, R133: footprint Resistor_SMD:R_0402_1005Metric -> valve_pcb_footprints:R_0402_1005Metric_GSE
- TP100, TP101, TP96, TP97, TP98, TP99: footprint TestPoint:TestPoint_Pad_D2.0mm -> TestPoint:TestPoint_Pad_D1.0mm
- TR1: footprint Transformer_SMD:Transformer_Wuerth_750315371 -> valve_pcb_footprints:Transformer_Wuerth_750315371
- U23: value SN6505BDBV -> SN6505BDBVR
Connections:
- net 5V_ISO: now reaches C80.1, D30.1 (K), D31.1 (K), R132.2, TP100.1, U25.3 (VI)
- net 5V_ISO_FILT: now reaches C51.1, C79.1, C81.1, R132.1, TP101.1, U24.16 (VCC2), U25.2 (VO)
- net B1: now reaches D30.2 (A), TP98.1, TR1.4
- net A2: now reaches TP97.1, TR1.1, U23.3 (D2)
- net A1: now reaches TP96.1, TR1.3, U23.1 (D1)
- net B2: now reaches D31.2 (A), TP99.1, TR1.6
Other:
- note added: "20"
- moved on the sheet: C51, C79, D30, D31, D32, J12, JP1, R130, R131, R133, TP96, TP97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

Commit message: Small updates
Parts:
- removed R129: 10k, valve_pcb_footprints:R_0603_1608Metric, symbol Device:R_Small_US
- removed U22: 74LVC1G17, Package_TO_SOT_SMD:SOT-23-5_HandSoldering, symbol 74xGxx:74LVC1G17
Connections:
- net +3V3: now also C54.1, C75.1, U24.1 (VCC1)
- net +5V: no longer C54.1, C75.1, U24.1 (VCC1)
- net MAIN_RX: now also U24.3 (R)
Other:
- note removed: "3.3V level shift"
- moved on the sheet: C54, C75

Commit message: Fixes
Added hops, fixed the planes, and fixed minor issues
Parts:
- renumbered C75 to C120, C54 to C121, C108 to C122, C51 to C123, C79 to C124, C80 to C125, C81 to C126, D30 to D40, D31 to D41, D32 to D42, J12 to J17, R130 to R209, R131 to R210, R132 to R211, R133 to R212, TP96 to TP141, TP97 to TP142, TP98 to TP143, TP99 to TP144, TP100 to TP145, TP101 to TP146, U23 to U22, U24 to U23, U25 to U24
