File: LRUs/Valve Control Unit/Electrical/Valve Power Board/valve_control_pcb/sd_card.kicad_sch (KiCad schematic)
At the start: 12 parts, among them J16 Micro_SD_Card_Det2, U32 TPD6E05U06RVZ

Commit message: Commit valve board updates
Parts:
- added TP199: TestPoint, TestPoint:TestPoint_Pad_D2.0mm, symbol Connector:TestPoint
- R169: Footprint_Size (none) -> 0603
Connections:
- net +3V3_SD renamed +3V3
- net +3V3: now also TP199.1
Other:
- note added: "SD CARD"
- title: (none) -> SD CARD
Changed lines of the file:
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@@
 	(generator_version "10.0")
 	(paper "A4")
-	(text_box "Add 22 Ohm resistors on \nMOSI, CLK, and CS near MCU\n"
+	(title_block
+		(title "SD CARD")
+		(date "2026-08-27")
+		(rev "A")
+	)
+	(text "SD CARD"
 		(exclude_from_sim no)
-		(at 135.382 74.422 0)
-		(size 31.75 6.35)
-		(margins 0.9525 0.9525 0.9525 0.9525)
-		(stroke
-			(width 0)
-			(type solid)
-		)
-		(fill
-			(type none)
-		)
+		(at 161.798 29.21 0)
 		(effects
 			(font
-				(size 1.27 1.27)
-			)
-			(justify left top)
+				(size 7.62 7.62)
+				(thickness 1.016)
+				(bold yes)
+				(color 0 0 0 1)
+			)
 		)
 	)
@@
 	(junction
 		(at 162.56 54.61)
+		(diameter 0)
+		(color 0 0 0 0)
+	)
+	(junction
+		(at 175.26 54.61)
 		(diameter 0)
 		(color 0 0 0 0)
@@
 		(dnp no)
 		(property "Reference" "R169"
-			(at 178.054 69.85 0)
+			(at 179.07 70.104 0)
 			(show_name no)
 			(do_not_autoplace no)
@@
 		)
 		(property "Value" "10k"
-			(at 178.562 72.39 0)
+			(at 178.308 71.882 0)
 			(show_name no)
 			(do_not_autoplace no)
@@
 		)
 		(property "Tolerance" "1%"
-			(at 177.546 74.676 0)
+			(at 178.054 73.66 0)
 			(show_name no)
 			(do_not_autoplace no)
@@
 			(at 175.26 72.39 0)
 			(hide yes)
+			(show_name no)
+			(do_not_autoplace no)
+			(effects
+				(font
+					(size 1.27 1.27)
+				)
+			)
+		)
+		(property "Footprint_Size" "0603"
+			(at 179.07 75.438 0)
 			(show_name no)
 			(do_not_autoplace no)
@@
 				(path "/4518b036-acbb-4d4f-82dd-00ce25d5ff09"
 					(reference "R167")
+					(unit 1)
+					(variant
+						(name "My VARIANT DARNIT")
+					)
+				)
+			)
+		)
+	)
+	(symbol
+		(lib_id "Connector:TestPoint")
+		(at 175.26 54.61 270)
+		(unit 1)
+		(body_style 1)
+		(exclude_from_sim no)
+		(in_bom yes)
+		(on_board yes)
+		(in_pos_files yes)
+		(dnp no)
+		(property "Reference" "TP199"
+			(at 182.88 54.61 90)
+			(show_name no)
+			(do_not_autoplace no)
+			(effects
+				(font
+					(size 1.27 1.27)
+				)
+			)
+		)
+		(property "Value" "TestPoint"
+			(at 184.404 54.61 90)
+			(hide yes)
+			(show_name no)
+			(do_not_autoplace no)
+			(effects
+				(font
+					(size 1.27 1.27)
+				)
+			)
+		)
+		(property "Footprint" "TestPoint:TestPoint_Pad_D2.0mm"
+			(at 175.26 59.69 0)
+			(hide yes)
+			(show_name no)
+			(do_not_autoplace no)
+			(effects
+				(font
+					(size 1.27 1.27)
+				)
+			)
+		)
+		(property "Datasheet" ""
+			(at 175.26 59.69 0)
+			(hide yes)
+			(show_name no)
+			(do_not_autoplace no)
+			(effects
+				(font
+					(size 1.27 1.27)
+				)
+			)
+		)
+		(property "Description" "test point"
+			(at 175.26 54.61 0)
+			(hide yes)
+			(show_name no)
+			(do_not_autoplace no)
+			(effects
+				(font
+					(size 1.27 1.27)
+				)
+			)
+		)
+		(property "Vf" ""
+			(at 175.26 54.61 0)
+			(show_name no)
+			(do_not_autoplace no)
+			(effects
+				(font
+					(size 1.27 1.27)
+				)
+			)
+		)
+		(property "Vz" ""
+			(at 175.26 54.61 0)
+			(show_name no)
+			(do_not_autoplace no)
+			(effects
+				(font
+					(size 1.27 1.27)
+				)
+			)
+		)
+		(property "JLCPCB Part #" "TP10"
+			(at 175.26 54.61 90)
+			(hide yes)
+			(show_name no)
+			(do_not_autoplace no)
+			(effects
+				(font
+					(size 1.27 1.27)
+				)
+			)
+		)
+		(property "VDS" "TestPoint"
+			(at 175.26 54.61 90)
+			(hide yes)
+			(show_name no)
+			(do_not_autoplace no)
+			(effects
+				(font
+					(size 1.27 1.27)
+				)
+			)
+		)
+		(pin "1"
+		)
+		(instances
+			(project "valve_control_pcb"
+				(path "/4518b036-acbb-4d4f-82dd-00ce25d5ff09"
+					(reference "TP199")
 					(unit 1)
 					(variant
@@
 		(in_pos_files yes)
 		(dnp no)
-		(fields_autoplaced yes)
 		(property "Reference" "#PWR0269"
 			(at 189.23 88.9 0)
@@
 			)
 		)
-		(property "Value" "+3V3_SD"
-			(at 189.23 80.01 0)
+		(property "Value" "+3V3"
+			(at 188.722 80.518 0)
 			(show_name no)
 			(do_not_autoplace no)
@@
 			(at 189.23 85.09 0)
 			(hide yes)
+			(show_name no)
+			(do_not_autoplace no)
+			(effects
+				(font
+					(size 1.27 1.27)
+				)
+			)
+		)
+		(property "Footprint_Size" ""
+			(at 189.23 85.09 0)
 			(show_name no)
 			(do_not_autoplace no)
@@
 		(in_pos_files yes)
 		(dnp no)
-		(fields_autoplaced yes)
 		(property "Reference" "#PWR0266"
 			(at 152.4 54.61 0)
@@
 			)
 		)
-		(property "Value" "+3V3_SD"
-			(at 152.4 45.72 0)
+		(property "Value" "+3V3"
+			(at 151.892 46.228 0)
 			(show_name no)
 			(do_not_autoplace no)
@@
 			(at 152.4 50.8 0)
 			(hide yes)
+			(show_name no)
+			(do_not_autoplace no)
+			(effects
+				(font
+					(size 1.27 1.27)
+				)
+			)
+		)
+		(property "Footprint_Size" ""
+			(at 152.4 50.8 0)
 			(show_name no)
 			(do_not_autoplace no)
@@
 	(sheet_instances
 		(path "/"
-			(page "23")
-		)
-	)
+			(page "14")
+		)
+	)

Commit message: Commit da changes
Parts:
- C107: footprint Capacitor_SMD:C_0805_2012Metric -> valve_pcb_footprints:C_0805_2012Metric
- C110: footprint Capacitor_SMD:C_0402_1005Metric -> valve_pcb_footprints:C_0402_1005Metric
- J16: JLCPCB Part # J5 -> C114218
- R165, R166, R167, R168, R169, R170, R171, R173: footprint Resistor_SMD:R_0603_1608Metric -> valve_pcb_footprints:R_0603_1608Metric
- TP199: footprint TestPoint:TestPoint_Pad_D2.0mm -> TestPoint:TestPoint_Pad_D1.0mm
- U32: Footprint_Size (none) -> USON-14; VR (none) -> 5.5V
Other:
- note added: "20"
Changed lines of the file:
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@@
 		(rev "A")
+	)
+	(text "20"
+		(exclude_from_sim no)
+		(at 29.21 85.344 0)
+		(effects
+			(font
+				(size 1.27 1.27)
+				(color 113 103 4 1)
+			)
+		)
 	)
 	(text "SD CARD"
@@
 			)
 		)
-		(property "Footprint" "Resistor_SMD:R_0603_1608Metric"
+		(property "Footprint" "valve_pcb_footprints:R_0603_1608Metric"
 			(at 134.62 87.63 0)
 			(hide yes)
@@
 			)
 		)
-		(property "Footprint" "Capacitor_SMD:C_0402_1005Metric"
+		(property "Footprint" "valve_pcb_footprints:C_0402_1005Metric"
 			(at 162.56 62.23 0)
 			(hide yes)
@@
 		(property "Footprint_Size" "0402"
 			(at 167.386 64.77 0)
+			(show_name no)
+			(do_not_autoplace no)
+			(effects
+				(font
+					(size 1.27 1.27)
+				)
+			)
+		)
+		(property "MPN" ""
+			(at 162.56 62.23 0)
+			(hide yes)
 			(show_name no)
 			(do_not_autoplace no)
@@
 			)
 		)
-		(property "Footprint" "Resistor_SMD:R_0603_1608Metric"
+		(property "Footprint" "valve_pcb_footprints:R_0603_1608Metric"
 			(at 175.26 72.39 0)
 			(hide yes)
@@
 			)
 		)
-		(property "Footprint" "Resistor_SMD:R_0603_1608Metric"
+		(property "Footprint" "valve_pcb_footprints:R_0603_1608Metric"
 			(at 116.84 92.71 0)
 			(hide yes)
@@
 			)
 		)
-		(property "Footprint" "TestPoint:TestPoint_Pad_D2.0mm"
+		(property "Footprint" "TestPoint:TestPoint_Pad_D1.0mm"
 			(at 175.26 59.69 0)
 			(hide yes)
@@
 			)
 		)
-		(property "JLCPCB Part #" "J5"
+		(property "JLCPCB Part #" "C114218"
 			(at 222.25 97.79 0)
 			(hide yes)
@@
 			(at 222.25 97.79 0)
 			(hide yes)
+			(show_name no)
+			(do_not_autoplace no)
+			(effects
+				(font
+					(size 1.27 1.27)
+				)
+			)
+		)
+		(property "Footprint_Size" ""
+			(at 222.25 97.79 0)
 			(show_name no)
 			(do_not_autoplace no)
@@
 			)
 		)
-		(property "Footprint" "Resistor_SMD:R_0603_1608Metric"
+		(property "Footprint" "valve_pcb_footprints:R_0603_1608Metric"
 			(at 116.84 102.87 0)
 			(hide yes)
@@
 			)
 		)
-		(property "Footprint" "Resistor_SMD:R_0603_1608Metric"
+		(property "Footprint" "valve_pcb_footprints:R_0603_1608Metric"
 			(at 125.73 90.17 0)
 			(hide yes)
@@
 			)
 		)
-		(property "Footprint" "Resistor_SMD:R_0603_1608Metric"
+		(property "Footprint" "valve_pcb_footprints:R_0603_1608Metric"
 			(at 107.95 105.41 0)
 			(hide yes)
@@
 			)
 		)
-		(property "Footprint" "Capacitor_SMD:C_0805_2012Metric"
+		(property "Footprint" "valve_pcb_footprints:C_0805_2012Metric"
 			(at 152.4 62.23 0)
 			(hide yes)
@@
 			)
 		)
-		(property "Footprint" "Resistor_SMD:R_0603_1608Metric"
+		(property "Footprint" "valve_pcb_footprints:R_0603_1608Metric"
 			(at 116.84 97.79 0)
 			(hide yes)
@@
 		(in_pos_files yes)
 		(dnp no)
-		(fields_autoplaced yes)
 		(property "Reference" "U32"
-			(at 140.97 129.5399 0)
+			(at 141.478 127.2539 0)
 			(show_name no)
 			(do_not_autoplace no)
@@
 		)
 		(property "Value" "TPD6E05U06RVZ"
-			(at 140.97 132.0799 0)
+			(at 141.478 129.7939 0)
 			(show_name no)
 			(do_not_autoplace no)
@@
 			(at 157.48 130.81 0)
 			(hide yes)
+			(show_name no)
+			(do_not_autoplace no)
+			(effects
+				(font
+					(size 1.27 1.27)
+				)
+			)
+		)
+		(property "Footprint_Size" "USON-14"
+			(at 136.652 134.112 0)
+			(show_name no)
+			(do_not_autoplace no)
+			(effects
+				(font
+					(size 1.27 1.27)
+				)
+			)
+		)
+		(property "VR" "5.5V"
+			(at 139.192 132.08 0)
 			(show_name no)
 			(do_not_autoplace no)
@@
 			)
 		)
-		(property "Footprint" "Resistor_SMD:R_0603_1608Metric"
+		(property "Footprint" "valve_pcb_footprints:R_0603_1608Metric"
 			(at 99.06 107.95 0)
 			(hide yes)
@@
 	(sheet_instances
 		(path "/"
-			(page "15")
-		)
-	)
+			(page "21")
+		)
+	)

Commit message: Fixes
Added hops, fixed the planes, and fixed minor issues
Parts:
- renumbered C107 to C114, C110 to C115, J16 to J15, R168 to R196, R170 to R197, R167 to R198, R173 to R199, R171 to R200, R166 to R201, R165 to R202, R169 to R203, TP199 to TP134, U32 to U20
Changed lines of the file:
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@@
 		(in_pos_files yes)
 		(dnp no)
-		(property "Reference" "R165"
+		(property "Reference" "R202"
 			(at 133.096 86.614 90)
 			(show_name no)
@@
 			(project "valve_control_pcb"
 				(path "/4518b036-acbb-4d4f-82dd-00ce25d5ff09"
-					(reference "R165")
+					(reference "R202")
 					(unit 1)
 					(variant
@@
 		(dnp no)
 		(fields_autoplaced yes)
-		(property "Reference" "#PWR0271"
+		(property "Reference" "#PWR0230"
 			(at 196.85 119.38 0)
 			(hide yes)
@@
 			(project "valve_control_pcb"
 				(path "/4518b036-acbb-4d4f-82dd-00ce25d5ff09"
-					(reference "#PWR0271")
+					(reference "#PWR0230")
 					(unit 1)
 				)
@@
 		(in_pos_files yes)
 		(dnp no)
-		(property "Reference" "C110"
+		(property "Reference" "C115"
 			(at 164.592 58.674 0)
 			(show_name no)
@@
 			(project "valve_control_pcb"
 				(path "/4518b036-acbb-4d4f-82dd-00ce25d5ff09"
-					(reference "C110")
+					(reference "C115")
 					(unit 1)
 					(variant
@@
 		(in_pos_files yes)
 		(dnp no)
-		(property "Reference" "R169"
+		(property "Reference" "R203"
 			(at 179.07 70.104 0)
 			(show_name no)
@@
 			(project "valve_control_pcb"
 				(path "/4518b036-acbb-4d4f-82dd-00ce25d5ff09"
-					(reference "R169")
+					(reference "R203")
 					(unit 1)
 					(variant
@@
 		(dnp no)
 		(fields_autoplaced yes)
-		(property "Reference" "#PWR0268"
+		(property "Reference" "#PWR0226"
 			(at 152.4 73.66 0)
 			(hide yes)
@@
 			(project "valve_control_pcb"
 				(path "/4518b036-acbb-4d4f-82dd-00ce25d5ff09"
-					(reference "#PWR0268")
+					(reference "#PWR0226")
 					(unit 1)
 				)
@@
 		(in_pos_files yes)
 		(dnp no)
-		(property "Reference" "R167"
+		(property "Reference" "R198"
 			(at 115.316 91.694 90)
 			(show_name no)
@@
 			(project "valve_control_pcb"
 				(path "/4518b036-acbb-4d4f-82dd-00ce25d5ff09"
-					(reference "R167")
+					(reference "R198")
 					(unit 1)
 					(variant
@@
 		(in_pos_files yes)
 		(dnp no)
-		(property "Reference" "TP199"
+		(property "Reference" "TP134"
 			(at 182.88 54.61 90)
 			(show_name no)
@@
 			(project "valve_control_pcb"
 				(path "/4518b036-acbb-4d4f-82dd-00ce25d5ff09"
-					(reference "TP199")
+					(reference "TP134")
 					(unit 1)
 					(variant
@@
 		(in_pos_files yes)
 		(dnp no)
-		(property "Reference" "J16"
+		(property "Reference" "J15"
 			(at 204.724 79.756 0)
 			(show_name no)
@@
 			(project "valve_control_pcb"
 				(path "/4518b036-acbb-4d4f-82dd-00ce25d5ff09"
-					(reference "J16")
+					(reference "J15")
 					(unit 1)
 					(variant
@@
 		(dnp no)
 		(fields_autoplaced yes)
-		(property "Reference" "#PWR0273"
+		(property "Reference" "#PWR0231"
 			(at 245.11 119.38 0)
 			(hide yes)
@@
 			(project "valve_control_pcb"
 				(path "/4518b036-acbb-4d4f-82dd-00ce25d5ff09"
-					(reference "#PWR0273")
+					(reference "#PWR0231")
 					(unit 1)
 				)
@@
 		(in_pos_files yes)
 		(dnp no)
-		(property "Reference" "R171"
+		(property "Reference" "R200"
 			(at 115.316 101.854 90)
 			(show_name no)
@@
 			(project "valve_control_pcb"
 				(path "/4518b036-acbb-4d4f-82dd-00ce25d5ff09"
-					(reference "R171")
+					(reference "R200")
 					(unit 1)
 					(variant
@@
 		(in_pos_files yes)
 		(dnp no)
-		(property "Reference" "#PWR0269"
+		(property "Reference" "#PWR0229"
 			(at 196.85 88.9 0)
 			(hide yes)
@@
 			(project "valve_control_pcb"
 				(path "/4518b036-acbb-4d4f-82dd-00ce25d5ff09"
-					(reference "#PWR0269")
+					(reference "#PWR0229")
 					(unit 1)
 				)
@@
 		(in_pos_files yes)
 		(dnp no)
-		(property "Reference" "R166"
+		(property "Reference" "R201"
 			(at 124.206 89.154 90)
 			(show_name no)
@@
 			(project "valve_control_pcb"
 				(path "/4518b036-acbb-4d4f-82dd-00ce25d5ff09"
-					(reference "R166")
+					(reference "R201")
 					(unit 1)
 					(variant
@@
 		(in_pos_files yes)
 		(dnp no)
-		(property "Reference" "R170"
+		(property "Reference" "R197"
 			(at 106.426 104.394 90)
 			(show_name no)
@@
 			(project "valve_control_pcb"
 				(path "/4518b036-acbb-4d4f-82dd-00ce25d5ff09"
-					(reference "R170")
+					(reference "R197")
 					(unit 1)
 					(variant
@@
 		(in_pos_files yes)
 		(dnp no)
-		(property "Reference" "C107"
+		(property "Reference" "C114"
 			(at 154.686 58.674 0)
 			(show_name no)
@@
 			(project "valve_control_pcb"
 				(path "/4518b036-acbb-4d4f-82dd-00ce25d5ff09"
-					(reference "C107")
+					(reference "C114")
 					(unit 1)
 					(variant
@@
 		(dnp no)
 		(fields_autoplaced yes)
-		(property "Reference" "#PWR0272"
+		(property "Reference" "#PWR0227"
 			(at 162.56 73.66 0)
 			(hide yes)
@@
 			(project "valve_control_pcb"
 				(path "/4518b036-acbb-4d4f-82dd-00ce25d5ff09"
-					(reference "#PWR0272")
+					(reference "#PWR0227")
 					(unit 1)
 				)
@@
 		(in_pos_files yes)
 		(dnp no)
-		(property "Reference" "#PWR0266"
+		(property "Reference" "#PWR0225"
 			(at 152.4 54.61 0)
 			(hide yes)
@@
 			(project "valve_control_pcb"
 				(path "/4518b036-acbb-4d4f-82dd-00ce25d5ff09"
-					(reference "#PWR0266")
+					(reference "#PWR0225")
 					(unit 1)
 				)
@@
 		(dnp no)
 		(fields_autoplaced yes)
-		(property "Reference" "#PWR0267"
+		(property "Reference" "#PWR0228"
 			(at 181.61 138.43 0)
 			(hide yes)
@@
 			(project "valve_control_pcb"
 				(path "/4518b036-acbb-4d4f-82dd-00ce25d5ff09"
-					(reference "#PWR0267")
+					(reference "#PWR0228")
 					(unit 1)
 				)
@@
 		(in_pos_files yes)
 		(dnp no)
-		(property "Reference" "R173"
+		(property "Reference" "R199"
 			(at 112.522 96.774 90)
 			(show_name no)
@@
 			(project "valve_control_pcb"
 				(path "/4518b036-acbb-4d4f-82dd-00ce25d5ff09"
-					(reference "R173")
+					(reference "R199")
 					(unit 1)
 					(variant
@@
 		(in_pos_files yes)
 		(dnp no)
-		(property "Reference" "U32"
+		(property "Reference" "U20"
 			(at 141.478 127.2539 0)
 			(show_name no)
@@
 			(project "valve_control_pcb"
 				(path "/4518b036-acbb-4d4f-82dd-00ce25d5ff09"
-					(reference "U32")
+					(reference "U20")
 					(unit 1)
 					(variant
@@
 		(in_pos_files yes)
 		(dnp no)
-		(property "Reference" "R168"
+		(property "Reference" "R196"
 			(at 97.536 106.934 90)
 			(show_name no)
@@
 			(project "valve_control_pcb"
 				(path "/4518b036-acbb-4d4f-82dd-00ce25d5ff09"
-					(reference "R168")
+					(reference "R196")
 					(unit 1)
 					(variant
