File: LRUs/Valve Control Unit/Electrical/Valve Power Board/valve_control_pcb/sensors.kicad_sch (KiCad schematic)
At the start: 2 parts

Commit message: Commit valve board updates
Parts:
- added TP173, TP174: TestPoint, TestPoint:TestPoint_Pad_D2.0mm, symbol Connector:TestPoint
Connections:
- net I2C1_SCL: now also TP174.1
- net I2C1_SDA: now also TP173.1
Other:
- note added: "TEMPERATURE SENSORS"
- title: (none) -> SENSORS

Commit message: Commit da changes
Parts:
- R85, R86: footprint Resistor_SMD:R_0603_1608Metric -> valve_pcb_footprints:R_0603_1608Metric
- TP173, TP174: footprint TestPoint:TestPoint_Pad_D2.0mm -> TestPoint:TestPoint_Pad_D1.0mm
Other:
- note added: "20"
- moved on the sheet: R85, R86, TP173, TP174

Commit message: Fixes
Added hops, fixed the planes, and fixed minor issues
Parts:
- renumbered R85 to R213, R86 to R214, TP173 to TP147, TP174 to TP148
Changed lines of the file:
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@@
 		(in_pos_files yes)
 		(dnp no)
-		(property "Reference" "#PWR083"
+		(property "Reference" "#PWR0273"
 			(at 163.83 104.14 0)
 			(hide yes)
@@
 			(project "valve_control_pcb"
 				(path "/8089a923-bb92-49be-ae97-55220516cf62"
-					(reference "#PWR083")
+					(reference "#PWR0273")
 					(unit 1)
 				)
@@
 		(in_pos_files yes)
 		(dnp no)
-		(property "Reference" "TP173"
+		(property "Reference" "TP147"
 			(at 30.48 26.67 90)
 			(show_name no)
@@
 			(project "valve_control_pcb"
 				(path "/8089a923-bb92-49be-ae97-55220516cf62"
-					(reference "TP173")
+					(reference "TP147")
 					(unit 1)
 					(variant
@@
 		(dnp no)
 		(fields_autoplaced yes)
-		(property "Reference" "#PWR076"
+		(property "Reference" "#PWR0266"
 			(at 165.1 67.31 0)
 			(hide yes)
@@
 			(project "valve_control_pcb"
 				(path "/8089a923-bb92-49be-ae97-55220516cf62"
-					(reference "#PWR076")
+					(reference "#PWR0266")
 					(unit 1)
 				)
@@
 		(in_pos_files yes)
 		(dnp no)
-		(property "Reference" "R86"
+		(property "Reference" "R214"
 			(at 82.55 22.352 0)
 			(show_name no)
@@
 			(project "valve_control_pcb"
 				(path "/8089a923-bb92-49be-ae97-55220516cf62"
-					(reference "R86")
+					(reference "R214")
 					(unit 1)
 					(variant
@@
 		(dnp no)
 		(fields_autoplaced yes)
-		(property "Reference" "#PWR075"
+		(property "Reference" "#PWR0265"
 			(at 165.1 43.18 0)
 			(hide yes)
@@
 			(project "valve_control_pcb"
 				(path "/8089a923-bb92-49be-ae97-55220516cf62"
-					(reference "#PWR075")
+					(reference "#PWR0265")
 					(unit 1)
 				)
@@
 		(in_pos_files yes)
 		(dnp no)
-		(property "Reference" "#PWR085"
+		(property "Reference" "#PWR0275"
 			(at 163.83 134.62 0)
 			(hide yes)
@@
 			(project "valve_control_pcb"
 				(path "/8089a923-bb92-49be-ae97-55220516cf62"
-					(reference "#PWR085")
+					(reference "#PWR0275")
 					(unit 1)
 				)
@@
 		(in_pos_files yes)
 		(dnp no)
-		(property "Reference" "#PWR074"
+		(property "Reference" "#PWR0264"
 			(at 81.28 24.13 0)
 			(hide yes)
@@
 			(project "valve_control_pcb"
 				(path "/8089a923-bb92-49be-ae97-55220516cf62"
-					(reference "#PWR074")
+					(reference "#PWR0264")
 					(unit 1)
 				)
@@
 		(in_pos_files yes)
 		(dnp no)
-		(property "Reference" "#PWR084"
+		(property "Reference" "#PWR0274"
 			(at 163.83 106.68 0)
 			(hide yes)
@@
 			(project "valve_control_pcb"
 				(path "/8089a923-bb92-49be-ae97-55220516cf62"
-					(reference "#PWR084")
+					(reference "#PWR0274")
 					(unit 1)
 				)
@@
 		(in_pos_files yes)
 		(dnp no)
-		(property "Reference" "#PWR073"
+		(property "Reference" "#PWR0263"
 			(at 72.39 24.13 0)
 			(hide yes)
@@
 			(project "valve_control_pcb"
 				(path "/8089a923-bb92-49be-ae97-55220516cf62"
-					(reference "#PWR073")
+					(reference "#PWR0263")
 					(unit 1)
 				)
@@
 		(in_pos_files yes)
 		(dnp no)
-		(property "Reference" "#PWR082"
+		(property "Reference" "#PWR0272"
 			(at 163.83 81.28 0)
 			(hide yes)
@@
 			(project "valve_control_pcb"
 				(path "/8089a923-bb92-49be-ae97-55220516cf62"
-					(reference "#PWR082")
+					(reference "#PWR0272")
 					(unit 1)
 				)
@@
 		(in_pos_files yes)
 		(dnp no)
-		(property "Reference" "#PWR081"
+		(property "Reference" "#PWR0271"
 			(at 163.83 54.61 0)
 			(hide yes)
@@
 			(project "valve_control_pcb"
 				(path "/8089a923-bb92-49be-ae97-55220516cf62"
-					(reference "#PWR081")
+					(reference "#PWR0271")
 					(unit 1)
 				)
@@
 		(in_pos_files yes)
 		(dnp no)
-		(property "Reference" "TP174"
+		(property "Reference" "TP148"
 			(at 30.48 36.83 90)
 			(show_name no)
@@
 			(project "valve_control_pcb"
 				(path "/8089a923-bb92-49be-ae97-55220516cf62"
-					(reference "TP174")
+					(reference "TP148")
 					(unit 1)
 					(variant
@@
 		(dnp no)
 		(fields_autoplaced yes)
-		(property "Reference" "#PWR077"
+		(property "Reference" "#PWR0267"
 			(at 166.37 91.44 0)
 			(hide yes)
@@
 			(project "valve_control_pcb"
 				(path "/8089a923-bb92-49be-ae97-55220516cf62"
-					(reference "#PWR077")
+					(reference "#PWR0267")
 					(unit 1)
 				)
@@
 		(in_pos_files yes)
 		(dnp no)
-		(property "Reference" "#PWR086"
+		(property "Reference" "#PWR0276"
 			(at 163.83 154.94 0)
 			(hide yes)
@@
 			(project "valve_control_pcb"
 				(path "/8089a923-bb92-49be-ae97-55220516cf62"
-					(reference "#PWR086")
+					(reference "#PWR0276")
 					(unit 1)
 				)
@@
 		(dnp no)
 		(fields_autoplaced yes)
-		(property "Reference" "#PWR078"
+		(property "Reference" "#PWR0268"
 			(at 166.37 116.84 0)
 			(hide yes)
@@
 			(project "valve_control_pcb"
 				(path "/8089a923-bb92-49be-ae97-55220516cf62"
-					(reference "#PWR078")
+					(reference "#PWR0268")
 					(unit 1)
 				)
@@
 		(in_pos_files yes)
 		(dnp no)
-		(property "Reference" "#PWR087"
+		(property "Reference" "#PWR0277"
 			(at 163.83 160.02 0)
 			(hide yes)
@@
 			(project "valve_control_pcb"
 				(path "/8089a923-bb92-49be-ae97-55220516cf62"
-					(reference "#PWR087")
+					(reference "#PWR0277")
 					(unit 1)
 				)
@@
 		(in_pos_files yes)
 		(dnp no)
-		(property "Reference" "R85"
+		(property "Reference" "R213"
 			(at 73.66 22.352 0)
 			(show_name no)
@@
 			(project "valve_control_pcb"
 				(path "/8089a923-bb92-49be-ae97-55220516cf62"
-					(reference "R85")
+					(reference "R213")
 					(unit 1)
 					(variant
@@
 		(dnp no)
 		(fields_autoplaced yes)
-		(property "Reference" "#PWR079"
+		(property "Reference" "#PWR0269"
 			(at 166.37 143.51 0)
 			(hide yes)
@@
 			(project "valve_control_pcb"
 				(path "/8089a923-bb92-49be-ae97-55220516cf62"
-					(reference "#PWR079")
+					(reference "#PWR0269")
 					(unit 1)
 				)
@@
 		(dnp no)
 		(fields_autoplaced yes)
-		(property "Reference" "#PWR080"
+		(property "Reference" "#PWR0270"
 			(at 166.37 168.91 0)
 			(hide yes)
@@
 			(project "valve_control_pcb"
 				(path "/8089a923-bb92-49be-ae97-55220516cf62"
-					(reference "#PWR080")
-					(unit 1)
-				)
+					(reference "#PWR0270")
+					(unit 1)
+				)
