File: LRUs/Valve Control Unit/Electrical/Valve Power Board/valve_control_pcb/top-level.kicad_sch (KiCad schematic)
At the start: 0 parts

Commit message: Fixes
Added hops, fixed the planes, and fixed minor issues
Changed lines of the file:
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@@
 		)
 	)
-	(text_box "RESPONSIBLE ENGINEER: \nNICHOLAS ALVES\n\nREVIEWERS:"
+	(text_box "RESPONSIBLE ENGINEER: \nNICHOLAS ALVES\n\nREVIEWERS:\nETHAN EGGERT\nMAX LEIBOWITZ"
 		(exclude_from_sim no)
-		(at 176.53 124.46 0)
-		(size 46.99 14.1705)
+		(at 176.53 113.03 0)
+		(size 46.99 20.3044)
 		(margins 0.9525 0.9525 0.9525 0.9525)
 		(stroke
