File: LRUs/Valve Control Unit/Electrical/Valve Power Board/valve_control_pcb/usb-c.kicad_sch (KiCad schematic)
At the start: 20 parts, among them J15 GSB1C41110SSHR, U31 AMS1117-3.3

Commit message: Commit valve board updates
Parts:
- removed C102, C105, C106: 10uF, Capacitor_SMD:C_0805_2012Metric, symbol Device:C_Small_US
- removed C103, C104: 1uF, Capacitor_SMD:C_0805_2012Metric, symbol Device:C_Small_US
- added C109, C111: 10uF, Capacitor_SMD:C_0805_2012Metric, symbol Device:C_Small_US
- added C55, C56: 1uF, Capacitor_SMD:C_0805_2012Metric, symbol Device:C_Small_US
- added TP193, TP194, TP195, TP196, TP197, TP198: TestPoint, TestPoint:TestPoint_Pad_D2.0mm, symbol Connector:TestPoint
- D33, D34, D35, D36, D37: Footprint_Size (none) -> X2SON2
- D38, R159, R160, R161, R162, R163, R164: Footprint_Size (none) -> 0603
Connections:
- net 3V3_USB: now also C109.1, C55.1
- net D_N: now also TP196.1
- net D_P: now also TP197.1
- net GND: now also C109.2, C111.2, C55.2, C56.2
- net USB_VBUS_DET: now also TP195.1
- net at D36.1 (K), J15.B5 (CC2), R161.1: now also TP194.1
- net at D34.1 (K), J15.A5 (CC1), R162.1: now also TP193.1
- net VBUS renamed V5P0_USB
- net V5P0_USB: now also C111.1, C56.1, TP198.1
Other:
- note added: "USB-C"
- moved on the sheet: D33, D38, R161, R164

Commit message: Committttt
Parts:
- D33, D34, D35, D36, D37: footprint footprints:X2SON2_DPL_TEX -> valve_pcb_footprints:X2SON2_DPL_TEX
- J15: footprint footprints:AMPHENOL_GSB1C41110SSHR -> valve_pcb_footprints:AMPHENOL_GSB1C41110SSHR
Changed lines of the file:
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@@
 			)
 		)
-		(property "Footprint" "footprints:AMPHENOL_GSB1C41110SSHR"
+		(property "Footprint" "valve_pcb_footprints:AMPHENOL_GSB1C41110SSHR"
 			(at 63.5 133.35 0)
 			(hide yes)
@@
 			)
 		)
+		(property "Footprint_Size" ""
+			(at 53.34 105.41 0)
+			(show_name no)
+			(do_not_autoplace no)
+			(effects
+				(font
+					(size 1.27 1.27)
+				)
+			)
+		)
 		(pin "SH3"
 		)
@@
 			)
 		)
-		(property "Footprint" "footprints:X2SON2_DPL_TEX"
+		(property "Footprint" "valve_pcb_footprints:X2SON2_DPL_TEX"
 			(at 101.6 144.78 0)
 			(hide yes)
@@
 			)
 		)
-		(property "Footprint" "footprints:X2SON2_DPL_TEX"
+		(property "Footprint" "valve_pcb_footprints:X2SON2_DPL_TEX"
 			(at 96.52 95.25 0)
 			(hide yes)
@@
 			)
 		)
-		(property "Footprint" "footprints:X2SON2_DPL_TEX"
+		(property "Footprint" "valve_pcb_footprints:X2SON2_DPL_TEX"
 			(at 83.82 95.25 0)
 			(hide yes)
@@
 			)
 		)
-		(property "Footprint" "footprints:X2SON2_DPL_TEX"
+		(property "Footprint" "valve_pcb_footprints:X2SON2_DPL_TEX"
 			(at 88.9 144.78 0)
 			(hide yes)
@@
 			)
 		)
-		(property "Footprint" "footprints:X2SON2_DPL_TEX"
+		(property "Footprint" "valve_pcb_footprints:X2SON2_DPL_TEX"
 			(at 143.51 86.36 0)
 			(hide yes)
@@
 	(sheet_instances
 		(path "/"
-			(page "15")
+			(page "16")
 		)
 	)

Commit message: Commit da changes
Parts:
- removed D38: WHITE, LED_SMD:LED_0603_1608Metric, symbol Device:LED
- removed R159, R160: 2.2k, Resistor_SMD:R_0603_1608Metric, symbol Device:R_Small_US
- added D44: GREEN, LED_SMD:LED_0805_2012Metric, symbol Device:LED
- added R243: 2k, valve_pcb_footprints:R_0603_1608Metric, symbol Device:R_Small_US
- C109, C111, C55, C56: footprint Capacitor_SMD:C_0805_2012Metric -> valve_pcb_footprints:C_0805_2012Metric
- J15: JLCPCB Part # (none) -> C34260841
- R161, R162, R163, R164: footprint Resistor_SMD:R_0603_1608Metric -> valve_pcb_footprints:R_0603_1608Metric
- TP193, TP194, TP195, TP196, TP197, TP198: footprint TestPoint:TestPoint_Pad_D2.0mm -> TestPoint:TestPoint_Pad_D1.0mm
Connections:
- net GND: now also D44.1 (K)
- net V5P0_USB: now also R243.2
- new net: D44.2 (A), R243.1
Other:
- note added: "20"
- note added: "3"
- moved on the sheet: TP195, TP196, TP197

Commit message: Small updates
Parts:
- D44: value GREEN -> WHITE; footprint LED_SMD:LED_0805_2012Metric -> LED_SMD:LED_0603_1608Metric; Footprint_Size 0805 -> 0603; JLCPCB Part # C2297 -> C2290
Changed lines of the file:
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@@
 	)
 	(junction
-		(at 73.66 100.33)
+		(at 73.66 102.87)
 		(diameter 0)
 		(color 0 0 0 0)
@@
 	)
 	(junction
+		(at 73.66 97.79)
+		(diameter 0)
+		(color 0 0 0 0)
+	)
+	(junction
 		(at 246.38 134.62)
 		(diameter 0)
@@
 	)
 	(junction
-		(at 73.66 105.41)
-		(diameter 0)
-		(color 0 0 0 0)
-	)
-	(junction
 		(at 227.33 78.74)
 		(diameter 0)
@@
 	(wire
 		(pts
+			(xy 73.66 97.79) (xy 73.66 100.33)
+		)
+		(stroke
+			(width 0)
+			(type default)
+		)
+	)
+	(wire
+		(pts
 			(xy 72.39 123.19) (xy 72.39 125.73)
 		)
@@
 	(wire
 		(pts
-			(xy 80.01 132.08) (xy 80.01 100.33)
+			(xy 80.01 132.08) (xy 80.01 97.79)
 		)
 		(stroke
@@
 	(wire
 		(pts
-			(xy 77.47 105.41) (xy 77.47 134.62)
+			(xy 77.47 102.87) (xy 77.47 134.62)
 		)
 		(stroke
@@
 	(wire
 		(pts
-			(xy 73.66 97.79) (xy 73.66 100.33)
-		)
-		(stroke
-			(width 0)
-			(type default)
-		)
-	)
-	(wire
-		(pts
 			(xy 31.75 125.73) (xy 35.56 125.73)
 		)
@@
 	(wire
 		(pts
-			(xy 80.01 100.33) (xy 73.66 100.33)
+			(xy 80.01 97.79) (xy 73.66 97.79)
 		)
 		(stroke
@@
 	(wire
 		(pts
-			(xy 73.66 105.41) (xy 77.47 105.41)
+			(xy 73.66 102.87) (xy 77.47 102.87)
 		)
 		(stroke
@@
 	)
 	(symbol
-		(lib_id "Device:LED")
-		(at 158.75 95.25 90)
-		(unit 1)
-		(body_style 1)
-		(exclude_from_sim no)
-		(in_bom yes)
-		(on_board yes)
-		(in_pos_files yes)
-		(dnp no)
-		(property "Reference" "D44"
-			(at 161.29 93.472 90)
-			(show_name no)
-			(do_not_autoplace no)
-			(effects
-				(font
-					(size 1.27 1.27)
-				)
-				(justify right)
-			)
-		)
-		(property "Value" "GREEN"
-			(at 161.29 95.25 90)
-			(show_name no)
-			(do_not_autoplace no)
-			(effects
-				(font
-					(size 1.27 1.27)
-				)
-				(justify right)
-			)
-		)
-		(property "Footprint" "LED_SMD:LED_0805_2012Metric"
-			(at 158.75 95.25 0)
-			(hide yes)
-			(show_name no)
-			(do_not_autoplace no)
-			(effects
-				(font
-					(size 1.27 1.27)
-				)
-			)
-		)
-		(property "Datasheet" ""
-			(at 158.75 95.25 0)
-			(hide yes)
-			(show_name no)
-			(do_not_autoplace no)
-			(effects
-				(font
-					(size 1.27 1.27)
-				)
-			)
-		)
-		(property "Description" "KT-0603R Red LED"
-			(at 158.75 95.25 0)
-			(hide yes)
-			(show_name no)
-			(do_not_autoplace no)
-			(effects
-				(font
-					(size 1.27 1.27)
-				)
-			)
-		)
-		(property "Sim.Pins" "1=K 2=A"
-			(at 158.75 95.25 0)
-			(hide yes)
-			(show_name no)
-			(do_not_autoplace no)
-			(effects
-				(font
-					(size 1.27 1.27)
-				)
-			)
-		)
-		(property "Vf" "3.1V"
-			(at 163.576 97.028 90)
-			(show_name no)
-			(do_not_autoplace no)
-			(effects
-				(font
-					(size 1.27 1.27)
-				)
-			)
-		)
-		(property "JLCPCB Part #" "C2297"
-			(at 158.75 95.25 90)
-			(hide yes)
-			(show_name no)
-			(do_not_autoplace no)
-			(effects
-				(font
-					(size 1.27 1.27)
-				)
-			)
-		)
-		(property "Footprint_Size" "0805"
-			(at 163.83 98.806 90)
-			(show_name no)
-			(do_not_autoplace no)
-			(effects
-				(font
-					(size 1.27 1.27)
-				)
-			)
-		)
-		(pin "1"
-		)
-		(pin "2"
-		)
-		(instances
-			(project "valve_control_pcb"
-				(path "/f86a0e95-9fb7-4edc-ad4b-275b6a59a091"
-					(reference "D44")
-					(unit 1)
-					(variant
-						(name "My VARIANT DARNIT")
-					)
-				)
-			)
-		)
-	)
-	(symbol
 		(lib_id "symbols:GSB1C41110SSHR")
 		(at 53.34 105.41 0)
@@
 					)
 				)
+			)
+		)
+	)
+	(symbol
+		(lib_id "Device:LED")
+		(at 158.75 95.25 90)
+		(unit 1)
+		(body_style 1)
+		(exclude_from_sim no)
+		(in_bom yes)
+		(on_board yes)
+		(in_pos_files yes)
+		(dnp no)
+		(property "Reference" "D44"
+			(at 161.544 92.456 90)
+			(show_name no)
+			(do_not_autoplace no)
+			(effects
+				(font
+					(size 1.27 1.27)
+				)
+				(justify right)
+			)
+		)
+		(property "Value" "WHITE"
+			(at 161.544 94.234 90)
+			(show_name no)
+			(do_not_autoplace no)
+			(effects
+				(font
+					(size 1.27 1.27)
+				)
+				(justify right)
+			)
+		)
+		(property "Footprint" "LED_SMD:LED_0603_1608Metric"
+			(at 158.75 95.25 0)
+			(hide yes)
+			(show_name no)
+			(do_not_autoplace no)
+			(effects
+				(font
+					(size 1.27 1.27)
+				)
+			)
+		)
+		(property "Datasheet" ""
+			(at 158.75 95.25 0)
+			(hide yes)
+			(show_name no)
+			(do_not_autoplace no)
+			(effects
+				(font
+					(size 1.27 1.27)
+				)
+			)
+		)
+		(property "Description" "KT-0603R Red LED"
+			(at 158.75 95.25 0)
+			(hide yes)
+			(show_name no)
+			(do_not_autoplace no)
+			(effects
+				(font
+					(size 1.27 1.27)
+				)
+			)
+		)
+		(property "Sim.Pins" "1=K 2=A"
+			(at 158.75 95.25 0)
+			(hide yes)
+			(show_name no)
+			(do_not_autoplace no)
+			(effects
+				(font
+					(size 1.27 1.27)
+				)
+			)
+		)
+		(property "Vf" "3.1V"
+			(at 163.83 96.012 90)
+			(show_name no)
+			(do_not_autoplace no)
+			(effects
+				(font
+					(size 1.27 1.27)
+				)
+			)
+		)
+		(property "JLCPCB Part #" "C2290"
+			(at 158.75 95.25 90)
+			(hide yes)
+			(show_name no)
+			(do_not_autoplace no)
+			(effects
+				(font
+					(size 1.27 1.27)
+				)
+			)
+		)
+		(property "Footprint_Size" "0603"
+			(at 164.084 98.044 90)
+			(show_name no)
+			(do_not_autoplace no)
+			(effects
+				(font
+					(size 1.27 1.27)
+				)
+			)
+		)
+		(pin "1"
+		)
+		(pin "2"
+		)
+		(instances
+			(project "valve_control_pcb"
+				(path "/f86a0e95-9fb7-4edc-ad4b-275b6a59a091"
+					(reference "D44")
+					(unit 1)
+					(variant
+						(name "My VARIANT DARNIT")
+					)
+				)

Commit message: Fixes
Added hops, fixed the planes, and fixed minor issues
Parts:
- renumbered C111 to C116, C56 to C117, C55 to C118, C109 to C119, D33 to D38, D44 to D39, FB3 to FB2, J15 to J16, R161 to R204, R162 to R205, R243 to R206, R163 to R207, R164 to R208, TP198 to TP135, TP193 to TP136, TP194 to TP137, TP195 to TP138, TP196 to TP139, TP197 to TP140, U31 to U21
Other:
- title: (none) -> USB-C
