File: LRUs/Valve Control Unit/Electrical/Valve Power Board/valve_control_pcb/valve_ctrl.kicad_sch (KiCad schematic)
At the start: 40 parts, among them J1 0436500215, Q1 SiR882ADP, U1 TPS27SA08CPWPR

Commit message: Commit valve board updates
Parts:
- added R186: 0, Resistor_SMD:R_0603_1608Metric, symbol Device:R_Small_US
- added R192, R198: 10k, Resistor_SMD:R_0402_1005Metric, symbol Device:R_Small_US
- added R204, R210: 90.9k, Resistor_SMD:R_0402_1005Metric, symbol Device:R_Small_US
- added TP91, TP92: TestPoint, TestPoint:TestPoint_Pad_D1.0mm, symbol Connector:TestPoint
- added U10: INA821IDRG, Package_SON:WSON-8-1EP_3x3mm_P0.5mm_EP1.45x2.4mm, symbol Amplifier_Instrumentation:INA821xDRG
- J1: value 0436500215 -> 0039299047; footprint Connector_Molex:Molex_Micro-Fit_3.0_43650-0215_1x02_P3.00mm_Vertical -> Connector_Molex:Molex_Mini-Fit_Jr_5566-04A2_2x02_P4.20mm_Vertical; symbol Connector_Generic:Conn_01x02 -> Connector_Generic:Conn_02x02_Counter_Clockwise; Footprint_Size 3.00mm -> 4.2mm; Imax (none) -> 9A
- TP13, TP14: footprint TestPoint:TestPoint_Pad_D2.0mm -> TestPoint:TestPoint_Pad_D1.0mm
Connections:
- net GND: now also R192.2, R198.2, U10.5 (Vs-), U10.6 (Ref), U10.9 (Vs-)
- new net +5V: U10.8 (Vs+)
- new net GAIN1: R186.2, U10.2 (Rg)
- new net GAIN2: R186.1, U10.3 (Rg)
- new net KELVIN_SENSE: U10.7
- new net VSENSE_DIV_N: R192.1, R204.1, U10.1 (-)
- new net VSENSE_DIV_P: R198.1, R210.1, U10.4 (+)
- new net VSENSE_N: J1.4 (Pin_4), R204.2, TP91.1
- new net VSENSE_P: J1.3 (Pin_3), R210.2, TP92.1
Other:
- note added: "20mΩ * 2A = 40mW"
- note added: "VALVE OUTPUT POWER"
- moved on the sheet: C1, C2, C3, C4, D1, D2, D3, D4, Q1, R1, R10, R11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

Commit message: Committttt
Parts:
- removed R186: 0, Resistor_SMD:R_0603_1608Metric, symbol Device:R_Small_US
- removed R192, R198: 10k, Resistor_SMD:R_0402_1005Metric, symbol Device:R_Small_US
- removed R204, R210: 90.9k, Resistor_SMD:R_0402_1005Metric, symbol Device:R_Small_US
- removed U10: INA821IDRG, Package_SON:WSON-8-1EP_3x3mm_P0.5mm_EP1.45x2.4mm, symbol Amplifier_Instrumentation:INA821xDRG
- Q1: Footprint_Size (none) -> SO-8
Other:
- moved on the sheet: TP91, TP92

Commit message: Commit da changes
Parts:
- removed R11: 100, Resistor_SMD:R_0603_1608Metric, symbol Device:R_Small_US
- removed R13: 47k, Resistor_SMD:R_0603_1608Metric, symbol Device:R_Small_US
- removed TP11: TestPoint, TestPoint:TestPoint_Pad_D2.0mm, symbol Connector:TestPoint
- added R121: 10k, valve_pcb_footprints:R_0603_1608Metric, symbol Device:R_Small_US
- added R248: 100, valve_pcb_footprints:R_0603_1608Metric, symbol Device:R_Small_US
- C1: footprint Capacitor_SMD:C_1206_3216Metric -> valve_pcb_footprints:C_1206_3216Metric
- C2: footprint Capacitor_SMD:C_0805_2012Metric -> valve_pcb_footprints:C_0805_2012Metric
- C3: footprint Capacitor_SMD:C_0402_1005Metric -> valve_pcb_footprints:C_0402_1005Metric
- C4: footprint Capacitor_SMD:C_0603_1608Metric -> valve_pcb_footprints:C_0603_1608Metric
- J1: footprint Connector_Molex:Molex_Mini-Fit_Jr_5566-04A2_2x02_P4.20mm_Vertical -> valve_pcb_footprints:Molex_Mini-Fit_Jr_5566-04A2_2x02_P4.20mm_Vertical
- Q1: value SiR882ADP -> SIR5108DP-T1-RE3-HXY; footprint Package_SO:PowerPAK_SO-8_Single -> valve_pcb_footprints:PowerPAK_SO-8_Single; JLCPCB Part # C553986 -> C53262900
- R1, R10, R14, R2, R3, R4, R5, R6, R7, R8, R9: footprint Resistor_SMD:R_0603_1608Metric -> valve_pcb_footprints:R_0603_1608Metric
- R12: footprint Resistor_SMD:R_0402_1005Metric -> valve_pcb_footprints:R_0402_1005Metric_GSE
- TP1, TP10, TP12, TP15, TP2, TP3, TP4, TP5, TP6, TP7, TP8: footprint TestPoint:TestPoint_Pad_D2.0mm -> TestPoint:TestPoint_Pad_D1.0mm
- U1: JLCPCB Part # (none) -> C2864601
Connections:
- net 12V_OUT+: now also J1.4 (Pin_4); no longer J1.1 (Pin_1)
- net 12V_OUT-: now also J1.3 (Pin_3); no longer J1.2 (Pin_2)
- net GND: now also R121.2
- net LFET_GATE: now also R121.1, R248.1
- net VALVE_LSS_EN: now also R248.2
- net VSENSE_N: now also J1.1 (Pin_1); no longer J1.4 (Pin_4)
- net VSENSE_P: now also J1.2 (Pin_2); no longer J1.3 (Pin_3)
Other:
- moved on the sheet: C1, C2, C3, C4, D1, D2, D3, D4, J1, Q1, R1, R10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

Commit message: Small updates
Parts:
- Q1: value SIR5108DP-T1-RE3-HXY -> SIR5108DP
Changed lines of the file:
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@@
 			)
 		)
-		(property "Value" "SIR5108DP-T1-RE3-HXY"
-			(at 237.998 82.804 0)
+		(property "Value" "SIR5108DP"
+			(at 231.14 82.804 0)
 			(show_name no)
 			(do_not_autoplace no)

Commit message: Fixes
Added hops, fixed the planes, and fixed minor issues
Parts:
- removed C2: 220nF, valve_pcb_footprints:C_0805_2012Metric, symbol Device:C_Small_US
- added C45, C46: 100nF, valve_pcb_footprints:C_0402_1005Metric, symbol Device:C_Small_US
- renumbered C1 to C44, C3 to C47, C4 to C48, D1 to D6, D2 to D7, D3 to D8, D4 to D9, J1 to J6, Q1 to Q7, R1 to R54, R2 to R55, R3 to R56, R4 to R57, R5 to R58, R6 to R59, R7 to R60, R8 to R61, R9 to R62, R10 to R63, R248 to R64, R121 to R65, R12 to R66, R14 to R67, TP3 to TP33, TP1 to TP34, TP2 to TP35, TP4 to TP36, TP5 to TP37, TP6 to TP38, TP7 to TP39, TP8 to TP40, TP9 to TP41, TP10 to TP42, TP12 to TP43, TP13 to TP44, TP14 to TP45, TP15 to TP46, TP91 to TP47, TP92 to TP48, U1 to U12
Connections:
- net GND: now also C45.2, C46.2
- net VIN: now also C45.1, C46.1
Other:
- moved on the sheet: C44
