File: LRUs/Valve Control Unit/Electrical/Valve Power Board/valve_control_pcb/connectors.kicad_sch (KiCad schematic)
At the start: 21 parts, among them J7 0768290110, J8 Conn_02x10_Odd_Even, U7 TPD6E05U06RVZ, U8 TPD6E05U06RVZ, U9 PCA9306DC

Commit message: Commit valve board updates
Parts:
- removed C25: 100pF, Capacitor_SMD:C_0402_1005Metric, symbol Device:C_Small_US
- removed R87: 200k, Resistor_SMD:R_0603_1608Metric, symbol Device:R_Small_US
- added C76: 100nF, Capacitor_SMD:C_0402_1005Metric, symbol Device:C_Small_US
- added H12: MountingHole_Pad, MountingHole:MountingHole_3.2mm_M3_ISO14580_Pad, symbol Mechanical:MountingHole_Pad
- added R172: 200k, Resistor_SMD:R_0603_1608Metric, symbol Device:R_Small_US
- added R174, R175, R176, R177, R178, R179, R180, R181: 0, Resistor_SMD:R_0603_1608Metric, symbol Device:R_Small_US
- added TP146, TP162, TP163, TP164, TP165, TP166, TP167, TP168, TP169, TP170, TP171, TP172: TestPoint, TestPoint:TestPoint_Pad_D2.0mm, symbol Connector:TestPoint
- J8: value Conn_02x10_Odd_Even -> IDC-Header_2x10
- R88, R89: Footprint_Size (none) -> 0603
Connections:
- net +3V3: now also C76.1, R172.2
- net GND: now also C76.2, H12.1, TP171.1
- net I2C_SCL: now also TP169.1
- net I2C_SDA: now also TP170.1
- net PIN12: now also R179.2
- net PIN13: now also R176.1
- net PIN16: now also R180.2
- net PIN17: now also R177.1
- net PIN20: now also R181.2
- net PIN5: now also R174.1
- net PIN8: now also R178.2
- net PIN9: now also R175.1
- net at U9.8 (EN): now also R172.1
- net at F1.1, J7.1 (Pin_1), J7.2 (Pin_2)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: now also TP172.1
- new net PIN12_STM32: R179.1, TP166.1
- new net PIN13_STM32: R176.2, TP163.1
- new net PIN16_STM32: R180.1, TP167.1
- new net PIN17_STM32: R177.2, TP164.1
- new net PIN20_STM32: R181.1, TP168.1
- new net PIN5_STM32: R174.2, TP146.1
- new net PIN8_STM32: R178.1, TP165.1
- new net PIN9_STM32: R175.2, TP162.1
Other:
- note added: "MECHANICAL"
- title: (none) -> MECHANICAL
- moved on the sheet: F1, H1, H10, H11, H2, H3, H4, H5, H6, H7, H8, H9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

Commit message: Commit da changes
Parts:
- removed H11, H12: MountingHole_Pad, MountingHole:MountingHole_3.2mm_M3_ISO14580_Pad, symbol Mechanical:MountingHole_Pad
- added FID1, FID2, FID3: Fiducial, Fiducial:Fiducial_1mm_Mask3mm, symbol Mechanical:Fiducial
- C76: footprint Capacitor_SMD:C_0402_1005Metric -> valve_pcb_footprints:C_0402_1005Metric
- J7: footprint Connector_Molex:Molex_Mega-Fit_76829-0110_2x05_P5.70mm_Vertical -> valve_pcb_footprints:Molex_Mega-Fit_76829-0110_2x05_P5.70mm_Vertical
- J8: JLCPCB Part # (none) -> C9132
- R172, R174, R175, R176, R177, R178, R179, R180, R181, R88, R89: footprint Resistor_SMD:R_0603_1608Metric -> valve_pcb_footprints:R_0603_1608Metric
- TP146, TP162, TP163, TP164, TP165, TP166, TP167, TP168, TP169, TP170, TP171, TP172: footprint TestPoint:TestPoint_Pad_D2.0mm -> TestPoint:TestPoint_Pad_D1.0mm
- U9: value PCA9306DC -> PCA9306DC1Z
Connections:
- net VBUS_CONN: now reaches F1.1, J7.1 (Pin_1), J7.2 (Pin_2), J7.3 (Pin_3), J7.4 (Pin_4), J7.5 (Pin_5), TP172.1
- net I2C_SCL renamed I2C3_SCL
- net I2C_SDA renamed I2C3_SDA
Other:
- note added: "20"
- note added: "3,9"
- note added: "CONTROLLER BOARD IO INTERFACE CONNECTOR"
- note added: "FIDUCIALS"
- note added: "I2C BUFFER"
- note added: "INPUT POWER"
- note added: "MOUNTING HOLES"
- note removed: "I2C buffer"
- moved on the sheet: C76, F1, H1, H10, H2, H3, H4, H5, H6, H7, H8, H9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

Commit message: Major changes due to architecture
Added battery muxing for valve power, igniter system, and separate system battery for control electronics
Parts:
- removed F1: 0297020, Fuse:Fuseholder_Blade_Mini_Keystone_3568, symbol Device:Fuse
- removed J7: 0768290110, valve_pcb_footprints:Molex_Mega-Fit_76829-0110_2x05_P5.70mm_Vertical, symbol Connector_Generic:Conn_02x05_Odd_Even
- removed TP171, TP172: TestPoint, TestPoint:TestPoint_Pad_D1.0mm, symbol Connector:TestPoint
- added J10, J22: 0768290106, valve_pcb_footprints:768290106, symbol Connector_Generic:Conn_02x03_Counter_Clockwise
- added J5: 0768290102, valve_pcb_footprints:768290102, symbol Connector_Generic:Conn_01x02
- added TP201, TP202, TP203, TP222: TestPoint, TestPoint:TestPoint_Pad_D1.0mm, symbol Connector:TestPoint
Connections:
- net GND: now also J10.1 (Pin_1), J10.2 (Pin_2), J10.3 (Pin_3), J22.1 (Pin_1), J22.2 (Pin_2), J22.3 (Pin_3), J5.2 (Pin_2), TP203.1, TP222.1
- net I2C_MASTER_SCL renamed I2C_SLAVE_SCL
- net I2C_MASTER_SDA renamed I2C_SLAVE_SDA
- new net VBUS1: J10.4 (Pin_4), J10.5 (Pin_5), J10.6 (Pin_6), TP201.1
- new net VBUS2: J22.4 (Pin_4), J22.5 (Pin_5), J22.6 (Pin_6), TP202.1
- new net VSYS: J5.1 (Pin_1)
Other:
- note added: "3"
- note added: "9"
- note added: "SYSTEM POWER"
- note added: "VALVE POWER"
- note removed: "3,9"
- note removed: "INPUT POWER"
- moved on the sheet: FID1, FID2, FID3, H1, H10, H2, H3, H4, H5, H6, H7, H8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

Commit message: Major changes
Parts:
- J8: now not fitted
Changed lines of the file:
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@@
 	(title_block
 		(title "MECHANICAL")
-		(date "2026-10-07")
+		(date "2026-10-08")
 		(rev "A")
 	)
@@
 		(on_board yes)
 		(in_pos_files yes)
-		(dnp no)
+		(dnp yes)
 		(fields_autoplaced yes)
 		(property "Reference" "J8"

Commit message: Fixes
Added hops, fixed the planes, and fixed minor issues
Parts:
- renumbered C76 to C135, J5 to J20, J22 to J21, J10 to J22, J8 to J23, R174 to R227, R175 to R228, R176 to R229, R177 to R230, R172 to R231, R88 to R232, R178 to R233, R179 to R234, R180 to R235, R181 to R236, R89 to R237, TP202 to TP185, TP222 to TP186, TP201 to TP187, TP203 to TP188, TP146 to TP189, TP162 to TP190, TP163 to TP191, TP164 to TP192, TP165 to TP193, TP166 to TP194, TP167 to TP195, TP168 to TP196, TP169 to TP197, TP170 to TP198, U9 to U31, U7 to U32, U8 to U33

Commit message: Delete a bunch of stuff
Parts:
- added J21: 0768290102, valve_pcb_footprints:768290102, symbol Connector_Generic:Conn_01x02
- J24: renamed from J23; now fitted
- renumbered J21 to J22, J22 to J23
Connections:
- net GND: now also J21.2 (Pin_2); no longer J20.2 (Pin_2)
- new net VSYS_BAT+: J20.2 (Pin_2), J21.1 (Pin_1)
Other:
- note added: "BATTERY"
- note added: "POWER SWITCH"
- moved on the sheet: J20
