File: LRUs/Valve Control Unit/Electrical/Valve Power Board/valve_control_pcb/input_mux.kicad_sch (KiCad schematic)
At the start: 24 parts, among them Q17 SiR882ADP, Q18 SiR882ADP, Q21 SiR882ADP, Q22 SiR882ADP, Q5 AO3400A, Q6 AO3400A, U5 LTC4359-MS8, U6 LTC4359-MS8

Commit message: Commit updates
Parts:
- R11, R13, R25, R27, R41, R53, R55: footprint Resistor_SMD:R_0603_1608Metric -> valve_pcb_footprints:R_0603_1608Metric
- R39: footprint Capacitor_SMD:C_0603_1608Metric -> valve_pcb_footprints:R_0603_1608Metric
Changed lines of the file:
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@@
 	(paper "A4")
 	(title_block
-		(date "2026-08-27")
+		(date "2026-10-07")
 	)
 	(text "Protect against MOSFET avalanche"
@@
 			)
 		)
-		(property "Footprint" "Resistor_SMD:R_0603_1608Metric"
+		(property "Footprint" "valve_pcb_footprints:R_0603_1608Metric"
 			(at 80.01 64.77 0)
 			(hide yes)
@@
 			)
 		)
-		(property "Footprint" "Resistor_SMD:R_0603_1608Metric"
+		(property "Footprint" "valve_pcb_footprints:R_0603_1608Metric"
 			(at 156.21 158.75 0)
 			(hide yes)
@@
 			)
 		)
-		(property "Footprint" "Resistor_SMD:R_0603_1608Metric"
+		(property "Footprint" "valve_pcb_footprints:R_0603_1608Metric"
 			(at 157.48 78.74 0)
 			(hide yes)
@@
 			)
 		)
-		(property "Footprint" "Resistor_SMD:R_0603_1608Metric"
+		(property "Footprint" "valve_pcb_footprints:R_0603_1608Metric"
 			(at 80.01 82.55 0)
 			(hide yes)
@@
 			)
 		)
-		(property "Footprint" "Resistor_SMD:R_0603_1608Metric"
+		(property "Footprint" "valve_pcb_footprints:R_0603_1608Metric"
 			(at 81.28 162.56 0)
 			(hide yes)
@@
 			)
 		)
-		(property "Footprint" "Capacitor_SMD:C_0603_1608Metric"
+		(property "Footprint" "valve_pcb_footprints:R_0603_1608Metric"
 			(at 102.87 58.42 0)
 			(hide yes)
@@
 			)
 		)
-		(property "Footprint" "Resistor_SMD:R_0603_1608Metric"
+		(property "Footprint" "valve_pcb_footprints:R_0603_1608Metric"
 			(at 81.28 144.78 0)
 			(hide yes)
@@
 			)
 		)
-		(property "Footprint" "Resistor_SMD:R_0603_1608Metric"
+		(property "Footprint" "valve_pcb_footprints:R_0603_1608Metric"
 			(at 102.87 138.43 0)
 			(hide yes)

Commit message: Major changes
Parts:
- removed D19, D20: SMAT70A-13-F, Diode_SMD:D_SMA, symbol Device:D_Zener
- removed D21, D22: MMSZ5245B, Diode_SMD:D_SOD-123, symbol Device:D_Zener
- removed Q17, Q22: SiR882ADP, Package_SO:PowerPAK_SO-8_Single, symbol Transistor_FET:SiR696DP
- removed R53, R55: 1k, valve_pcb_footprints:R_0603_1608Metric, symbol Device:R_Small_US
- removed U5, U6: LTC4359-MS8, Package_SO:MSOP-8_3x3mm_P0.65mm, symbol Power_Management:LTC4359-MS8
- added C144, C145: 100nF, valve_pcb_footprints:C_0402_1005Metric, symbol Device:C_Small_US
- added U16, U29: LM74700, Package_TO_SOT_SMD:SOT-23-6_Handsoldering, symbol Power_Management:LM74700
- Q18, Q21: value SiR882ADP -> SIR5108DP; footprint Package_SO:PowerPAK_SO-8_Single -> valve_pcb_footprints:PowerPAK_SO-8_Single; JLCPCB Part # C553986 -> C53262900
Connections:
- net VIN1_SRC is gone; now on net VIN_1: Q18.1 (S), Q18.2 (S), Q18.3 (S)
- net VIN2_SRC is gone; now on net VIN_2: Q21.1 (S), Q21.2 (S), Q21.3 (S)
- net GND: now also U16.2 (GND), U29.2 (GND)
- net VIN1_GATE: now also U16.5 (GATE)
- net VIN2_GATE: now also U29.5 (GATE)
- net VIN_1: now also C144.1, U16.6 (ANODE); no longer Q18.5 (D)
- net VIN_2: now also C145.1, U29.6 (ANODE)
- net VOUT: now also Q18.5 (D), U16.4 (CATHODE), U29.4 (CATHODE)
- net ~{VIN1_SHDN}: now also U16.3 (EN)
- net ~{VIN2_SHDN}: now also U29.3 (EN)
- new net: C144.2, U16.1 (VCAP)
- new net: C145.2, U29.1 (VCAP)
Other:
- title: (none) -> INPUT MUX
- moved on the sheet: D17

Commit message: Fixes
Added hops, fixed the planes, and fixed minor issues
Parts:
- added C17, C18: 100nF, valve_pcb_footprints:C_0402_1005Metric, symbol Device:C_Small_US
- renumbered C144 to C19, C145 to C20, C18 to C21, C17 to C22, D17 to D3, D18 to D4, Q5 to Q1, Q6 to Q2, Q21 to Q3, Q18 to Q4, R11 to R20, R13 to R21, R25 to R22, R27 to R23, R39 to R24, R41 to R25, U29 to U6, U16 to U7
Connections:
- net GND: now also C17.2, C18.2
- net VIN_1: now also C17.1
- net VIN_2: now also C18.1
Other:
- note removed: "Protect against MOSFET avalanche"
- moved on the sheet: C19, C20, C21, C22, D3, D4

Commit message: Delete a bunch of stuff
Other:
- note added: "INPUT MUX"
Changed lines of the file:
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@@
 		(rev "A")
+	)
+	(text "INPUT MUX"
+		(exclude_from_sim no)
+		(at 233.68 144.526 0)
+		(effects
+			(font
+				(size 7.62 7.62)
+				(thickness 1.016)
+				(bold yes)
+				(color 0 0 0 1)
+			)
+		)
 	)
 	(junction
