File: LRUs/Valve Control Unit/Electrical/Valve Power Board/valve_control_pcb/ldo_3V3.kicad_sch (KiCad schematic)
At the start: 7 parts, among them U17 AMS1117-3.3

Commit message: Small updates
Parts:
- removed D42: GREEN, LED_SMD:LED_0805_2012Metric, symbol Device:LED
- added D19: RED, LED_SMD:LED_0603_1608Metric, symbol Device:LED
Connections:
- net GND: now also D19.1 (K)
- net at R242.2: now also D19.2 (A)
Changed lines of the file:
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@@
+	)
+	(symbol
+		(lib_id "Device:LED")
+		(at 194.31 111.76 90)
+		(unit 1)
+		(body_style 1)
+		(exclude_from_sim no)
+		(in_bom yes)
+		(on_board yes)
+		(in_pos_files yes)
+		(dnp no)
+		(property "Reference" "D19"
+			(at 196.85 109.728 90)
+			(show_name no)
+			(do_not_autoplace no)
+			(effects
+				(font
+					(size 1.27 1.27)
+				)
+				(justify right)
+			)
+		)
+		(property "Value" "RED"
+			(at 196.85 111.506 90)
+			(show_name no)
+			(do_not_autoplace no)
+			(effects
+				(font
+					(size 1.27 1.27)
+				)
+				(justify right)
+			)
+		)
+		(property "Footprint" "LED_SMD:LED_0603_1608Metric"
+			(at 194.31 111.76 0)
+			(hide yes)
+			(show_name no)
+			(do_not_autoplace no)
+			(effects
+				(font
+					(size 1.27 1.27)
+				)
+			)
+		)
+		(property "Datasheet" ""
+			(at 194.31 111.76 0)
+			(hide yes)
+			(show_name no)
+			(do_not_autoplace no)
+			(effects
+				(font
+					(size 1.27 1.27)
+				)
+			)
+		)
+		(property "Description" "KT-0603R Red LED"
+			(at 194.31 111.76 0)
+			(hide yes)
+			(show_name no)
+			(do_not_autoplace no)
+			(effects
+				(font
+					(size 1.27 1.27)
+				)
+			)
+		)
+		(property "Sim.Pins" "1=K 2=A"
+			(at 194.31 111.76 0)
+			(hide yes)
+			(show_name no)
+			(do_not_autoplace no)
+			(effects
+				(font
+					(size 1.27 1.27)
+				)
+			)
+		)
+		(property "Vf" "2V"
+			(at 198.12 113.284 90)
+			(show_name no)
+			(do_not_autoplace no)
+			(effects
+				(font
+					(size 1.27 1.27)
+				)
+			)
+		)
+		(property "JLCPCB Part #" "C2286"
+			(at 194.31 111.76 90)
+			(hide yes)
+			(show_name no)
+			(do_not_autoplace no)
+			(effects
+				(font
+					(size 1.27 1.27)
+				)
+			)
+		)
+		(property "Footprint_Size" "0603"
+			(at 199.39 115.062 90)
+			(show_name no)
+			(do_not_autoplace no)
+			(effects
+				(font
+					(size 1.27 1.27)
+				)
+			)
+		)
+		(pin "1"
+		)
+		(pin "2"
+		)
+		(instances
+			(project "valve_control_pcb"
+				(path "/5d72873d-bf63-43c9-aa68-e8ad4e59e232/e3918634-dfcc-4cc2-a043-1fe32896c4e0"
+					(reference "D19")
+					(unit 1)
+					(variant
+						(name "My VARIANT DARNIT")
+					)
+				)
+			)
+		)
 	)
 	(symbol
@@
 				)
 			)
-		)
-	)
-	(symbol
-		(lib_id "Device:LED")
-		(at 194.31 111.76 90)
-		(unit 1)
-		(body_style 1)
-		(exclude_from_sim no)
-		(in_bom yes)
-		(on_board yes)
-		(in_pos_files yes)
-		(dnp no)
-		(property "Reference" "D42"
-			(at 196.85 109.982 90)
-			(show_name no)
-			(do_not_autoplace no)
-			(effects
-				(font
-					(size 1.27 1.27)
-				)
-				(justify right)
-			)
-		)
-		(property "Value" "GREEN"
-			(at 196.85 111.76 90)
-			(show_name no)
-			(do_not_autoplace no)
-			(effects
-				(font
-					(size 1.27 1.27)
-				)
-				(justify right)
-			)
-		)
-		(property "Footprint" "LED_SMD:LED_0805_2012Metric"
-			(at 194.31 111.76 0)
-			(hide yes)
-			(show_name no)
-			(do_not_autoplace no)
-			(effects
-				(font
-					(size 1.27 1.27)
-				)
-			)
-		)
-		(property "Datasheet" ""
-			(at 194.31 111.76 0)
-			(hide yes)
-			(show_name no)
-			(do_not_autoplace no)
-			(effects
-				(font
-					(size 1.27 1.27)
-				)
-			)
-		)
-		(property "Description" "KT-0603R Red LED"
-			(at 194.31 111.76 0)
-			(hide yes)
-			(show_name no)
-			(do_not_autoplace no)
-			(effects
-				(font
-					(size 1.27 1.27)
-				)
-			)
-		)
-		(property "Sim.Pins" "1=K 2=A"
-			(at 194.31 111.76 0)
-			(hide yes)
-			(show_name no)
-			(do_not_autoplace no)
-			(effects
-				(font
-					(size 1.27 1.27)
-				)
-			)
-		)
-		(property "Vf" "3.1V"
-			(at 199.136 113.538 90)
-			(show_name no)
-			(do_not_autoplace no)
-			(effects
-				(font
-					(size 1.27 1.27)
-				)
-			)
-		)
-		(property "JLCPCB Part #" "C2297"
-			(at 194.31 111.76 90)
-			(hide yes)
-			(show_name no)
-			(do_not_autoplace no)
-			(effects
-				(font
-					(size 1.27 1.27)
-				)
-			)
-		)
-		(property "Footprint_Size" "0805"
-			(at 199.39 115.316 90)
-			(show_name no)
-			(do_not_autoplace no)
-			(effects
-				(font
-					(size 1.27 1.27)
-				)
-			)
-		)
-		(pin "1"
-		)
-		(pin "2"
-		)
-		(instances
-			(project "valve_control_pcb"
-				(path "/5d72873d-bf63-43c9-aa68-e8ad4e59e232/e3918634-dfcc-4cc2-a043-1fe32896c4e0"
-					(reference "D42")
-					(unit 1)
-					(variant
-						(name "My VARIANT DARNIT")
-					)
-				)
-			)

Commit message: Fixes
Added hops, fixed the planes, and fixed minor issues
Parts:
- renumbered C63 to C10, C65 to C11, C61 to C9, D19 to D2, R242 to R13, TP107 to TP7, U17 to U3
Changed lines of the file:
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@@
 		(in_pos_files yes)
 		(dnp no)
-		(property "Reference" "D19"
+		(property "Reference" "D2"
 			(at 196.85 109.728 90)
 			(show_name no)
@@
 			(project "valve_control_pcb"
 				(path "/5d72873d-bf63-43c9-aa68-e8ad4e59e232/e3918634-dfcc-4cc2-a043-1fe32896c4e0"
-					(reference "D19")
+					(reference "D2")
 					(unit 1)
 					(variant
@@
 		(dnp no)
 		(fields_autoplaced yes)
-		(property "Reference" "#PWR0170"
+		(property "Reference" "#PWR021"
 			(at 167.64 109.22 0)
 			(hide yes)
@@
 			(project "valve_control_pcb"
 				(path "/5d72873d-bf63-43c9-aa68-e8ad4e59e232/e3918634-dfcc-4cc2-a043-1fe32896c4e0"
-					(reference "#PWR0170")
+					(reference "#PWR021")
 					(unit 1)
 				)
@@
 		(in_pos_files yes)
 		(dnp no)
-		(property "Reference" "C63"
+		(property "Reference" "C10"
 			(at 169.164 96.774 0)
 			(show_name no)
@@
 			(project "valve_control_pcb"
 				(path "/5d72873d-bf63-43c9-aa68-e8ad4e59e232/e3918634-dfcc-4cc2-a043-1fe32896c4e0"
-					(reference "C63")
+					(reference "C10")
 					(unit 1)
 					(variant
@@
 		(in_pos_files yes)
 		(dnp no)
-		(property "Reference" "TP107"
+		(property "Reference" "TP7"
 			(at 181.61 91.44 90)
 			(show_name no)
@@
 			(project "valve_control_pcb"
 				(path "/5d72873d-bf63-43c9-aa68-e8ad4e59e232/e3918634-dfcc-4cc2-a043-1fe32896c4e0"
-					(reference "TP107")
+					(reference "TP7")
 					(unit 1)
 					(variant
@@
 		(dnp no)
 		(fields_autoplaced yes)
-		(property "Reference" "#PWR0172"
+		(property "Reference" "#PWR022"
 			(at 180.34 109.22 0)
 			(hide yes)
@@
 			(project "valve_control_pcb"
 				(path "/5d72873d-bf63-43c9-aa68-e8ad4e59e232/e3918634-dfcc-4cc2-a043-1fe32896c4e0"
-					(reference "#PWR0172")
+					(reference "#PWR022")
 					(unit 1)
 				)
@@
 		(dnp no)
 		(fields_autoplaced yes)
-		(property "Reference" "#PWR0318"
+		(property "Reference" "#PWR023"
 			(at 194.31 124.46 0)
 			(hide yes)
@@
 			(project "valve_control_pcb"
 				(path "/5d72873d-bf63-43c9-aa68-e8ad4e59e232/e3918634-dfcc-4cc2-a043-1fe32896c4e0"
-					(reference "#PWR0318")
+					(reference "#PWR023")
 					(unit 1)
 				)
@@
 		(dnp no)
 		(fields_autoplaced yes)
-		(property "Reference" "U17"
+		(property "Reference" "U3"
 			(at 147.32 87.63 0)
 			(show_name no)
@@
 			(project "valve_control_pcb"
 				(path "/5d72873d-bf63-43c9-aa68-e8ad4e59e232/e3918634-dfcc-4cc2-a043-1fe32896c4e0"
-					(reference "U17")
+					(reference "U3")
 					(unit 1)
 				)
@@
 		(dnp no)
 		(fields_autoplaced yes)
-		(property "Reference" "#PWR0168"
+		(property "Reference" "#PWR020"
 			(at 147.32 109.22 0)
 			(hide yes)
@@
 			(project "valve_control_pcb"
 				(path "/5d72873d-bf63-43c9-aa68-e8ad4e59e232/e3918634-dfcc-4cc2-a043-1fe32896c4e0"
-					(reference "#PWR0168")
+					(reference "#PWR020")
 					(unit 1)
 				)
@@
 		(dnp no)
 		(fields_autoplaced yes)
-		(property "Reference" "#FLG05"
+		(property "Reference" "#FLG01"
 			(at 132.08 92.075 0)
 			(hide yes)
@@
 			(project "valve_control_pcb"
 				(path "/5d72873d-bf63-43c9-aa68-e8ad4e59e232/e3918634-dfcc-4cc2-a043-1fe32896c4e0"
-					(reference "#FLG05")
+					(reference "#FLG01")
 					(unit 1)
 				)
@@
 		(in_pos_files yes)
 		(dnp no)
-		(property "Reference" "C65"
+		(property "Reference" "C11"
 			(at 182.118 97.028 0)
 			(show_name no)
@@
 			(project "valve_control_pcb"
 				(path "/5d72873d-bf63-43c9-aa68-e8ad4e59e232/e3918634-dfcc-4cc2-a043-1fe32896c4e0"
-					(reference "C65")
+					(reference "C11")
 					(unit 1)
 					(variant
@@
 		(dnp no)
 		(fields_autoplaced yes)
-		(property "Reference" "#PWR0163"
+		(property "Reference" "#PWR019"
 			(at 124.46 109.22 0)
 			(hide yes)
@@
 			(project "valve_control_pcb"
 				(path "/5d72873d-bf63-43c9-aa68-e8ad4e59e232/e3918634-dfcc-4cc2-a043-1fe32896c4e0"
-					(reference "#PWR0163")
+					(reference "#PWR019")
 					(unit 1)
 				)
@@
 		(in_pos_files yes)
 		(dnp no)
-		(property "Reference" "C61"
+		(property "Reference" "C9"
 			(at 126.238 96.774 0)
 			(show_name no)
@@
 			(project "valve_control_pcb"
 				(path "/5d72873d-bf63-43c9-aa68-e8ad4e59e232/e3918634-dfcc-4cc2-a043-1fe32896c4e0"
-					(reference "C61")
+					(reference "C9")
 					(unit 1)
 					(variant
@@
 		(in_pos_files yes)
 		(dnp no)
-		(property "Reference" "R242"
+		(property "Reference" "R13"
 			(at 198.374 99.06 0)
 			(show_name no)
@@
 			(project "valve_control_pcb"
 				(path "/5d72873d-bf63-43c9-aa68-e8ad4e59e232/e3918634-dfcc-4cc2-a043-1fe32896c4e0"
-					(reference "R242")
+					(reference "R13")
 					(unit 1)
 					(variant

Commit message: Delete a bunch of stuff
Other:
- note added: "LDO 3V3"
Changed lines of the file:
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@@
 		(rev "A")
+	)
+	(text "LDO 3V3"
+		(exclude_from_sim no)
+		(at 147.32 52.578 0)
+		(effects
+			(font
+				(size 7.62 7.62)
+				(thickness 1.016)
+				(bold yes)
+				(color 0 0 0 1)
+			)
+		)
 	)
 	(junction
