File: LRUs/Valve Control Unit/Electrical/Valve Power Board/valve_control_pcb/lsw_3V3.kicad_sch (KiCad schematic)
At the start: 7 parts, among them J11 Conn_01x02_Pin, U21 TPS22810DBV

Commit message: Fixes
Added hops, fixed the planes, and fixed minor issues
Parts:
- renumbered C64 to C12, J11 to J2, R123 to R17, R125 to R18, R241 to R19, TP145 to TP9, U21 to U5
Changed lines of the file:
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@@
 		(in_pos_files yes)
 		(dnp no)
-		(property "Reference" "R241"
+		(property "Reference" "R19"
 			(at 191.516 95.25 90)
 			(show_name no)
@@
 			(project "valve_control_pcb"
 				(path "/5d72873d-bf63-43c9-aa68-e8ad4e59e232/6376898b-44f3-4f20-a970-57c6f45bf2f7"
-					(reference "R241")
+					(reference "R19")
 					(unit 1)
 					(variant
@@
 		(dnp no)
 		(fields_autoplaced yes)
-		(property "Reference" "#PWR0166"
+		(property "Reference" "#PWR027"
 			(at 119.38 116.84 0)
 			(hide yes)
@@
 			(project "valve_control_pcb"
 				(path "/5d72873d-bf63-43c9-aa68-e8ad4e59e232/6376898b-44f3-4f20-a970-57c6f45bf2f7"
-					(reference "#PWR0166")
+					(reference "#PWR027")
 					(unit 1)
 				)
@@
 		(in_pos_files yes)
 		(dnp no)
-		(property "Reference" "R123"
+		(property "Reference" "R17"
 			(at 121.158 94.488 0)
 			(show_name no)
@@
 			(project "valve_control_pcb"
 				(path "/5d72873d-bf63-43c9-aa68-e8ad4e59e232/6376898b-44f3-4f20-a970-57c6f45bf2f7"
-					(reference "R123")
+					(reference "R17")
 					(unit 1)
 					(variant
@@
 		(dnp no)
 		(fields_autoplaced yes)
-		(property "Reference" "#PWR0171"
+		(property "Reference" "#PWR029"
 			(at 163.83 111.76 0)
 			(hide yes)
@@
 			(project "valve_control_pcb"
 				(path "/5d72873d-bf63-43c9-aa68-e8ad4e59e232/6376898b-44f3-4f20-a970-57c6f45bf2f7"
-					(reference "#PWR0171")
+					(reference "#PWR029")
 					(unit 1)
 				)
@@
 		(in_pos_files yes)
 		(dnp no)
-		(property "Reference" "J11"
+		(property "Reference" "J2"
 			(at 100.584 105.156 0)
 			(show_name no)
@@
 			(project "valve_control_pcb"
 				(path "/5d72873d-bf63-43c9-aa68-e8ad4e59e232/6376898b-44f3-4f20-a970-57c6f45bf2f7"
-					(reference "J11")
+					(reference "J2")
 					(unit 1)
 				)
@@
 		(dnp no)
 		(fields_autoplaced yes)
-		(property "Reference" "#PWR0169"
+		(property "Reference" "#PWR028"
 			(at 149.86 109.22 0)
 			(hide yes)
@@
 			(project "valve_control_pcb"
 				(path "/5d72873d-bf63-43c9-aa68-e8ad4e59e232/6376898b-44f3-4f20-a970-57c6f45bf2f7"
-					(reference "#PWR0169")
+					(reference "#PWR028")
 					(unit 1)
 				)
@@
 		(in_pos_files yes)
 		(dnp no)
-		(property "Reference" "TP145"
+		(property "Reference" "TP9"
 			(at 172.72 96.52 90)
 			(show_name no)
@@
 			(project "valve_control_pcb"
 				(path "/5d72873d-bf63-43c9-aa68-e8ad4e59e232/6376898b-44f3-4f20-a970-57c6f45bf2f7"
-					(reference "TP145")
+					(reference "TP9")
 					(unit 1)
 					(variant
@@
 		(in_pos_files yes)
 		(dnp no)
-		(property "Reference" "C64"
+		(property "Reference" "C12"
 			(at 166.116 99.568 0)
 			(show_name no)
@@
 			(project "valve_control_pcb"
 				(path "/5d72873d-bf63-43c9-aa68-e8ad4e59e232/6376898b-44f3-4f20-a970-57c6f45bf2f7"
-					(reference "C64")
+					(reference "C12")
 					(unit 1)
 					(variant
@@
 		(dnp no)
 		(fields_autoplaced yes)
-		(property "Reference" "U21"
+		(property "Reference" "U5"
 			(at 149.86 83.82 0)
 			(show_name no)
@@
 			(project "valve_control_pcb"
 				(path "/5d72873d-bf63-43c9-aa68-e8ad4e59e232/6376898b-44f3-4f20-a970-57c6f45bf2f7"
-					(reference "U21")
+					(reference "U5")
 					(unit 1)
 				)
@@
 		(in_pos_files yes)
 		(dnp no)
-		(property "Reference" "R125"
+		(property "Reference" "R18"
 			(at 121.158 104.14 0)
 			(show_name no)
@@
 			(project "valve_control_pcb"
 				(path "/5d72873d-bf63-43c9-aa68-e8ad4e59e232/6376898b-44f3-4f20-a970-57c6f45bf2f7"
-					(reference "R125")
+					(reference "R18")
 					(unit 1)
 					(variant
@@
 		(dnp no)
 		(fields_autoplaced yes)
-		(property "Reference" "#PWR0164"
+		(property "Reference" "#PWR026"
 			(at 111.76 116.84 0)
 			(hide yes)
@@
 			(project "valve_control_pcb"
 				(path "/5d72873d-bf63-43c9-aa68-e8ad4e59e232/6376898b-44f3-4f20-a970-57c6f45bf2f7"
-					(reference "#PWR0164")
+					(reference "#PWR026")
 					(unit 1)
 				)

Commit message: Delete a bunch of stuff
Other:
- note added: "LSW 3V3"
Changed lines of the file:
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@@
+		)
+	)
+	(text "LSW 3V3"
+		(exclude_from_sim no)
+		(at 146.812 55.88 0)
+		(effects
+			(font
+				(size 7.62 7.62)
+				(thickness 1.016)
+				(bold yes)
+				(color 0 0 0 1)
+			)
 		)
 	)
