File: LRUs/Valve Control Unit/Electrical/Valve Power Board/valve_control_pcb/lsw_5V.kicad_sch (KiCad schematic)
At the start: 7 parts, among them J17 01x02_PinHeader, U20 TPS22810DBV

Commit message: Fixes
Added hops, fixed the planes, and fixed minor issues
Parts:
- renumbered C128 to C8, J17 to J1, R238 to R10, R239 to R11, R240 to R12, TP144 to TP6, U20 to U2
Changed lines of the file:
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@@
 		(in_pos_files yes)
 		(dnp no)
-		(property "Reference" "R238"
+		(property "Reference" "R10"
 			(at 124.968 97.028 0)
 			(show_name no)
@@
 			(project "valve_control_pcb"
 				(path "/5d72873d-bf63-43c9-aa68-e8ad4e59e232/04da9a24-fd32-4df1-a058-64d5dac33734"
-					(reference "R238")
+					(reference "R10")
 					(unit 1)
 					(variant
@@
 		(dnp no)
 		(fields_autoplaced yes)
-		(property "Reference" "#PWR0296"
+		(property "Reference" "#PWR015"
 			(at 118.11 119.38 0)
 			(hide yes)
@@
 			(project "valve_control_pcb"
 				(path "/5d72873d-bf63-43c9-aa68-e8ad4e59e232/04da9a24-fd32-4df1-a058-64d5dac33734"
-					(reference "#PWR0296")
+					(reference "#PWR015")
 					(unit 1)
 				)
@@
 		(in_pos_files yes)
 		(dnp no)
-		(property "Reference" "TP144"
+		(property "Reference" "TP6"
 			(at 176.53 99.06 90)
 			(show_name no)
@@
 			(project "valve_control_pcb"
 				(path "/5d72873d-bf63-43c9-aa68-e8ad4e59e232/04da9a24-fd32-4df1-a058-64d5dac33734"
-					(reference "TP144")
+					(reference "TP6")
 					(unit 1)
 					(variant
@@
 		(in_pos_files yes)
 		(dnp no)
-		(property "Reference" "R239"
+		(property "Reference" "R11"
 			(at 127.508 106.68 0)
 			(show_name no)
@@
 			(project "valve_control_pcb"
 				(path "/5d72873d-bf63-43c9-aa68-e8ad4e59e232/04da9a24-fd32-4df1-a058-64d5dac33734"
-					(reference "R239")
+					(reference "R11")
 					(unit 1)
 					(variant
@@
 		(in_pos_files yes)
 		(dnp no)
-		(property "Reference" "R240"
+		(property "Reference" "R12"
 			(at 190.246 100.076 90)
 			(show_name no)
@@
 			(project "valve_control_pcb"
 				(path "/5d72873d-bf63-43c9-aa68-e8ad4e59e232/04da9a24-fd32-4df1-a058-64d5dac33734"
-					(reference "R240")
+					(reference "R12")
 					(unit 1)
 					(variant
@@
 		(dnp no)
 		(fields_autoplaced yes)
-		(property "Reference" "U20"
+		(property "Reference" "U2"
 			(at 149.86 86.36 0)
 			(show_name no)
@@
 			(project "valve_control_pcb"
 				(path "/5d72873d-bf63-43c9-aa68-e8ad4e59e232/04da9a24-fd32-4df1-a058-64d5dac33734"
-					(reference "U20")
+					(reference "U2")
 					(unit 1)
 				)
@@
 		(in_pos_files yes)
 		(dnp no)
-		(property "Reference" "C128"
+		(property "Reference" "C8"
 			(at 169.418 101.854 0)
 			(show_name no)
@@
 			(project "valve_control_pcb"
 				(path "/5d72873d-bf63-43c9-aa68-e8ad4e59e232/04da9a24-fd32-4df1-a058-64d5dac33734"
-					(reference "C128")
+					(reference "C8")
 					(unit 1)
 					(variant
@@
 		(dnp no)
 		(fields_autoplaced yes)
-		(property "Reference" "#PWR0299"
+		(property "Reference" "#PWR018"
 			(at 167.64 114.3 0)
 			(hide yes)
@@
 			(project "valve_control_pcb"
 				(path "/5d72873d-bf63-43c9-aa68-e8ad4e59e232/04da9a24-fd32-4df1-a058-64d5dac33734"
-					(reference "#PWR0299")
+					(reference "#PWR018")
 					(unit 1)
 				)
@@
 		(in_pos_files yes)
 		(dnp no)
-		(property "Reference" "J17"
+		(property "Reference" "J1"
 			(at 106.934 107.696 0)
 			(show_name no)
@@
 			(project "valve_control_pcb"
 				(path "/5d72873d-bf63-43c9-aa68-e8ad4e59e232/04da9a24-fd32-4df1-a058-64d5dac33734"
-					(reference "J17")
+					(reference "J1")
 					(unit 1)
 				)
@@
 		(dnp no)
 		(fields_autoplaced yes)
-		(property "Reference" "#PWR0297"
+		(property "Reference" "#PWR016"
 			(at 123.19 119.38 0)
 			(hide yes)
@@
 			(project "valve_control_pcb"
 				(path "/5d72873d-bf63-43c9-aa68-e8ad4e59e232/04da9a24-fd32-4df1-a058-64d5dac33734"
-					(reference "#PWR0297")
+					(reference "#PWR016")
 					(unit 1)
 				)
@@
 		(dnp no)
 		(fields_autoplaced yes)
-		(property "Reference" "#PWR0298"
+		(property "Reference" "#PWR017"
 			(at 149.86 110.49 0)
 			(hide yes)
@@
 			(project "valve_control_pcb"
 				(path "/5d72873d-bf63-43c9-aa68-e8ad4e59e232/04da9a24-fd32-4df1-a058-64d5dac33734"
-					(reference "#PWR0298")
+					(reference "#PWR017")
 					(unit 1)
 				)

Commit message: Delete a bunch of stuff
Other:
- note added: "LSW 5V"
Changed lines of the file:
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@@
+		)
+	)
+	(text "LSW 5V"
+		(exclude_from_sim no)
+		(at 150.114 54.102 0)
+		(effects
+			(font
+				(size 7.62 7.62)
+				(thickness 1.016)
+				(bold yes)
+				(color 0 0 0 1)
+			)
 		)
 	)
