File: LRUs/Valve Control Unit/Electrical/Valve Power Board/valve_control_pcb/mux_3V3.kicad_sch (KiCad schematic)
At the start: 5 parts, among them U18 TPS2116DRL

Commit message: Fixes
Added hops, fixed the planes, and fixed minor issues
Parts:
- renumbered R118 to R14, R119 to R15, R122 to R16, TP110 to TP8, U18 to U4
Changed lines of the file:
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@@
 		(dnp no)
 		(fields_autoplaced yes)
-		(property "Reference" "#PWR0158"
+		(property "Reference" "#PWR025"
 			(at 153.67 114.3 0)
 			(hide yes)
@@
 			(project "valve_control_pcb"
 				(path "/5d72873d-bf63-43c9-aa68-e8ad4e59e232/3289eb84-03de-481c-8338-449ebd0f80fb"
-					(reference "#PWR0158")
+					(reference "#PWR025")
 					(unit 1)
 				)
@@
 		(in_pos_files yes)
 		(dnp no)
-		(property "Reference" "R119"
+		(property "Reference" "R15"
 			(at 121.92 95.25 0)
 			(show_name no)
@@
 			(project "valve_control_pcb"
 				(path "/5d72873d-bf63-43c9-aa68-e8ad4e59e232/3289eb84-03de-481c-8338-449ebd0f80fb"
-					(reference "R119")
+					(reference "R15")
 					(unit 1)
 					(variant
@@
 		(dnp no)
 		(fields_autoplaced yes)
-		(property "Reference" "U18"
+		(property "Reference" "U4"
 			(at 153.67 83.82 0)
 			(show_name no)
@@
 			(project "valve_control_pcb"
 				(path "/5d72873d-bf63-43c9-aa68-e8ad4e59e232/3289eb84-03de-481c-8338-449ebd0f80fb"
-					(reference "U18")
+					(reference "U4")
 					(unit 1)
 					(variant
@@
 		(in_pos_files yes)
 		(dnp no)
-		(property "Reference" "TP110"
+		(property "Reference" "TP8"
 			(at 176.53 88.9 90)
 			(show_name no)
@@
 			(project "valve_control_pcb"
 				(path "/5d72873d-bf63-43c9-aa68-e8ad4e59e232/3289eb84-03de-481c-8338-449ebd0f80fb"
-					(reference "TP110")
+					(reference "TP8")
 					(unit 1)
 					(variant
@@
 		(in_pos_files yes)
 		(dnp no)
-		(property "Reference" "R122"
+		(property "Reference" "R16"
 			(at 178.816 93.98 0)
 			(show_name no)
@@
 			(project "valve_control_pcb"
 				(path "/5d72873d-bf63-43c9-aa68-e8ad4e59e232/3289eb84-03de-481c-8338-449ebd0f80fb"
-					(reference "R122")
+					(reference "R16")
 					(unit 1)
 					(variant
@@
 		(in_pos_files yes)
 		(dnp no)
-		(property "Reference" "R118"
+		(property "Reference" "R14"
 			(at 119.38 83.82 0)
 			(show_name no)
@@
 			(project "valve_control_pcb"
 				(path "/5d72873d-bf63-43c9-aa68-e8ad4e59e232/3289eb84-03de-481c-8338-449ebd0f80fb"
-					(reference "R118")
+					(reference "R14")
 					(unit 1)
 					(variant
@@
 		(dnp no)
 		(fields_autoplaced yes)
-		(property "Reference" "#PWR0157"
+		(property "Reference" "#PWR024"
 			(at 118.11 114.3 0)
 			(hide yes)
@@
 			(project "valve_control_pcb"
 				(path "/5d72873d-bf63-43c9-aa68-e8ad4e59e232/3289eb84-03de-481c-8338-449ebd0f80fb"
-					(reference "#PWR0157")
+					(reference "#PWR024")
 					(unit 1)
 				)

Commit message: Delete a bunch of stuff
Other:
- note added: "MUX 3V3"
Changed lines of the file:
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@@
 		(rev "A")
+	)
+	(text "MUX 3V3"
+		(exclude_from_sim no)
+		(at 153.416 53.34 0)
+		(effects
+			(font
+				(size 7.62 7.62)
+				(thickness 1.016)
+				(bold yes)
+				(color 0 0 0 1)
+			)
+		)
 	)
 	(text "lower threshold for \nswitch to main board rail: 3V\n"
