File: LRUs/Valve Control Unit/Electrical/Valve Power Board/valve_control_pcb/igniter.kicad_sch (KiCad schematic)
At the start: 70 parts, among them J18 XT-60, J19 B4B-XH-A, J20 1x2 Screw Terminal, J21 1x2 Screw Terminal, K1 J107F1CS205VDC.45, Q13 AO3400A, Q14 STD52P3LLH6, Q15 AO3400A, Q16 AO3400A, U28 TPS259830ONRGER

Commit message: Commit updates
Parts:
- C135, C141, C143: footprint Capacitor_SMD:C_0402_1005Metric -> valve_pcb_footprints:C_0402_1005Metric
- C136, C137: footprint Capacitor_SMD:C_0603_1608Metric -> valve_pcb_footprints:C_0603_1608Metric
- R244, R245, R247, R252, R253, R259, R260, R262, R263, R264, R265, R266, R267, R268, R269, R270, R271, R272, R273, R274, R275, R276, R277, R278: footprint Resistor_SMD:R_0603_1608Metric -> valve_pcb_footprints:R_0603_1608Metric
- R258, R261: footprint Resistor_SMD:R_0603_1608Metric -> valve_pcb_footprints:R_0603_1608Metric; Footprint_Size (none) -> 0603
Other:
- title: (none) -> IGNITER SYSTEM
Changed lines of the file:
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@@
 	(generator_version "10.0")
 	(paper "A3")
+	(title_block
+		(title "IGNITER SYSTEM")
+		(date "2026-10-07")
+		(rev "A")
+	)
 	(rectangle
 		(start 331.724 200.66)
@@
 			)
 		)
-		(property "Footprint" "Capacitor_SMD:C_0402_1005Metric"
+		(property "Footprint" "valve_pcb_footprints:C_0402_1005Metric"
 			(at 317.5 170.18 0)
 			(hide yes)
@@
 			)
 		)
-		(property "Footprint" "Resistor_SMD:R_0603_1608Metric"
+		(property "Footprint" "valve_pcb_footprints:R_0603_1608Metric"
 			(at 187.96 109.22 0)
 			(hide yes)
@@
 			)
 		)
-		(property "Footprint" "Capacitor_SMD:C_0603_1608Metric"
+		(property "Footprint" "valve_pcb_footprints:C_0603_1608Metric"
 			(at 176.53 133.35 0)
 			(hide yes)
@@
 			)
 		)
-		(property "Footprint" "Capacitor_SMD:C_0402_1005Metric"
+		(property "Footprint" "valve_pcb_footprints:C_0402_1005Metric"
 			(at 356.87 177.8 0)
 			(hide yes)
@@
 			)
 		)
-		(property "Footprint" "Resistor_SMD:R_0603_1608Metric"
+		(property "Footprint" "valve_pcb_footprints:R_0603_1608Metric"
 			(at 303.53 226.06 0)
 			(hide yes)
@@
 			)
 		)
-		(property "Footprint" "Resistor_SMD:R_0603_1608Metric"
+		(property "Footprint" "valve_pcb_footprints:R_0603_1608Metric"
 			(at 162.56 231.14 0)
 			(hide yes)
@@
 			)
 		)
-		(property "Footprint" "Resistor_SMD:R_0603_1608Metric"
+		(property "Footprint" "valve_pcb_footprints:R_0603_1608Metric"
 			(at 109.22 130.81 0)
 			(hide yes)
@@
 			)
 		)
-		(property "Footprint" "Resistor_SMD:R_0603_1608Metric"
+		(property "Footprint" "valve_pcb_footprints:R_0603_1608Metric"
 			(at 187.96 238.76 0)
 			(hide yes)
@@
 			)
 		)
-		(property "Footprint" "Resistor_SMD:R_0603_1608Metric"
+		(property "Footprint" "valve_pcb_footprints:R_0603_1608Metric"
 			(at 278.13 92.71 0)
 			(hide yes)
@@
 			)
 		)
-		(property "Footprint" "Capacitor_SMD:C_0402_1005Metric"
+		(property "Footprint" "valve_pcb_footprints:C_0402_1005Metric"
 			(at 107.95 91.44 0)
 			(hide yes)
@@
 			)
 		)
-		(property "Footprint" "Resistor_SMD:R_0603_1608Metric"
+		(property "Footprint" "valve_pcb_footprints:R_0603_1608Metric"
 			(at 349.25 172.72 0)
 			(hide yes)
@@
 			)
 		)
-		(property "Footprint" "Resistor_SMD:R_0603_1608Metric"
+		(property "Footprint" "valve_pcb_footprints:R_0603_1608Metric"
 			(at 78.74 130.81 0)
 			(hide yes)
@@
 			)
 		)
-		(property "Footprint" "Resistor_SMD:R_0603_1608Metric"
+		(property "Footprint" "valve_pcb_footprints:R_0603_1608Metric"
 			(at 200.66 227.33 0)
 			(hide yes)
@@
 			)
 		)
-		(property "Footprint" "Capacitor_SMD:C_0603_1608Metric"
+		(property "Footprint" "valve_pcb_footprints:C_0603_1608Metric"
 			(at 175.26 101.6 0)
 			(hide yes)
@@
 			)
 		)
-		(property "Footprint" "Resistor_SMD:R_0603_1608Metric"
+		(property "Footprint" "valve_pcb_footprints:R_0603_1608Metric"
 			(at 242.57 45.72 0)
 			(hide yes)
@@
 			)
 		)
-		(property "Footprint" "Resistor_SMD:R_0603_1608Metric"
+		(property "Footprint" "valve_pcb_footprints:R_0603_1608Metric"
 			(at 264.16 144.78 0)
 			(hide yes)
@@
 			)
 		)
-		(property "Footprint" "Resistor_SMD:R_0603_1608Metric"
+		(property "Footprint" "valve_pcb_footprints:R_0603_1608Metric"
 			(at 78.74 91.44 0)
 			(hide yes)
@@
 			)
 		)
-		(property "Footprint" "Resistor_SMD:R_0603_1608Metric"
+		(property "Footprint" "valve_pcb_footprints:R_0603_1608Metric"
 			(at 303.53 207.01 0)
 			(hide yes)
@@
 			)
 		)
-		(property "Footprint" "Resistor_SMD:R_0603_1608Metric"
+		(property "Footprint" "valve_pcb_footprints:R_0603_1608Metric"
 			(at 213.36 78.74 0)
 			(hide yes)
@@
 			)
 		)
-		(property "Footprint" "Resistor_SMD:R_0603_1608Metric"
+		(property "Footprint" "valve_pcb_footprints:R_0603_1608Metric"
 			(at 99.06 130.81 0)
 			(hide yes)
@@
 			)
 		)
-		(property "Footprint" "Resistor_SMD:R_0603_1608Metric"
+		(property "Footprint" "valve_pcb_footprints:R_0603_1608Metric"
 			(at 255.27 139.7 0)
 			(hide yes)
@@
 			)
 		)
-		(property "Footprint" "Resistor_SMD:R_0603_1608Metric"
+		(property "Footprint" "valve_pcb_footprints:R_0603_1608Metric"
 			(at 134.62 231.14 0)
 			(hide yes)
@@
 			)
 		)
-		(property "Footprint" "Resistor_SMD:R_0603_1608Metric"
+		(property "Footprint" "valve_pcb_footprints:R_0603_1608Metric"
 			(at 138.43 68.58 0)
 			(hide yes)
@@
 			)
 		)
-		(property "Footprint" "Resistor_SMD:R_0603_1608Metric"
+		(property "Footprint" "valve_pcb_footprints:R_0603_1608Metric"
 			(at 222.25 74.93 0)
 			(hide yes)
@@
 			)
 		)
-		(property "Footprint" "Resistor_SMD:R_0603_1608Metric"
+		(property "Footprint" "valve_pcb_footprints:R_0603_1608Metric"
 			(at 278.13 104.14 0)
 			(hide yes)
@@
 			)
 		)
-		(property "Footprint" "Resistor_SMD:R_0603_1608Metric"
+		(property "Footprint" "valve_pcb_footprints:R_0603_1608Metric"
 			(at 195.58 133.35 0)
 			(hide yes)
@@
 			)
 		)
+		(property "Footprint_Size" ""
+			(at 195.58 133.35 0)
+			(show_name no)
+			(do_not_autoplace no)
+			(effects
+				(font
+					(size 1.27 1.27)
+				)
+			)
+		)
 		(pin "1"
 		)
@@
 			)
 		)
-		(property "Footprint" "Resistor_SMD:R_0603_1608Metric"
+		(property "Footprint" "valve_pcb_footprints:R_0603_1608Metric"
 			(at 306.07 162.56 0)
 			(hide yes)
@@
 			)
 		)
-		(property "Footprint" "Resistor_SMD:R_0603_1608Metric"
+		(property "Footprint" "valve_pcb_footprints:R_0603_1608Metric"
 			(at 68.58 130.81 0)
 			(hide yes)
@@
 			)
 		)
-		(property "Footprint" "Resistor_SMD:R_0603_1608Metric"
+		(property "Footprint" "valve_pcb_footprints:R_0603_1608Metric"
 			(at 185.42 133.35 0)
 			(hide yes)
@@
 		(dnp no)
 		(property "Reference" "R258"
-			(at 125.984 228.6 0)
+			(at 127 228.854 0)
 			(show_name no)
 			(do_not_autoplace no)
@@
 		)
 		(property "Value" "10k"
-			(at 126.492 231.14 0)
+			(at 126.238 230.632 0)
 			(show_name no)
 			(do_not_autoplace no)
@@
 			)
 		)
-		(property "Footprint" "Resistor_SMD:R_0603_1608Metric"
+		(property "Footprint" "valve_pcb_footprints:R_0603_1608Metric"
 			(at 123.19 231.14 0)
 			(hide yes)
@@
 		)
 		(property "Tolerance" "1%"
-			(at 125.476 233.426 0)
+			(at 125.984 232.664 0)
 			(show_name no)
 			(do_not_autoplace no)
@@
 			)
 		)
+		(property "Footprint_Size" "0603"
+			(at 127 234.442 0)
+			(show_name no)
+			(do_not_autoplace no)
+			(effects
+				(font
+					(size 1.27 1.27)
+				)
+			)
+		)
 		(pin "1"
 		)
@@
 		(dnp no)
 		(property "Reference" "R261"
-			(at 151.384 228.6 0)
+			(at 152.4 228.6 0)
 			(show_name no)
 			(do_not_autoplace no)
@@
 		)
 		(property "Value" "10k"
-			(at 151.892 231.14 0)
+			(at 151.892 230.378 0)
 			(show_name no)
 			(do_not_autoplace no)
@@
 			)
 		)
-		(property "Footprint" "Resistor_SMD:R_0603_1608Metric"
+		(property "Footprint" "valve_pcb_footprints:R_0603_1608Metric"
 			(at 148.59 231.14 0)
 			(hide yes)
@@
 		)
 		(property "Tolerance" "1%"
-			(at 150.876 233.426 0)
+			(at 151.638 232.156 0)
 			(show_name no)
 			(do_not_autoplace no)
@@
 			(show_name no)
 			(do_not_autoplace no)
+			(effects
+				(font
+					(size 1.27 1.27)
+				)
+			)
+		)
+		(property "Footprint_Size" "0603"
+			(at 152.654 233.934 0)
+			(show_name no)
+			(do_not_autoplace no)

Commit message: Major changes
Parts:
- C134, C140: footprint Capacitor_SMD:C_0805_2012Metric -> valve_pcb_footprints:C_0805_2012Metric
Changed lines of the file:
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@@
 	(title_block
 		(title "IGNITER SYSTEM")
-		(date "2026-10-07")
+		(date "2026-10-08")
 		(rev "A")
 	)
@@
 			)
 		)
-		(property "Footprint" "Capacitor_SMD:C_0805_2012Metric"
+		(property "Footprint" "valve_pcb_footprints:C_0805_2012Metric"
 			(at 316.23 90.17 0)
 			(hide yes)
@@
 			)
 		)
-		(property "Footprint" "Capacitor_SMD:C_0805_2012Metric"
+		(property "Footprint" "valve_pcb_footprints:C_0805_2012Metric"
 			(at 97.79 91.44 0)
 			(hide yes)

Commit message: Small updates
Parts:
- removed D29, D38: RED, LED_SMD:LED_0603_1608Metric, symbol Device:LED
- added D51, D52: WHITE, LED_SMD:LED_0603_1608Metric, symbol Device:LED
- D45, D46, D48: value RED -> WHITE; JLCPCB Part # C2286 -> C2290; Vf 2V -> 3.1V
- R247: JLCPCB Part # C13167 -> C23231
Connections:
- net GND: now also D51.1 (K), D52.1 (K)
- net at R262.2: now also D52.2 (A); no longer D46.2 (A)
- net at R258.2: now also D45.2 (A)
- net at R259.2: now also D46.2 (A)
- net at R261.2: now also D51.2 (A); no longer D45.2 (A)

Commit message: Fixes
Added hops, fixed the planes, and fixed minor issues
Parts:
- renumbered C133 to C64, C134 to C65, C135 to C66, C136 to C67, C137 to C68, C138 to C69, C139 to C70, C140 to C71, C141 to C72, C142 to C73, C143 to C74, D45 to D22, D46 to D23, D51 to D24, D52 to D25, D47 to D26, D48 to D27, D49 to D28, D50 to D29, F2 to F1, J18 to J10, J19 to J11, J20 to J12, J21 to J13, Q13 to Q11, Q14 to Q12, Q15 to Q13, Q16 to Q14, R244 to R110, R245 to R111, R247 to R112, R252 to R113, R253 to R114, R258 to R115, R259 to R116, R260 to R117, R261 to R118, R262 to R119, R263 to R120, R264 to R121, R265 to R122, R266 to R123, R267 to R124, R268 to R125, R269 to R126, R270 to R127, R271 to R128, R272 to R129, R273 to R130, R274 to R131, R275 to R132, R276 to R133, R277 to R134, R278 to R135, TP62 to TP100, TP63 to TP101, TP64 to TP102, TP65 to TP103, TP66 to TP104, TP67 to TP105, TP68 to TP106, TP69 to TP107, TP70 to TP108, TP71 to TP109, TP41 to TP97, TP56 to TP98, TP61 to TP99, U28 to U16

Commit message: Delete a bunch of stuff
Parts:
- removed J12, J13: 1x2 Screw Terminal, TerminalBlock_Phoenix:TerminalBlock_Phoenix_MKDS-1,5-2-5.08_1x02_P5.08mm_Horizontal, symbol Connector:Screw_Terminal_01x02
- added J12: 0768290102, valve_pcb_footprints:768290102, symbol Connector_Generic:Conn_01x02
- added J13: 0039299047, valve_pcb_footprints:Molex_Mini-Fit_Jr_5566-04A2_2x02_P4.20mm_Vertical, symbol Connector_Generic:Conn_02x02_Counter_Clockwise
Connections:
- net +5V: no longer C73.1
- net GND: now also J13.1 (Pin_1), J13.2 (Pin_2)
- net at C69.1, C70.1, C71.1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: now also J13.3 (Pin_3), J13.4 (Pin_4)
- net at Q14.3 (D): now also J12.2 (Pin_2)
- new net +12V: C73.1, J12.1 (Pin_1)

Commit message: Commit
Other:
- note added: "LED"
- note added: "SW"
Changed lines of the file:
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@@
+		)
+	)
+	(text "SW"
+		(exclude_from_sim no)
+		(at 199.644 47.498 0)
+		(effects
+			(font
+				(size 1.27 1.27)
+			)
 		)
 	)
@@
 		(exclude_from_sim no)
 		(at 183.134 83.058 0)
+		(effects
+			(font
+				(size 1.27 1.27)
+			)
+		)
+	)
+	(text "LED"
+		(exclude_from_sim no)
+		(at 199.39 52.324 0)
 		(effects
 			(font
@@
 		)
 		(stroke
+			(width 0)
+			(type default)
+		)
+	)
+	(polyline
+		(pts
+			(xy 195.58 49.53) (xy 200.66 49.53)
+		)
+		(stroke
