File: LRUs/Valve Control Unit/Electrical/Valve Power Board/valve_control_pcb/master_efuse.kicad_sch (KiCad schematic)
At the start: 14 parts

Commit message: Commit valve board updates
Parts:
- removed R137: 10k, Resistor_SMD:R_0603_1608Metric, symbol Device:R_Small_US
- added TP129, TP130, TP131, TP132, TP133, TP134, TP135, TP136, TP137, TP138: TestPoint, TestPoint:TestPoint_Pad_D1.0mm, symbol Connector:TestPoint
- R134: value 150k -> 1M; Footprint_Size (none) -> 0603; JLCPCB Part # C22807 -> C22935
- R135: value 18k -> 100k; Footprint_Size (none) -> 0603; JLCPCB Part # C25810 -> C25803
- R136: value 27k -> 22k; Footprint_Size (none) -> 0603; JLCPCB Part # C22967 -> C31850
- R138, R139, R143: Footprint_Size (none) -> 0603
- U26: value (none) -> TPS259830
Connections:
- net DVDT: now also TP131.1
- net GND: now also R135.1, TP135.1, TP136.1
- net ILIM: now also TP132.1
- net IMON_IC: now also TP133.1
- net ITIM: now also TP134.1
- net VIN: now also TP138.1
- net VOUT: now also TP137.1
- net at R136.2, U26.6 (EN/UVLO): now also R134.1, TP129.1; no longer R135.1
- net at R135.2: now also R136.1, U26.12 (OVLO), TP130.1; no longer R134.1
Other:
- note added: "4mΩ * 12A = 48mW"
- note added: "EFUSE"
- title: (none) -> EFUSE
- moved on the sheet: C83, C84, R140, R141, R142, R143

Commit message: Commit da changes
Parts:
- removed TP136: TestPoint, TestPoint:TestPoint_Pad_D1.0mm, symbol Connector:TestPoint
- added J27: B2B-XH-A, Connector_JST:JST_XH_B2B-XH-A_1x02_P2.50mm_Vertical, symbol Connector_Generic:Conn_01x02
- C82, C83: footprint Capacitor_SMD:C_0603_1608Metric -> valve_pcb_footprints:C_0603_1608Metric
- C84: footprint Capacitor_SMD:C_0402_1005Metric -> valve_pcb_footprints:C_0402_1005Metric
- R134, R135, R136, R138, R139, R140, R141, R142, R143: footprint Resistor_SMD:R_0603_1608Metric -> valve_pcb_footprints:R_0603_1608Metric
- U26: JLCPCB Part # (none) -> C20607218
Connections:
- net at R136.2, TP129.1, U26.6 (EN/UVLO): now also J27.2 (Pin_2); no longer R134.1
- new net: J27.1 (Pin_1), R134.1
Other:
- note removed: "4mΩ * 12A = 48mW"
- moved on the sheet: C82, C83, C84, R134, R135, R136, R138, R139, R140, R141, R142, R143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

Commit message: Fixes
Added hops, fixed the planes, and fixed minor issues
Parts:
- renumbered C82 to C37, C83 to C38, C84 to C39, J27 to J5, R134 to R41, R136 to R42, R135 to R43, R138 to R44, R139 to R45, R141 to R46, R140 to R47, R142 to R48, R143 to R49, TP138 to TP24, TP129 to TP25, TP130 to TP26, TP135 to TP27, TP131 to TP28, TP134 to TP29, TP133 to TP30, TP132 to TP31, TP137 to TP32, U26 to U9

Commit message: Commit
Connections:
- net VALVE_EN: now reaches J5.2 (Pin_2), R42.2, TP25.1, U9.6 (EN/UVLO)
Changed lines of the file:
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@@
+		)
+	)
+	(label "VALVE_EN"
+		(at 113.03 92.71 0)
+		(effects
+			(font
+				(size 1.27 1.27)
+			)
+			(justify left bottom)
 		)
 	)
